Commit message: Adding collisions.

File: rough_mocks/urdf/mocks.xacro (robot description, xacro)
@@ -11,4 +11,13 @@
         </material>
       </visual>
+      <collision>
+        <origin xyz="0.0 0.0 ${1.6002/2}" rpy="0 0 0"/>
+        <geometry>
+          <box size="1.27 0.89535 1.6002"/>
+        </geometry>
+        <material name="red">
+          <color rgba="1.0 0 0 0.5"/>
+        </material>
+      </collision>
     </link>
     <joint name="trainer_bench" type="fixed">
@@ -27,4 +36,13 @@
         </material>
       </visual>
+      <collision>
+        <origin xyz="0.0 0.0 ${0.10/2}" rpy="0 0 0"/>
+        <geometry>
+          <box size="0.7112 0.89535 0.10"/>
+        </geometry>
+        <material name="green">
+          <color rgba="0.0 1.0 0 0.5"/>
+        </material>
+      </collision>
     </link>
     <joint name="trainer_hatch" type="fixed">
@@ -43,4 +61,13 @@
         </material>
       </visual>
+      <collision>
+        <origin xyz="0.0 0.0 ${0.508/2}" rpy="0 0 0"/>
+        <geometry>
+          <box size="0.635 1.27 0.508"/>
+        </geometry>
+        <material name="blue">
+          <color rgba="0.0 0 1.0 0.5"/>
+        </material>
+      </collision>
     </link>
     <joint name="hatch_bottom_left" type="fixed">
@@ -59,4 +86,13 @@
         </material>
       </visual>
+      <collision>
+        <origin xyz="0.0 0.0 ${1.016/2}" rpy="0 0 0"/>
+        <geometry>
+          <box size="0.635 0.127 1.016"/>
+        </geometry>
+        <material name="blue">
+          <color rgba="0.0 0 1.0 0.5"/>
+        </material>
+      </collision>
     </link>
     <joint name="hatch_bottom_right" type="fixed">
@@ -75,4 +111,13 @@
         </material>
       </visual>
+      <collision>
+        <origin xyz="0.0 0.0 ${1.016/2}" rpy="0 0 0"/>
+        <geometry>
+          <box size="0.635 0.127 1.016"/>
+        </geometry>
+        <material name="blue">
+          <color rgba="0.0 0 1.0 0.5"/>
+        </material>
+      </collision>
     </link>
     <joint name="hatch_bottom_top" type="fixed">
@@ -91,4 +136,13 @@
         </material>
       </visual>
+      <collision>
+        <origin xyz="0.0 0.0 ${0.5842/2}" rpy="0 0 0"/>
+        <geometry>
+          <box size="0.635 1.27 0.5842"/>
+        </geometry>
+        <material name="blue">
+          <color rgba="0.0 0 1.0 0.5"/>
+        </material>
+      </collision>
     </link>
 </robot>
