Commit message: Adding the bench.

File: combined_mocks/urdf/combined_mocks.urdf.xacro (robot description, xacro)
@@ -5,8 +5,12 @@
   <xacro:include filename="$(find trainer)/urdf/trainer_frame.xacro"/>
   <xacro:include filename="$(find hatch_frame)/urdf/hatch_frame.xacro"/>
+  <xacro:include filename="$(find bench)/urdf/bench_seat.xacro"/>
   <link name="world"/>
   <xacro:trainer_frame name="$(arg name)" prefix="$(arg prefix)" parent="world">
-    <origin xyz="0 0 0" rpy="0 0 0"/>
+    <origin xyz="0.0 0 0" rpy="0 0 0"/>
   </xacro:trainer_frame>
+  <xacro:bench_seat name="$(arg name)" prefix="$(arg prefix)" parent="world">
+    <origin xyz="1.27 0 0.4969" rpy="0 0 0"/>
+  </xacro:bench_seat>
   <xacro:hatch_frame name="$(arg name)" prefix="$(arg prefix)" parent="world">
     <origin xyz="0 0.896112 0" rpy="0 0 0"/>
