Commit message: Adding colors.

File: hatch_frame/urdf/hatch_frame.urdf.xacro (robot description, xacro)
@@ -3,4 +3,5 @@
   <xacro:arg name="name" default=""/>
   <xacro:arg name="prefix" default=""/>
+  <xacro:include filename="$(find hatch_frame)/urdf/colors.xacro"/>
   <xacro:include filename="$(find hatch_frame)/urdf/hatch_frame.xacro"/>
   <link name="world"/>

File: hatch_frame/urdf/hatch_frame.xacro (robot description, xacro)
@@ -17,7 +17,5 @@
             <mesh filename="file://$(find hatch_frame)/meshes/visual/ivr_hatch_frame.stl"/>
           </geometry>
-        <material name="red">
-          <color rgba="1.0 0 0 0.75"/>
-        </material>
+        <material name="gray"/>
       </visual>
     </link>
@@ -28,5 +26,5 @@
     </joint>
     <link name="hatch_bottom">
-      <!--TODO: set proper inertia-->
+      <!--TODO set proper inertia-->
       <inertial>
         <origin rpy="0 0 0" xyz="0.0 0.0 0.0"/>
@@ -39,7 +37,5 @@
           <box size="0.675 1.307 0.04"/>
         </geometry>
-        <material name="blue">
-          <color rgba="0.0 0.0 1.0 1.0"/>
-        </material>
+        <material name="red"/>
       </collision>
     </link>
@@ -55,7 +51,5 @@
           <box size="0.1 1.307 0.610"/>
         </geometry>
-        <material name="blue">
-          <color rgba="0.0 0.0 1.0 1.0"/>
-        </material>
+        <material name="red"/>
       </collision>
     </link>
@@ -71,7 +65,5 @@
           <box size="0.1 1.307 0.610"/>
         </geometry>
-        <material name="blue">
-          <color rgba="0.0 0.0 1.0 1.0"/>
-        </material>
+        <material name="red"/>
       </collision>
     </link>
@@ -87,7 +79,5 @@
           <box size="0.675 0.1 2.1082"/>
         </geometry>
-        <material name="blue">
-          <color rgba="0.0 0.0 1.0 1.0"/>
-        </material>
+        <material name="red"/>
       </collision>
     </link>
@@ -103,7 +93,5 @@
           <box size="0.675 0.1 2.1082"/>
         </geometry>
-        <material name="blue">
-          <color rgba="0.0 0.0 1.0 1.0"/>
-        </material>
+        <material name="red"/>
       </collision>
     </link>
@@ -119,7 +107,5 @@
           <box size="0.1 1.307 0.197"/>
         </geometry>
-        <material name="blue">
-          <color rgba="0.0 0.0 1.0 1.0"/>
-        </material>
+        <material name="red"/>
       </collision>
     </link>
