Commit message: Adding the 2nd cubby.

File: trainer/urdf/trainer.urdf.xacro (robot description, xacro)
@@ -11,8 +11,11 @@
   </xacro:trainer_frame>
   <xacro:side_face name="$(arg name)" prefix="$(arg prefix)" parent="world">
-    <origin xyz="0.8119 0.8865 0.04" rpy="0 0 0"/>
+    <origin xyz="0.812 0.887 0.04" rpy="0 0 0"/>
   </xacro:side_face>
-  <xacro:cubby name="$(arg name)" prefix="$(arg prefix)" parent="world">
-    <origin xyz="1.2596 0.04 0.8308" rpy="0 0 0"/>
+  <xacro:cubby name="$(arg name)" prefix="$(arg prefix)1_" parent="trainer_frame">
+    <origin xyz="1.260 0.254 0.830" rpy="0 0 0"/>
+  </xacro:cubby>
+  <xacro:cubby name="$(arg name)" prefix="$(arg prefix)2_" parent="trainer_frame">
+    <origin xyz="1.260 0.254 1.162" rpy="0 0 0"/>
   </xacro:cubby>
 </robot>

Commit message: Combining bench and adding ceiling.

File: trainer/urdf/trainer.urdf.xacro (robot description, xacro)
@@ -3,14 +3,22 @@
   <xacro:arg name="name" default=""/>
   <xacro:arg name="prefix" default=""/>
+  <xacro:property name="ceiling_prop" value="true"/>
   <xacro:include filename="$(find trainer)/urdf/trainer_frame.xacro"/>
+  <xacro:include filename="$(find trainer)/urdf/bench_seat.xacro"/>
+  <xacro:include filename="$(find trainer)/urdf/trainer_cubby.xacro"/>
   <xacro:include filename="$(find trainer)/urdf/trainer_side.xacro"/>
-  <xacro:include filename="$(find trainer)/urdf/trainer_cubby.xacro"/>
   <link name="world"/>
   <xacro:trainer_frame name="$(arg name)" prefix="$(arg prefix)" parent="world">
     <origin xyz="0 0 0" rpy="0 0 0"/>
   </xacro:trainer_frame>
-  <xacro:side_face name="$(arg name)" prefix="$(arg prefix)" parent="world">
-    <origin xyz="0.812 0.887 0.04" rpy="0 0 0"/>
-  </xacro:side_face>
+  <xacro:bench_seat name="$(arg name)" prefix="$(arg prefix)" parent="trainer_frame">
+    <origin xyz="1.27 0 0.4969" rpy="0 0 0"/>
+  </xacro:bench_seat>
+  <xacro:if value="${ceiling_prop}">
+    <xacro:include filename="$(find trainer)/urdf/ceiling.xacro"/>
+    <xacro:ceiling name="$(arg name)" prefix="$(arg prefix)" parent="trainer_frame">
+      <origin xyz="0.0 0.0 1.6002" rpy="0 0 0"/>
+    </xacro:ceiling>
+  </xacro:if>
   <xacro:cubby name="$(arg name)" prefix="$(arg prefix)1_" parent="trainer_frame">
     <origin xyz="1.260 0.254 0.830" rpy="0 0 0"/>
@@ -19,3 +27,6 @@
     <origin xyz="1.260 0.254 1.162" rpy="0 0 0"/>
   </xacro:cubby>
+  <xacro:side_face name="$(arg name)" prefix="$(arg prefix)" parent="trainer_frame">
+    <origin xyz="0.812 0.887 0.04" rpy="0 0 0"/>
+  </xacro:side_face>
 </robot>

Commit message: Adding the left front face plate.

File: trainer/urdf/trainer.urdf.xacro (robot description, xacro)
@@ -6,4 +6,5 @@
   <xacro:include filename="$(find trainer)/urdf/trainer_frame.xacro"/>
   <xacro:include filename="$(find trainer)/urdf/bench_seat.xacro"/>
+  <xacro:include filename="$(find trainer)/urdf/trainer_front.xacro"/>
   <xacro:include filename="$(find trainer)/urdf/trainer_cubby.xacro"/>
   <xacro:include filename="$(find trainer)/urdf/trainer_side.xacro"/>
@@ -21,4 +22,7 @@
     </xacro:ceiling>
   </xacro:if>
+  <xacro:front_face_plate name="$(arg name)" prefix="$(arg prefix)" parent="world">
+    <origin xyz="1.25 0.08 0.45683932" rpy="0 0 0"/>
+  </xacro:front_face_plate>
   <xacro:cubby name="$(arg name)" prefix="$(arg prefix)1_" parent="trainer_frame">
     <origin xyz="1.260 0.254 0.830" rpy="0 0 0"/>

File: trainer/urdf/trainer_front.urdf.xacro (robot description, xacro)
@@ -5,6 +5,6 @@
   <xacro:include filename="$(find trainer)/urdf/trainer_front.xacro"/>
   <link name="world"/>
-  <xacro:trainer_front name="$(arg name)" prefix="$(arg prefix)" parent="world">
+  <xacro:front_face_plate name="$(arg name)" prefix="$(arg prefix)" parent="world">
     <origin xyz="0 0 0" rpy="0 0 0"/>
-  </xacro:trainer_front>
+  </xacro:front_face_plate>
 </robot>

Commit message: Needs cleaned up but the cubbies are in the right place.

File: trainer/urdf/trainer.urdf.xacro (robot description, xacro)
@@ -3,11 +3,12 @@
   <xacro:arg name="name" default=""/>
   <xacro:arg name="prefix" default=""/>
+  <xacro:property name="shelf" default="false"/>
   <xacro:property name="ceiling_prop" value="true"/>
+  <link name="world"/>
   <xacro:include filename="$(find trainer)/urdf/trainer_frame.xacro"/>
-  <xacro:include filename="$(find trainer)/urdf/bench_seat.xacro"/>
-  <link name="world"/>
   <xacro:trainer_frame name="$(arg name)" prefix="$(arg prefix)" parent="world">
     <origin xyz="0 0 0" rpy="0 0 0"/>
   </xacro:trainer_frame>
+  <xacro:include filename="$(find trainer)/urdf/bench_seat.xacro"/>
   <xacro:bench_seat name="$(arg name)" prefix="$(arg prefix)" parent="trainer_frame">
     <origin xyz="1.27 0 0.4969" rpy="0 0 0"/>
@@ -19,20 +20,11 @@
     </xacro:ceiling>
   </xacro:if>
-  <xacro:include filename="$(find trainer)/urdf/trainer_front.xacro"/>
-  <xacro:front_face_plate name="$(arg name)" prefix="$(arg prefix)" parent="world">
+  <xacro:include filename="$(find trainer)/urdf/trainer_front_left_face.xacro"/>
+  <xacro:trainer_front_left_face name="$(arg name)" prefix="$(arg prefix)" parent="trainer_frame" shelf="${shelf}">
     <origin xyz="1.25 0.08 0.45683932" rpy="0 0 0"/>
-  </xacro:front_face_plate>
-  <xacro:include filename="$(find trainer)/urdf/trainer_cubby.xacro"/>
-  <xacro:cubby name="$(arg name)" prefix="$(arg prefix)1_" parent="trainer_frame">
-    <origin xyz="1.260 0.254 0.830" rpy="0 0 0"/>
-  </xacro:cubby>
-  <xacro:cubby name="$(arg name)" prefix="$(arg prefix)2_" parent="trainer_frame">
-    <origin xyz="1.260 0.254 1.162" rpy="0 0 0"/>
-  </xacro:cubby>
-  <!--
+  </xacro:trainer_front_left_face>
   <xacro:include filename="$(find trainer)/urdf/trainer_side.xacro"/>
   <xacro:side_face name="$(arg name)" prefix="$(arg prefix)" parent="trainer_frame">
     <origin xyz="0.812 0.887 0.04" rpy="0 0 0"/>
   </xacro:side_face>
-  -->
 </robot>

File: trainer/urdf/trainer_cubby_2.urdf.xacro (robot description, xacro)
@@ -3,5 +3,5 @@
   <xacro:arg name="name" default=""/>
   <xacro:arg name="prefix" default=""/>
-  <xacro:include filename="$(find trainer)/urdf/trainer_cubby_1.xacro"/>
+  <xacro:include filename="$(find trainer)/urdf/trainer_cubby_2.xacro"/>
   <link name="world"/>
   <xacro:cubby name="$(arg name)" prefix="$(arg prefix)" parent="world">

Commit message: Adding right front face.

File: trainer/urdf/trainer.urdf.xacro (robot description, xacro)
@@ -22,6 +22,10 @@
   <xacro:include filename="$(find trainer)/urdf/trainer_front_left_face.xacro"/>
   <xacro:trainer_front_left_face name="$(arg name)" prefix="$(arg prefix)" parent="trainer_frame" shelf="${shelf}">
-    <origin xyz="1.25 0.08 0.45683932" rpy="0 0 0"/>
+    <origin xyz="1.25 0.08 0.457" rpy="0 0 0"/>
   </xacro:trainer_front_left_face>
+  <xacro:include filename="$(find trainer)/urdf/trainer_front_right_face.xacro"/>
+  <xacro:trainer_front_right_face name="$(arg name)" prefix="$(arg prefix)" parent="trainer_frame">
+    <origin xyz="1.25 0.465 0.457" rpy="0 0 0"/>
+  </xacro:trainer_front_right_face>
   <xacro:include filename="$(find trainer)/urdf/trainer_side.xacro"/>
   <xacro:side_face name="$(arg name)" prefix="$(arg prefix)" parent="trainer_frame">

File: trainer/urdf/trainer_front_left_face.xacro (robot description, xacro)
@@ -7,5 +7,5 @@
     *origin
     shelf:='true'">
-  <joint name="${prefix}trainer_front_face_base_joint" type="fixed">
+  <joint name="${prefix}trainer_front_left_face_joint" type="fixed">
     <parent link="${parent}"/>
     <child link="${prefix}front_left_face"/>
