Commit message: Switching to global colors.

File: trainer/urdf/bench_seat.urdf.xacro (robot description, xacro)
@@ -4,4 +4,16 @@
   <xacro:arg name="prefix" default=""/>
   <xacro:include filename="$(find trainer)/urdf/bench_seat.xacro"/>
+  <material name="red">
+    <color rgba="1.0 0 0 1"/>
+  </material>
+  <material name="green">
+    <color rgba="1.0 0 0 1"/>
+  </material>
+  <material name="blue">
+    <color rgba="0 0 1.0 1"/>
+  </material>
+  <material name="gray">
+    <color rgba="0.85 0.85 0.85 0.75"/>
+  </material>
   <link name="world"/>
   <xacro:bench_seat name="$(arg name)" prefix="$(arg prefix)" parent="world">

File: trainer/urdf/bench_seat.xacro (robot description, xacro)
@@ -23,7 +23,5 @@
           <box size="0.127 0.895 0.05"/>
         </geometry>
-        <material name="gray">
-          <color rgba="0.85 0.85 0.85 0.75"/>
-        </material>
+        <material name="gray"/>
       </visual>
       <collision>
@@ -32,7 +30,5 @@
           <box size="0.127 0.895 0.05"/>
         </geometry>
-        <material name="red">
-          <color rgba="1.0 0.0 0.0 0.75"/>
-        </material>
+        <material name="red"/>
       </collision>
     </link>
@@ -48,7 +44,5 @@
           <box size="0.708 0.05 0.05"/>
         </geometry>
-        <material name="gray">
-          <color rgba="0.85 0.85 0.85 0.75"/>
-        </material>
+        <material name="gray"/>
       </visual>
       <collision>
@@ -57,7 +51,5 @@
           <box size="0.708 0.05 0.05"/>
         </geometry>
-        <material name="red">
-          <color rgba="1.0 0.0 0.0 0.75"/>
-        </material>
+        <material name="red"/>
       </collision>
     </link>
@@ -73,7 +65,5 @@
           <box size="0.708 0.05 0.05"/>
         </geometry>
-        <material name="gray">
-          <color rgba="0.85 0.85 0.85 0.75"/>
-        </material>
+        <material name="gray"/>
       </visual>
       <collision>
@@ -82,7 +72,5 @@
           <box size="0.708 0.05 0.05"/>
         </geometry>
-        <material name="red">
-          <color rgba="1.0 0.0 0.0 0.75"/>
-        </material>
+        <material name="red"/>
       </collision>
     </link>
@@ -98,7 +86,5 @@
           <box size="0.05 0.895 0.05"/>
         </geometry>
-        <material name="gray">
-          <color rgba="0.85 0.85 0.85 0.75"/>
-        </material>
+        <material name="gray"/>
       </visual>
       <collision>
@@ -107,7 +93,5 @@
           <box size="0.05 0.895 0.05"/>
         </geometry>
-        <material name="red">
-          <color rgba="1.0 0.0 0.0 0.75"/>
-        </material>
+        <material name="red"/>
       </collision>
     </link>
@@ -131,7 +115,5 @@
           <box size="0.603 0.895 0.05"/>
         </geometry>
-        <material name="blue">
-          <color rgba="0.0 0.0 1.0 0.5"/>
-        </material>
+        <material name="blue"/>
       </visual>
       <collision>
@@ -140,7 +122,5 @@
           <box size="0.603 0.895 0.05"/>
         </geometry>
-        <material name="blue">
-          <color rgba="0.0 0.0 1.0 0.5"/>
-        </material>
+        <material name="blue"/>
       </collision>
     </link>

File: trainer/urdf/ceiling.xacro (robot description, xacro)
@@ -17,7 +17,5 @@
           <box size="1.901 1.4694 0.05"/>
         </geometry>
-        <material name="gray">
-          <color rgba="0.85 0.85 0.85 0.75"/>
-        </material>
+        <material name="gray"/>
       </visual>
       <collision>
@@ -26,7 +24,5 @@
           <box size="1.901 1.4694 0.05"/>
         </geometry>
-        <material name="red">
-          <color rgba="1.0 0.0 0.0 0.75"/>
-        </material>
+        <material name="red"/>
       </collision>
     </link>

File: trainer/urdf/trainer.urdf.xacro (robot description, xacro)
@@ -5,4 +5,16 @@
   <xacro:property name="shelf" default="false"/>
   <xacro:property name="ceiling_prop" value="true"/>
+  <material name="red">
+    <color rgba="1.0 0 0 1"/>
+  </material>
+  <material name="green">
+    <color rgba="1.0 0 0 1"/>
+  </material>
+  <material name="blue">
+    <color rgba="0 0 1.0 1"/>
+  </material>
+  <material name="gray">
+    <color rgba="0.85 0.85 0.85 0.75"/>
+  </material>
   <link name="world"/>
   <xacro:include filename="$(find trainer)/urdf/trainer_frame.xacro"/>

File: trainer/urdf/trainer_frame.urdf.xacro (robot description, xacro)
@@ -4,4 +4,16 @@
   <xacro:arg name="prefix" default=""/>
   <xacro:include filename="$(find trainer)/urdf/trainer_frame.xacro"/>
+  <material name="red">
+    <color rgba="1.0 0 0 1"/>
+  </material>
+  <material name="green">
+    <color rgba="1.0 0 0 1"/>
+  </material>
+  <material name="blue">
+    <color rgba="0 0 1.0 1"/>
+  </material>
+  <material name="gray">
+    <color rgba="0.85 0.85 0.85 0.75"/>
+  </material>
   <link name="world"/>
   <xacro:trainer_frame name="$(arg name)" prefix="$(arg prefix)" parent="world">

File: trainer/urdf/trainer_frame.xacro (robot description, xacro)
@@ -17,7 +17,5 @@
           <mesh filename="file://$(find trainer)/meshes/visual/ivr_tasktrainer_frame.stl"/>
         </geometry>
-        <material name="gray">
-          <color rgba="0.85 0.85 0.85 0.75"/>
-        </material>
+        <material name="gray"/>
       </visual>
     </link>
@@ -39,7 +37,5 @@
           <box size="1.27 0.816 0.47"/>
         </geometry>
-        <material name="red">
-          <color rgba="1.0 0 0 0.5"/>
-        </material>
+        <material name="red"/>
       </collision>
     </link>
@@ -55,7 +51,5 @@
           <box size="1.27 0.816 0.1"/>
         </geometry>
-        <material name="red">
-          <color rgba="1.0 0 0 1.0"/>
-        </material>
+        <material name="red"/>
       </collision>
     </link>
@@ -71,7 +65,5 @@
           <box size="1.27 0.1 1.60"/>
         </geometry>
-        <material name="red">
-          <color rgba="1.0 0 0 0.5"/>
-        </material>
+        <material name="red"/>
       </collision>
     </link>
@@ -87,7 +79,5 @@
           <box size="1.27 0.05 1.60"/>
         </geometry>
-        <material name="red">
-          <color rgba="1.0 0 0 0.5"/>
-        </material>
+        <material name="red"/>
       </collision>
     </link>
@@ -103,7 +93,5 @@
           <box size="0.810 0.1 1.60"/>
         </geometry>
-        <material name="red">
-          <color rgba="1.0 0 0 0.5"/>
-        </material>
+        <material name="red"/>
       </collision>
     </link>
@@ -119,7 +107,5 @@
           <box size="0.13335 0.1 1.60"/>
         </geometry>
-        <material name="red">
-          <color rgba="1.0 0 0 0.5"/>
-        </material>
+        <material name="red"/>
       </collision>
     </link>

File: trainer/urdf/trainer_front_left_face.urdf.xacro (robot description, xacro)
@@ -4,4 +4,16 @@
   <xacro:arg name="prefix" default=""/>
   <xacro:property name="shelf" default="true"/>
+  <material name="red">
+    <color rgba="1.0 0 0 1"/>
+  </material>
+  <material name="green">
+    <color rgba="1.0 0 0 1"/>
+  </material>
+  <material name="blue">
+    <color rgba="0 0 1.0 1"/>
+  </material>
+  <material name="gray">
+    <color rgba="0.85 0.85 0.85 0.75"/>
+  </material>
   <link name="world"/>
   <xacro:include filename="$(find trainer)/urdf/trainer_front_left_face.xacro"/>

File: trainer/urdf/trainer_front_left_face.xacro (robot description, xacro)
@@ -24,7 +24,5 @@
         <mesh filename="file://$(find trainer)/meshes/visual/front_left_face.stl"/>
       </geometry>
-      <material name="gray">
-        <color rgba="0.85 0.85 0.85 0.75"/>
-      </material>
+      <material name="gray"/>
     </visual>
     <collision>
@@ -33,7 +31,5 @@
         <mesh filename="file://$(find trainer)/meshes/collision/front_left_face.stl"/>
       </geometry>
-      <material name="red">
-        <color rgba="1.0 0 0 0.75"/>
-      </material>
+      <material name="red"/>
     </collision>
   </link>
@@ -55,7 +51,5 @@
         <mesh filename="file://$(find trainer)/meshes/visual/cubby_1.stl"/>
       </geometry>
-      <material name="gray">
-        <color rgba="0.85 0.85 0.85 0.75"/>
-      </material>
+      <material name="gray"/>
     </visual>
     <collision>
@@ -64,7 +58,5 @@
         <mesh filename="file://$(find trainer)/meshes/collision/cubby_1.stl"/>
       </geometry>
-      <material name="red">
-        <color rgba="1.0 0 0 0.75"/>
-      </material>
+      <material name="red"/>
     </collision>
   </link>
@@ -86,7 +78,5 @@
         <mesh filename="file://$(find trainer)/meshes/visual/cubby_2.stl"/>
       </geometry>
-      <material name="gray">
-        <color rgba="0.85 0.85 0.85 0.75"/>
-      </material>
+      <material name="gray"/>
     </visual>
     <collision>
@@ -95,7 +85,5 @@
         <mesh filename="file://$(find trainer)/meshes/collision/cubby_2.stl"/>
       </geometry>
-      <material name="red">
-        <color rgba="1.0 0 0 0.75"/>
-      </material>
+      <material name="red"/>
     </collision>
   </link>
@@ -118,7 +106,5 @@
           <box size="0.173 0.428 0.02"/>
         </geometry>
-        <material name="gray">
-          <color rgba="0.85 0.85 0.85 0.75"/>
-        </material>
+        <material name="gray"/>
       </visual>
       <collision>
@@ -127,7 +113,5 @@
           <box size="0.173 0.428 0.02"/>
         </geometry>
-        <material name="red">
-          <color rgba="1.0 0.0 0 0.75"/>
-        </material>
+        <material name="red"/>
       </collision>
     </link>

File: trainer/urdf/trainer_front_right_face.urdf.xacro (robot description, xacro)
@@ -3,4 +3,16 @@
   <xacro:arg name="name" default=""/>
   <xacro:arg name="prefix" default=""/>
+  <material name="red">
+    <color rgba="1.0 0 0 1"/>
+  </material>
+  <material name="green">
+    <color rgba="1.0 0 0 1"/>
+  </material>
+  <material name="blue">
+    <color rgba="0 0 1.0 1"/>
+  </material>
+  <material name="gray">
+    <color rgba="0.85 0.85 0.85 0.75"/>
+  </material>
   <link name="world"/>
   <xacro:include filename="$(find trainer)/urdf/trainer_front_right_face.xacro"/>

File: trainer/urdf/trainer_front_right_face.xacro (robot description, xacro)
@@ -23,7 +23,5 @@
         <mesh filename="file://$(find trainer)/meshes/visual/front_right_face.stl"/>
       </geometry>
-      <material name="gray">
-        <color rgba="0.85 0.85 0.85 0.75"/>
-      </material>
+      <material name="gray"/>
     </visual>
     <collision>
@@ -32,7 +30,5 @@
         <mesh filename="file://$(find trainer)/meshes/collision/front_right_face.stl"/>
       </geometry>
-      <material name="red">
-        <color rgba="1.0 0 0 0.75"/>
-      </material>
+      <material name="red"/>
     </collision>
   </link>
@@ -56,7 +52,5 @@
         <mesh filename="file://$(find trainer)/meshes/visual/cabinet_door_1.stl"/>
       </geometry>
-      <material name="blue">
-        <color rgba="0 0 1.0 0.75"/>
-      </material>
+      <material name="blue"/>
     </visual>
     <collision>
@@ -65,7 +59,5 @@
         <mesh filename="file://$(find trainer)/meshes/collision/cabinet_door_1.stl"/>
       </geometry>
-      <material name="red">
-        <color rgba="1.0 0 0 0.75"/>
-      </material>
+      <material name="red"/>
     </collision>
   </link>
@@ -89,7 +81,5 @@
         <mesh filename="file://$(find trainer)/meshes/visual/cabinet_door_2.stl"/>
       </geometry>
-      <material name="blue">
-        <color rgba="0 0 1.0 0.75"/>
-      </material>
+      <material name="blue"/>
     </visual>
     <collision>
@@ -98,7 +88,5 @@
         <mesh filename="file://$(find trainer)/meshes/collision/cabinet_door_2.stl"/>
       </geometry>
-      <material name="red">
-        <color rgba="1.0 0 0 0.75"/>
-      </material>
+      <material name="red"/>
     </collision>
   </link>
@@ -122,7 +110,5 @@
         <mesh filename="file://$(find trainer)/meshes/visual/cabinet_door_3.stl"/>
       </geometry>
-      <material name="blue">
-        <color rgba="0 0 1.0 0.75"/>
-      </material>
+      <material name="blue"/>
     </visual>
     <collision>
@@ -131,7 +117,5 @@
         <mesh filename="file://$(find trainer)/meshes/collision/cabinet_door_3.stl"/>
       </geometry>
-      <material name="red">
-        <color rgba="1.0 0 0 0.75"/>
-      </material>
+      <material name="red"/>
     </collision>
   </link>

File: trainer/urdf/trainer_side.urdf.xacro (robot description, xacro)
@@ -4,4 +4,16 @@
   <xacro:arg name="prefix" default=""/>
   <xacro:include filename="$(find trainer)/urdf/trainer_side.xacro"/>
+  <material name="red">
+    <color rgba="1.0 0 0 1"/>
+  </material>
+  <material name="green">
+    <color rgba="1.0 0 0 1"/>
+  </material>
+  <material name="blue">
+    <color rgba="0 0 1.0 1"/>
+  </material>
+  <material name="gray">
+    <color rgba="0.85 0.85 0.85 0.75"/>
+  </material>
   <link name="world"/>
   <xacro:side_face name="$(arg name)" prefix="$(arg prefix)" parent="world">

File: trainer/urdf/trainer_side.xacro (robot description, xacro)
@@ -23,7 +23,5 @@
           <mesh filename="file://$(find trainer)/meshes/visual/side_bottom_face.stl"/>
         </geometry>
-        <material name="gray">
-          <color rgba="0.85 0.85 0.85 0.75"/>
-        </material>
+        <material name="gray"/>
       </visual>
       <collision>
@@ -32,7 +30,5 @@
             <mesh filename="file://$(find trainer)/meshes/collision/side_bottom_face.stl"/>
           </geometry>
-        <material name="red">
-          <color rgba="1.0 0 0 0.75"/>
-        </material>
+        <material name="red"/>
       </collision>
     </link>
@@ -54,7 +50,5 @@
           <mesh filename="file://$(find trainer)/meshes/visual/side_top_face.stl"/>
         </geometry>
-        <material name="gray">
-          <color rgba="0.85 0.85 0.85 0.75"/>
-        </material>
+        <material name="gray"/>
       </visual>
       <collision>
@@ -63,7 +57,5 @@
             <mesh filename="file://$(find trainer)/meshes/collision/side_top_face.stl"/>
           </geometry>
-        <material name="red">
-          <color rgba="1.0 0 0 0.75"/>
-        </material>
+        <material name="red"/>
       </collision>
     </link>
@@ -87,7 +79,5 @@
         <mesh filename="file://$(find trainer)/meshes/visual/cabinet_door_4.stl"/>
       </geometry>
-      <material name="blue">
-        <color rgba="0 0 1.0 0.75"/>
-      </material>
+      <material name="blue"/>
     </visual>
     <collision>
@@ -96,7 +86,5 @@
         <mesh filename="file://$(find trainer)/meshes/collision/cabinet_door_4.stl"/>
       </geometry>
-      <material name="red">
-        <color rgba="1.0 0 0 0.75"/>
-      </material>
+      <material name="red"/>
     </collision>
   </link>
@@ -120,7 +108,5 @@
         <mesh filename="file://$(find trainer)/meshes/visual/drawer_1_face.stl"/>
       </geometry>
-      <material name="blue">
-        <color rgba="0 0 1.0 0.75"/>
-      </material>
+      <material name="blue"/>
     </visual>
     <collision>
@@ -129,7 +115,5 @@
         <mesh filename="file://$(find trainer)/meshes/collision/drawer_1_face.stl"/>
       </geometry>
-      <material name="red">
-        <color rgba="1.0 0 0 0.75"/>
-      </material>
+      <material name="red"/>
     </collision>
   </link>
@@ -151,16 +135,12 @@
         <box size="0.013 0.305 0.096"/>
       </geometry>
-      <material name="blue">
-        <color rgba="0 0 1.0 0.75"/>
-      </material>
-    </visual>
-    <collision>
-      <origin xyz="${0.013/2} ${0.305/2} ${0.096/2}" rpy="0 0 0"/>
-      <geometry>
-        <box size="0.013 0.305 0.096"/>
-      </geometry>
-      <material name="red">
-        <color rgba="1.0 0 0 0.75"/>
-      </material>
+      <material name="blue"/>
+    </visual>
+    <collision>
+      <origin xyz="${0.013/2} ${0.305/2} ${0.096/2}" rpy="0 0 0"/>
+      <geometry>
+        <box size="0.013 0.305 0.096"/>
+      </geometry>
+      <material name="red"/>
     </collision>
   </link>
@@ -182,16 +162,12 @@
         <box size="0.013 0.305 0.096"/>
       </geometry>
-      <material name="blue">
-        <color rgba="0 0 1.0 0.75"/>
-      </material>
-    </visual>
-    <collision>
-      <origin xyz="${0.013/2} ${0.305/2} ${0.096/2}" rpy="0 0 0"/>
-      <geometry>
-        <box size="0.013 0.305 0.096"/>
-      </geometry>
-      <material name="red">
-        <color rgba="1.0 0 0 0.75"/>
-      </material>
+      <material name="blue"/>
+    </visual>
+    <collision>
+      <origin xyz="${0.013/2} ${0.305/2} ${0.096/2}" rpy="0 0 0"/>
+      <geometry>
+        <box size="0.013 0.305 0.096"/>
+      </geometry>
+      <material name="red"/>
     </collision>
   </link>
@@ -213,7 +189,5 @@
         <box size="0.293 0.305 0.013"/>
       </geometry>
-      <material name="blue">
-        <color rgba="0 0 1.0 0.75"/>
-      </material>
+      <material name="blue"/>
     </visual>
     <collision>
@@ -222,7 +196,5 @@
         <box size="0.293 0.305 0.013"/>
       </geometry>
-      <material name="red">
-        <color rgba="1.0 0 0 0.75"/>
-      </material>
+      <material name="red"/>
     </collision>
   </link>
@@ -246,7 +218,5 @@
         <mesh filename="file://$(find trainer)/meshes/visual/drawer_2_face.stl"/>
       </geometry>
-      <material name="blue">
-        <color rgba="0 0 1.0 0.75"/>
-      </material>
+      <material name="blue"/>
     </visual>
     <collision>
@@ -255,7 +225,5 @@
         <mesh filename="file://$(find trainer)/meshes/collision/drawer_2_face.stl"/>
       </geometry>
-      <material name="red">
-        <color rgba="1.0 0 0 0.75"/>
-      </material>
+      <material name="red"/>
     </collision>
   </link>
@@ -277,16 +245,12 @@
         <box size="0.013 0.305 0.096"/>
       </geometry>
-      <material name="blue">
-        <color rgba="0 0 1.0 0.75"/>
-      </material>
-    </visual>
-    <collision>
-      <origin xyz="${0.013/2} ${0.305/2} ${0.096/2}" rpy="0 0 0"/>
-      <geometry>
-        <box size="0.013 0.305 0.096"/>
-      </geometry>
-      <material name="red">
-        <color rgba="1.0 0 0 0.75"/>
-      </material>
+      <material name="blue"/>
+    </visual>
+    <collision>
+      <origin xyz="${0.013/2} ${0.305/2} ${0.096/2}" rpy="0 0 0"/>
+      <geometry>
+        <box size="0.013 0.305 0.096"/>
+      </geometry>
+      <material name="red"/>
     </collision>
   </link>
@@ -308,16 +272,12 @@
         <box size="0.013 0.305 0.096"/>
       </geometry>
-      <material name="blue">
-        <color rgba="0 0 1.0 0.75"/>
-      </material>
-    </visual>
-    <collision>
-      <origin xyz="${0.013/2} ${0.305/2} ${0.096/2}" rpy="0 0 0"/>
-      <geometry>
-        <box size="0.013 0.305 0.096"/>
-      </geometry>
-      <material name="red">
-        <color rgba="1.0 0 0 0.75"/>
-      </material>
+      <material name="blue"/>
+    </visual>
+    <collision>
+      <origin xyz="${0.013/2} ${0.305/2} ${0.096/2}" rpy="0 0 0"/>
+      <geometry>
+        <box size="0.013 0.305 0.096"/>
+      </geometry>
+      <material name="red"/>
     </collision>
   </link>
@@ -339,7 +299,5 @@
         <box size="0.293 0.305 0.013"/>
       </geometry>
-      <material name="blue">
-        <color rgba="0 0 1.0 0.75"/>
-      </material>
+      <material name="blue"/>
     </visual>
     <collision>
@@ -348,7 +306,5 @@
         <box size="0.293 0.305 0.013"/>
       </geometry>
-      <material name="red">
-        <color rgba="1.0 0 0 0.75"/>
-      </material>
+      <material name="red"/>
     </collision>
   </link>
