Commit message: Switching to a common colors file.

File: trainer/urdf/bench_seat.urdf.xacro (robot description, xacro)
@@ -3,17 +3,6 @@
   <xacro:arg name="name" default=""/>
   <xacro:arg name="prefix" default=""/>
+  <xacro:include filename="$(find trainer)/urdf/colors.xacro"/>
   <xacro:include filename="$(find trainer)/urdf/bench_seat.xacro"/>
-  <material name="red">
-    <color rgba="1.0 0 0 1"/>
-  </material>
-  <material name="green">
-    <color rgba="1.0 0 0 1"/>
-  </material>
-  <material name="blue">
-    <color rgba="0 0 1.0 1"/>
-  </material>
-  <material name="gray">
-    <color rgba="0.85 0.85 0.85 0.75"/>
-  </material>
   <link name="world"/>
   <xacro:bench_seat name="$(arg name)" prefix="$(arg prefix)" parent="world">

File: trainer/urdf/trainer.urdf.xacro (robot description, xacro)
@@ -5,16 +5,5 @@
   <xacro:property name="shelf" default="false"/>
   <xacro:property name="ceiling_prop" value="true"/>
-  <material name="red">
-    <color rgba="1.0 0 0 1"/>
-  </material>
-  <material name="green">
-    <color rgba="1.0 0 0 1"/>
-  </material>
-  <material name="blue">
-    <color rgba="0 0 1.0 1"/>
-  </material>
-  <material name="gray">
-    <color rgba="0.85 0.85 0.85 0.75"/>
-  </material>
+  <xacro:include filename="$(find trainer)/urdf/colors.xacro"/>
   <link name="world"/>
   <xacro:include filename="$(find trainer)/urdf/trainer_frame.xacro"/>

File: trainer/urdf/trainer_frame.urdf.xacro (robot description, xacro)
@@ -3,17 +3,6 @@
   <xacro:arg name="name" default=""/>
   <xacro:arg name="prefix" default=""/>
+  <xacro:include filename="$(find trainer)/urdf/colors.xacro"/>
   <xacro:include filename="$(find trainer)/urdf/trainer_frame.xacro"/>
-  <material name="red">
-    <color rgba="1.0 0 0 1"/>
-  </material>
-  <material name="green">
-    <color rgba="1.0 0 0 1"/>
-  </material>
-  <material name="blue">
-    <color rgba="0 0 1.0 1"/>
-  </material>
-  <material name="gray">
-    <color rgba="0.85 0.85 0.85 0.75"/>
-  </material>
   <link name="world"/>
   <xacro:trainer_frame name="$(arg name)" prefix="$(arg prefix)" parent="world">

File: trainer/urdf/trainer_front_left_face.urdf.xacro (robot description, xacro)
@@ -4,16 +4,5 @@
   <xacro:arg name="prefix" default=""/>
   <xacro:property name="shelf" default="true"/>
-  <material name="red">
-    <color rgba="1.0 0 0 1"/>
-  </material>
-  <material name="green">
-    <color rgba="1.0 0 0 1"/>
-  </material>
-  <material name="blue">
-    <color rgba="0 0 1.0 1"/>
-  </material>
-  <material name="gray">
-    <color rgba="0.85 0.85 0.85 0.75"/>
-  </material>
+  <xacro:include filename="$(find trainer)/urdf/colors.xacro"/>
   <link name="world"/>
   <xacro:include filename="$(find trainer)/urdf/trainer_front_left_face.xacro"/>

File: trainer/urdf/trainer_front_right_face.urdf.xacro (robot description, xacro)
@@ -3,16 +3,5 @@
   <xacro:arg name="name" default=""/>
   <xacro:arg name="prefix" default=""/>
-  <material name="red">
-    <color rgba="1.0 0 0 1"/>
-  </material>
-  <material name="green">
-    <color rgba="1.0 0 0 1"/>
-  </material>
-  <material name="blue">
-    <color rgba="0 0 1.0 1"/>
-  </material>
-  <material name="gray">
-    <color rgba="0.85 0.85 0.85 0.75"/>
-  </material>
+  <xacro:include filename="$(find trainer)/urdf/colors.xacro"/>
   <link name="world"/>
   <xacro:include filename="$(find trainer)/urdf/trainer_front_right_face.xacro"/>

File: trainer/urdf/trainer_side.urdf.xacro (robot description, xacro)
@@ -3,17 +3,6 @@
   <xacro:arg name="name" default=""/>
   <xacro:arg name="prefix" default=""/>
+  <xacro:include filename="$(find trainer)/urdf/colors.xacro"/>
   <xacro:include filename="$(find trainer)/urdf/trainer_side.xacro"/>
-  <material name="red">
-    <color rgba="1.0 0 0 1"/>
-  </material>
-  <material name="green">
-    <color rgba="1.0 0 0 1"/>
-  </material>
-  <material name="blue">
-    <color rgba="0 0 1.0 1"/>
-  </material>
-  <material name="gray">
-    <color rgba="0.85 0.85 0.85 0.75"/>
-  </material>
   <link name="world"/>
   <xacro:side_face name="$(arg name)" prefix="$(arg prefix)" parent="world">
