Commit message: Adding updated stls.

File: trainer/urdf/trainer_front_left_face.xacro (robot description, xacro)
@@ -22,5 +22,5 @@
       <origin xyz="0.0 0.0 0.0" rpy="0 0 0"/>
       <geometry>
-        <mesh filename="file://$(find trainer)/meshes/visual/front_face_plate.stl"/>
+        <mesh filename="file://$(find trainer)/meshes/visual/front_left_face.stl"/>
       </geometry>
       <material name="red">
@@ -31,5 +31,5 @@
       <origin xyz="0.0 0.0 0.0" rpy="0 0 0"/>
       <geometry>
-        <mesh filename="file://$(find trainer)/meshes/collision/front_face_plate.stl"/>
+        <mesh filename="file://$(find trainer)/meshes/collision/front_left_face.stl"/>
       </geometry>
       <material name="red">

Commit message: Updating names.

File: trainer/urdf/trainer_front_left_face.xacro (robot description, xacro)
@@ -9,8 +9,8 @@
   <joint name="${prefix}trainer_front_face_base_joint" type="fixed">
     <parent link="${parent}"/>
-    <child link="${prefix}front_face_plate"/>
+    <child link="${prefix}front_left_face"/>
     <xacro:insert_block name="origin"/>
   </joint>
-  <link name="${prefix}front_face_plate">
+  <link name="${prefix}front_left_face">
     <!--TODO set proper inertia-->
     <inertial>
@@ -22,5 +22,5 @@
       <origin xyz="0.0 0.0 0.0" rpy="0 0 0"/>
       <geometry>
-        <mesh filename="file://$(find trainer)/meshes/visual/front_face_plate.stl"/>
+        <mesh filename="file://$(find trainer)/meshes/visual/front_left_face.stl"/>
       </geometry>
       <material name="red">
@@ -31,5 +31,5 @@
       <origin xyz="0.0 0.0 0.0" rpy="0 0 0"/>
       <geometry>
-        <mesh filename="file://$(find trainer)/meshes/collision/front_face_plate.stl"/>
+        <mesh filename="file://$(find trainer)/meshes/collision/front_left_face.stl"/>
       </geometry>
       <material name="red">
@@ -39,5 +39,5 @@
   </link>
   <joint name="${prefix}cubby_1_joint" type="fixed">
-    <parent link="${prefix}front_face_plate"/>
+    <parent link="${prefix}front_left_face"/>
     <child link="${prefix}cubby_1"/>
     <origin xyz="0.0 0.002 0.525" rpy="0 0 0"/>
@@ -70,5 +70,5 @@
   </link>
   <joint name="${prefix}cubby_2_joint" type="fixed">
-    <parent link="${prefix}front_face_plate"/>
+    <parent link="${prefix}front_left_face"/>
     <child link="${prefix}cubby_2"/>
     <origin xyz="0.0 0.002 0.875" rpy="0 0 0"/>
@@ -102,5 +102,5 @@
   <xacro:if value="${shelf}">
     <joint name="${prefix}trainer_cubby_shelf_joint" type="fixed">
-      <parent link="${prefix}front_face_plate"/>
+      <parent link="${prefix}front_left_face"/>
       <child link="${prefix}cubby_shelf"/>
       <origin xyz="-0.173 -0.04 0.031" rpy="0 0 0"/>

Commit message: Correction for MR.

File: trainer/urdf/trainer_front_left_face.xacro (robot description, xacro)
@@ -37,5 +37,5 @@
     <parent link="${prefix}front_left_face"/>
     <child link="${prefix}cubby_1"/>
-    <origin xyz="0.0 0.002 0.525" rpy="0 0 0"/>
+    <origin xyz="0.0 0.0 0.525" rpy="0 0 0"/>
   </joint>
   <link name="${prefix}cubby_1">

Commit message: Needed to fix the other cubby.

File: trainer/urdf/trainer_front_left_face.xacro (robot description, xacro)
@@ -64,5 +64,5 @@
     <parent link="${prefix}front_left_face"/>
     <child link="${prefix}cubby_2"/>
-    <origin xyz="0.0 0.002 0.875" rpy="0 0 0"/>
+    <origin xyz="0.0 0.0 0.875" rpy="0 0 0"/>
   </joint>
   <link name="${prefix}cubby_2">
