Commit message: Adding cabinet doors.

File: trainer/urdf/trainer_front_right_face.xacro (robot description, xacro)
@@ -37,4 +37,103 @@
     </collision>
   </link>
+  <joint name="${prefix}cabinet_1_joint" type="revolute">
+    <axis xyz="0 0 1"/>
+    <limit effort="10.0" lower="0.0" upper="3.14" velocity="0.5"/>
+    <parent link="${prefix}front_right_face"/>
+    <child link="${prefix}cabinet_1"/>
+    <origin xyz="0.006 0.342 0.713" rpy="0 0 0"/>
+  </joint>
+  <link name="${prefix}cabinet_1">
+    <!--TODO set proper inertia-->
+    <inertial>
+      <origin rpy="0 0 0" xyz="0.0 0.0 0.0"/>
+      <mass value="0.0"/>
+      <inertia ixx="0.0" ixy="0.0" ixz="0.0" iyy="0.0" iyz="0.0" izz="0.0"/>
+    </inertial>
+    <visual>
+      <origin xyz="0.0 0.0 0.0" rpy="0 0 0"/>
+      <geometry>
+        <mesh filename="file://$(find trainer)/meshes/visual/cabinet_door_1.stl"/>
+      </geometry>
+      <material name="blue">
+        <color rgba="0 0 1.0 0.75"/>
+      </material>
+    </visual>
+    <collision>
+      <origin xyz="0.0 0.0 0.0" rpy="0 0 0"/>
+      <geometry>
+        <mesh filename="file://$(find trainer)/meshes/collision/cabinet_door_1.stl"/>
+      </geometry>
+      <material name="blue">
+        <color rgba="0 0 1.0 0.75"/>
+      </material>
+    </collision>
+  </link>
+  <joint name="${prefix}cabinet_2_joint" type="revolute">
+    <axis xyz="0 0 -1"/>
+    <limit effort="10.0" lower="0.0" upper="3.14" velocity="0.5"/>
+    <parent link="${prefix}front_right_face"/>
+    <child link="${prefix}cabinet_2"/>
+    <origin xyz="0.006 0.004 0.379" rpy="0 0 0"/>
+  </joint>
+  <link name="${prefix}cabinet_2">
+    <!--TODO set proper inertia-->
+    <inertial>
+      <origin rpy="0 0 0" xyz="0.0 0.0 0.0"/>
+      <mass value="0.0"/>
+      <inertia ixx="0.0" ixy="0.0" ixz="0.0" iyy="0.0" iyz="0.0" izz="0.0"/>
+    </inertial>
+    <visual>
+      <origin xyz="0.0 0.0 0.0" rpy="0 0 0"/>
+      <geometry>
+        <mesh filename="file://$(find trainer)/meshes/visual/cabinet_door_2.stl"/>
+      </geometry>
+      <material name="blue">
+        <color rgba="0 0 1.0 0.75"/>
+      </material>
+    </visual>
+    <collision>
+      <origin xyz="0.0 0.0 0.0" rpy="0 0 0"/>
+      <geometry>
+        <mesh filename="file://$(find trainer)/meshes/collision/cabinet_door_2.stl"/>
+      </geometry>
+      <material name="blue">
+        <color rgba="0 0 1.0 0.75"/>
+      </material>
+    </collision>
+  </link>
+  <joint name="${prefix}cabinet_3_joint" type="revolute">
+    <axis xyz="0 0 1"/>
+    <limit effort="10.0" lower="0.0" upper="3.14" velocity="0.5"/>
+    <parent link="${prefix}front_right_face"/>
+    <child link="${prefix}cabinet_3"/>
+    <origin xyz="0.006 0.342 0.007" rpy="0 0 0"/>
+  </joint>
+  <link name="${prefix}cabinet_3">
+    <!--TODO set proper inertia-->
+    <inertial>
+      <origin rpy="0 0 0" xyz="0.0 0.0 0.0"/>
+      <mass value="0.0"/>
+      <inertia ixx="0.0" ixy="0.0" ixz="0.0" iyy="0.0" iyz="0.0" izz="0.0"/>
+    </inertial>
+    <visual>
+      <origin xyz="0.0 0.0 0.0" rpy="0 0 0"/>
+      <geometry>
+        <mesh filename="file://$(find trainer)/meshes/visual/cabinet_door_3.stl"/>
+      </geometry>
+      <material name="blue">
+        <color rgba="0 0 1.0 0.75"/>
+      </material>
+    </visual>
+    <collision>
+      <origin xyz="0.0 0.0 0.0" rpy="0 0 0"/>
+      <geometry>
+        <mesh filename="file://$(find trainer)/meshes/collision/cabinet_door_3.stl"/>
+      </geometry>
+      <material name="blue">
+        <color rgba="0 0 1.0 0.75"/>
+      </material>
+    </collision>
+  </link>
   </xacro:macro>
 </robot>

Commit message: Fixing the front hatches.

File: trainer/urdf/trainer_front_right_face.xacro (robot description, xacro)
@@ -38,5 +38,5 @@
     <parent link="${prefix}front_right_face"/>
     <child link="${prefix}cabinet_1"/>
-    <origin xyz="0.006 0.342 0.713" rpy="0 0 0"/>
+    <origin xyz="0.017 0.344 0.713" rpy="0 0 0"/>
   </joint>
   <link name="${prefix}cabinet_1">
@@ -48,5 +48,5 @@
     </inertial>
     <visual>
-      <origin xyz="0.0 0.0 0.0" rpy="0 0 0"/>
+      <origin xyz="-0.0075 -0.00186 0.0" rpy="0 0 0"/>
       <geometry>
         <mesh filename="file://$(find trainer)/meshes/visual/cabinet_door_1.stl"/>
@@ -55,5 +55,5 @@
     </visual>
     <collision>
-      <origin xyz="0.0 0.0 0.0" rpy="0 0 0"/>
+      <origin xyz="-0.0075 -0.00186 0.0" rpy="0 0 0"/>
       <geometry>
         <mesh filename="file://$(find trainer)/meshes/collision/cabinet_door_1.stl"/>
@@ -67,5 +67,5 @@
     <parent link="${prefix}front_right_face"/>
     <child link="${prefix}cabinet_2"/>
-    <origin xyz="0.006 0.004 0.379" rpy="0 0 0"/>
+    <origin xyz="0.017 0.002 0.379" rpy="0 0 0"/>
   </joint>
   <link name="${prefix}cabinet_2">
@@ -77,5 +77,5 @@
     </inertial>
     <visual>
-      <origin xyz="0.0 0.0 0.0" rpy="0 0 0"/>
+      <origin xyz="-0.0075 -0.00186 0.0" rpy="0 0 0"/>
       <geometry>
         <mesh filename="file://$(find trainer)/meshes/visual/cabinet_door_2.stl"/>
@@ -84,5 +84,5 @@
     </visual>
     <collision>
-      <origin xyz="0.0 0.0 0.0" rpy="0 0 0"/>
+      <origin xyz="-0.0075 -0.00186 0.0" rpy="0 0 0"/>
       <geometry>
         <mesh filename="file://$(find trainer)/meshes/collision/cabinet_door_2.stl"/>
@@ -96,5 +96,5 @@
     <parent link="${prefix}front_right_face"/>
     <child link="${prefix}cabinet_3"/>
-    <origin xyz="0.006 0.342 0.007" rpy="0 0 0"/>
+    <origin xyz="0.017 0.342 0.007" rpy="0 0 0"/>
   </joint>
   <link name="${prefix}cabinet_3">
@@ -106,5 +106,5 @@
     </inertial>
     <visual>
-      <origin xyz="0.0 0.0 0.0" rpy="0 0 0"/>
+      <origin xyz="-0.0075 -0.00186 0.0" rpy="0 0 0"/>
       <geometry>
         <mesh filename="file://$(find trainer)/meshes/visual/cabinet_door_3.stl"/>
@@ -113,5 +113,5 @@
     </visual>
     <collision>
-      <origin xyz="0.0 0.0 0.0" rpy="0 0 0"/>
+      <origin xyz="-0.0075 -0.00186 0.0" rpy="0 0 0"/>
       <geometry>
         <mesh filename="file://$(find trainer)/meshes/collision/cabinet_door_3.stl"/>

Commit message: Adding the round latch.

File: trainer/urdf/trainer_front_right_face.xacro (robot description, xacro)
@@ -58,4 +58,60 @@
       <geometry>
         <mesh filename="file://$(find trainer)/meshes/collision/cabinet_door_1.stl"/>
+      </geometry>
+      <material name="red"/>
+    </collision>
+  </link>
+  <joint name="${prefix}round_latch_face_joint" type="fixed">
+    <parent link="${prefix}cabinet_1"/>
+    <child link="${prefix}round_latch_face"/>
+    <origin xyz="0.0032 -0.286 0.167" rpy="${pi} 0 0"/>
+  </joint>
+  <link name="${prefix}round_latch_face">
+    <!--TODO set proper inertia-->
+    <inertial>
+      <origin rpy="0 0 0" xyz="0.0 0.0 0.0"/>
+      <mass value="0.0"/>
+      <inertia ixx="0.0" ixy="0.0" ixz="0.0" iyy="0.0" iyz="0.0" izz="0.0"/>
+    </inertial>
+    <visual>
+      <origin xyz="0.0 0.0 0.0" rpy="0 0 0"/>
+      <geometry>
+        <mesh filename="file://$(find trainer)/meshes/visual/round_latch_face.stl"/>
+      </geometry>
+      <material name="blue"/>
+    </visual>
+    <collision>
+      <origin xyz="0.0 0.0 0.0" rpy="0 0 0"/>
+      <geometry>
+        <mesh filename="file://$(find trainer)/meshes/collision/round_latch_face.stl"/>
+      </geometry>
+      <material name="red"/>
+    </collision>
+  </link>
+  <joint name="${prefix}round_latch_joint" type="revolute">
+    <axis xyz="0 0 -1"/>
+    <limit effort="10.0" lower="0.0" upper="3.14" velocity="0.5"/>
+    <parent link="${prefix}round_latch_face"/>
+    <child link="${prefix}round_latch"/>
+    <origin xyz="0.0 -0.0212 -0.0035" rpy="0 0 0"/>
+  </joint>
+  <link name="${prefix}round_latch">
+    <!--TODO set proper inertia-->
+    <inertial>
+      <origin rpy="0 0 0" xyz="0.0 0.0 0.0"/>
+      <mass value="0.0"/>
+      <inertia ixx="0.0" ixy="0.0" ixz="0.0" iyy="0.0" iyz="0.0" izz="0.0"/>
+    </inertial>
+    <visual>
+      <origin xyz="0.0 0.0 0.0" rpy="0 0 0"/>
+      <geometry>
+        <mesh filename="file://$(find trainer)/meshes/visual/round_latch.stl"/>
+      </geometry>
+      <material name="blue"/>
+    </visual>
+    <collision>
+      <origin xyz="0.0 0.0 0.0" rpy="0 0 0"/>
+      <geometry>
+        <mesh filename="file://$(find trainer)/meshes/collision/round_latch.stl"/>
       </geometry>
       <material name="red"/>

Commit message: MR updates.

File: trainer/urdf/trainer_front_right_face.xacro (robot description, xacro)
@@ -77,5 +77,5 @@
     </inertial>
     <visual>
-      <origin xyz="-0.0075 -0.00186 0.0" rpy="0 0 0"/>
+      <origin xyz="-0.0075 0.00186 0.0" rpy="0 0 0"/>
       <geometry>
         <mesh filename="file://$(find trainer)/meshes/visual/cabinet_door_2.stl"/>
@@ -84,5 +84,5 @@
     </visual>
     <collision>
-      <origin xyz="-0.0075 -0.00186 0.0" rpy="0 0 0"/>
+      <origin xyz="-0.0075 0.00186 0.0" rpy="0 0 0"/>
       <geometry>
         <mesh filename="file://$(find trainer)/meshes/collision/cabinet_door_2.stl"/>

Commit message: MR updates.

File: trainer/urdf/trainer_front_right_face.xacro (robot description, xacro)
@@ -96,5 +96,5 @@
     <parent link="${prefix}front_right_face"/>
     <child link="${prefix}cabinet_3"/>
-    <origin xyz="0.017 0.342 0.007" rpy="0 0 0"/>
+    <origin xyz="0.017 0.344 0.007" rpy="0 0 0"/>
   </joint>
   <link name="${prefix}cabinet_3">

Commit message: updating hinge details to account for various offsets

File: trainer/urdf/trainer_front_right_face.xacro (robot description, xacro)
@@ -38,5 +38,5 @@
     <parent link="${prefix}front_right_face"/>
     <child link="${prefix}cabinet_1"/>
-    <origin xyz="0.017 0.344 0.713" rpy="0 0 0"/>
+    <origin xyz="0.017 ${0.344 + 0.0018} 0.713" rpy="0 0 0"/>
   </joint>
   <link name="${prefix}cabinet_1">
@@ -48,5 +48,5 @@
     </inertial>
     <visual>
-      <origin xyz="-0.0075 -0.00186 0.0" rpy="0 0 0"/>
+      <origin xyz="${-0.0075 - 0.003175} -0.00366 0.0" rpy="0 0 0"/>
       <geometry>
         <mesh filename="file://$(find trainer)/meshes/visual/cabinet_door_1.stl"/>
@@ -55,5 +55,5 @@
     </visual>
     <collision>
-      <origin xyz="-0.0075 -0.00186 0.0" rpy="0 0 0"/>
+      <origin xyz="${-0.0075 - 0.003175} -0.00366 0.0" rpy="0 0 0"/>
       <geometry>
         <mesh filename="file://$(find trainer)/meshes/collision/cabinet_door_1.stl"/>
@@ -67,5 +67,5 @@
     <parent link="${prefix}front_right_face"/>
     <child link="${prefix}cabinet_2"/>
-    <origin xyz="0.017 0.002 0.379" rpy="0 0 0"/>
+    <origin xyz="0.017 -0.0018 0.379" rpy="0 0 0"/>
   </joint>
   <link name="${prefix}cabinet_2">
@@ -77,5 +77,5 @@
     </inertial>
     <visual>
-      <origin xyz="-0.0075 0.00186 0.0" rpy="0 0 0"/>
+      <origin xyz="${-0.0075 - 0.003175} 0.00366 0.0" rpy="0 0 0"/>
       <geometry>
         <mesh filename="file://$(find trainer)/meshes/visual/cabinet_door_2.stl"/>
@@ -84,5 +84,5 @@
     </visual>
     <collision>
-      <origin xyz="-0.0075 0.00186 0.0" rpy="0 0 0"/>
+      <origin xyz="${-0.0075 - 0.003175} 0.00366 0.0" rpy="0 0 0"/>
       <geometry>
         <mesh filename="file://$(find trainer)/meshes/collision/cabinet_door_2.stl"/>
@@ -96,5 +96,5 @@
     <parent link="${prefix}front_right_face"/>
     <child link="${prefix}cabinet_3"/>
-    <origin xyz="0.017 0.344 0.007" rpy="0 0 0"/>
+    <origin xyz="0.017 ${0.344 + 0.0018} 0.007" rpy="0 0 0"/>
   </joint>
   <link name="${prefix}cabinet_3">
@@ -106,5 +106,5 @@
     </inertial>
     <visual>
-      <origin xyz="-0.0075 -0.00186 0.0" rpy="0 0 0"/>
+      <origin xyz="${-0.0075 - 0.003175} -0.00366 0.0" rpy="0 0 0"/>
       <geometry>
         <mesh filename="file://$(find trainer)/meshes/visual/cabinet_door_3.stl"/>
@@ -113,5 +113,5 @@
     </visual>
     <collision>
-      <origin xyz="-0.0075 -0.00186 0.0" rpy="0 0 0"/>
+      <origin xyz="${-0.0075 - 0.003175} -0.00366 0.0" rpy="0 0 0"/>
       <geometry>
         <mesh filename="file://$(find trainer)/meshes/collision/cabinet_door_3.stl"/>

Commit message: Renaming the round and adding the push latch housing.

File: trainer/urdf/trainer_front_right_face.xacro (robot description, xacro)
@@ -62,27 +62,27 @@
     </collision>
   </link>
-  <joint name="${prefix}round_latch_face_joint" type="fixed">
+  <joint name="${prefix}round_latch_housing_joint" type="fixed">
     <parent link="${prefix}cabinet_1"/>
-    <child link="${prefix}round_latch_face"/>
+    <child link="${prefix}round_latch_housing"/>
     <origin xyz="0.0032 -0.286 0.167" rpy="${pi} 0 0"/>
   </joint>
-  <link name="${prefix}round_latch_face">
-    <!--TODO set proper inertia-->
-    <inertial>
-      <origin rpy="0 0 0" xyz="0.0 0.0 0.0"/>
-      <mass value="0.0"/>
-      <inertia ixx="0.0" ixy="0.0" ixz="0.0" iyy="0.0" iyz="0.0" izz="0.0"/>
-    </inertial>
-    <visual>
-      <origin xyz="0.0 0.0 0.0" rpy="0 0 0"/>
-      <geometry>
-        <mesh filename="file://$(find trainer)/meshes/visual/round_latch_face.stl"/>
-      </geometry>
-      <material name="blue"/>
-    </visual>
-    <collision>
-      <origin xyz="0.0 0.0 0.0" rpy="0 0 0"/>
-      <geometry>
-        <mesh filename="file://$(find trainer)/meshes/collision/round_latch_face.stl"/>
+  <link name="${prefix}round_latch_housing">
+    <!--TODO set proper inertia-->
+    <inertial>
+      <origin rpy="0 0 0" xyz="0.0 0.0 0.0"/>
+      <mass value="0.0"/>
+      <inertia ixx="0.0" ixy="0.0" ixz="0.0" iyy="0.0" iyz="0.0" izz="0.0"/>
+    </inertial>
+    <visual>
+      <origin xyz="0.0 0.0 0.0" rpy="0 0 0"/>
+      <geometry>
+        <mesh filename="file://$(find trainer)/meshes/visual/round_latch_housing.stl"/>
+      </geometry>
+      <material name="gray"/>
+    </visual>
+    <collision>
+      <origin xyz="0.0 0.0 0.0" rpy="0 0 0"/>
+      <geometry>
+        <mesh filename="file://$(find trainer)/meshes/collision/round_latch_housing.stl"/>
       </geometry>
       <material name="red"/>
@@ -92,26 +92,26 @@
     <axis xyz="0 0 -1"/>
     <limit effort="10.0" lower="0.0" upper="3.14" velocity="0.5"/>
-    <parent link="${prefix}round_latch_face"/>
-    <child link="${prefix}round_latch"/>
+    <parent link="${prefix}round_latch_housing"/>
+    <child link="${prefix}round_latch_handle"/>
     <origin xyz="0.0 -0.0212 -0.0035" rpy="0 0 0"/>
   </joint>
-  <link name="${prefix}round_latch">
-    <!--TODO set proper inertia-->
-    <inertial>
-      <origin rpy="0 0 0" xyz="0.0 0.0 0.0"/>
-      <mass value="0.0"/>
-      <inertia ixx="0.0" ixy="0.0" ixz="0.0" iyy="0.0" iyz="0.0" izz="0.0"/>
-    </inertial>
-    <visual>
-      <origin xyz="0.0 0.0 0.0" rpy="0 0 0"/>
-      <geometry>
-        <mesh filename="file://$(find trainer)/meshes/visual/round_latch.stl"/>
-      </geometry>
-      <material name="blue"/>
-    </visual>
-    <collision>
-      <origin xyz="0.0 0.0 0.0" rpy="0 0 0"/>
-      <geometry>
-        <mesh filename="file://$(find trainer)/meshes/collision/round_latch.stl"/>
+  <link name="${prefix}round_latch_handle">
+    <!--TODO set proper inertia-->
+    <inertial>
+      <origin rpy="0 0 0" xyz="0.0 0.0 0.0"/>
+      <mass value="0.0"/>
+      <inertia ixx="0.0" ixy="0.0" ixz="0.0" iyy="0.0" iyz="0.0" izz="0.0"/>
+    </inertial>
+    <visual>
+      <origin xyz="0.0 0.0 0.0" rpy="0 0 0"/>
+      <geometry>
+        <mesh filename="file://$(find trainer)/meshes/visual/round_latch_handle.stl"/>
+      </geometry>
+      <material name="blue"/>
+    </visual>
+    <collision>
+      <origin xyz="0.0 0.0 0.0" rpy="0 0 0"/>
+      <geometry>
+        <mesh filename="file://$(find trainer)/meshes/collision/round_latch_handle.stl"/>
       </geometry>
       <material name="red"/>
@@ -147,4 +147,31 @@
     </collision>
   </link>
+  <joint name="${prefix}push_latch_housing_joint" type="fixed">
+    <parent link="${prefix}cabinet_2"/>
+    <child link="${prefix}push_latch_housing"/>
+    <origin xyz="0.0032 0.2185 0.134" rpy="0 0 0"/>
+  </joint>
+  <link name="${prefix}push_latch_housing">
+    <!--TODO set proper inertia-->
+    <inertial>
+      <origin rpy="0 0 0" xyz="0.0 0.0 0.0"/>
+      <mass value="0.0"/>
+      <inertia ixx="0.0" ixy="0.0" ixz="0.0" iyy="0.0" iyz="0.0" izz="0.0"/>
+    </inertial>
+    <visual>
+      <origin xyz="0.0 0.0 0.0" rpy="0 0 0"/>
+      <geometry>
+        <mesh filename="file://$(find trainer)/meshes/visual/push_latch_housing.stl"/>
+      </geometry>
+      <material name="gray"/>
+    </visual>
+    <collision>
+      <origin xyz="0.0 0.0 0.0" rpy="0 0 0"/>
+      <geometry>
+        <mesh filename="file://$(find trainer)/meshes/collision/push_latch_housing.stl"/>
+      </geometry>
+      <material name="red"/>
+    </collision>
+  </link>
   <joint name="${prefix}cabinet_3_joint" type="revolute">
     <axis xyz="0 0 1"/>

Commit message: Adding the rest of the push latch and fixing the recessed joint.

File: trainer/urdf/trainer_front_right_face.xacro (robot description, xacro)
@@ -150,5 +150,5 @@
     <parent link="${prefix}cabinet_2"/>
     <child link="${prefix}push_latch_housing"/>
-    <origin xyz="0.0032 0.2185 0.134" rpy="0 0 0"/>
+    <origin xyz="-0.0075 0.2185 0.134" rpy="0 0 0"/>
   </joint>
   <link name="${prefix}push_latch_housing">
@@ -170,4 +170,63 @@
       <geometry>
         <mesh filename="file://$(find trainer)/meshes/collision/push_latch_housing.stl"/>
+      </geometry>
+      <material name="red"/>
+    </collision>
+  </link>
+  <joint name="${prefix}push_latch_button_joint" type="prismatic">
+    <axis xyz="-1 0 0"/>
+    <!--TODO button travel is a complete guess at this point-->
+    <limit effort="10.0" lower="0.0" upper="0.005" velocity="0.5"/>
+    <parent link="${prefix}push_latch_housing"/>
+    <child link="${prefix}push_latch_button"/>
+    <origin xyz="-0.0125 0.0285 0.0045" rpy="0 0 ${pi/8}"/>
+  </joint>
+  <link name="${prefix}push_latch_button">
+    <!--TODO set proper inertia-->
+    <inertial>
+      <origin rpy="0 0 0" xyz="0.0 0.0 0.0"/>
+      <mass value="0.0"/>
+      <inertia ixx="0.0" ixy="0.0" ixz="0.0" iyy="0.0" iyz="0.0" izz="0.0"/>
+    </inertial>
+    <visual>
+      <origin xyz="0.0 0.0 0.0" rpy="0 0 0"/>
+      <geometry>
+        <mesh filename="file://$(find trainer)/meshes/visual/push_latch_button.stl"/>
+      </geometry>
+      <material name="blue"/>
+    </visual>
+    <collision>
+      <origin xyz="0.0 0.0 0.0" rpy="0 0 0"/>
+      <geometry>
+        <mesh filename="file://$(find trainer)/meshes/collision/push_latch_button.stl"/>
+      </geometry>
+      <material name="red"/>
+    </collision>
+  </link>
+  <joint name="${prefix}push_latch_handle_joint" type="revolute">
+    <axis xyz="0 0 1"/>
+    <limit effort="10.0" lower="0.0" upper="${pi/3}" velocity="0.5"/>
+    <parent link="${prefix}push_latch_housing"/>
+    <child link="${prefix}push_latch_handle"/>
+    <origin xyz="-0.003 0.079 0.0045" rpy="0 0 0"/>
+  </joint>
+  <link name="${prefix}push_latch_handle">
+    <!--TODO set proper inertia-->
+    <inertial>
+      <origin rpy="0 0 0" xyz="0.0 0.0 0.0"/>
+      <mass value="0.0"/>
+      <inertia ixx="0.0" ixy="0.0" ixz="0.0" iyy="0.0" iyz="0.0" izz="0.0"/>
+    </inertial>
+    <visual>
+      <origin xyz="0.0 0.0 0.0" rpy="0 0 0"/>
+      <geometry>
+        <mesh filename="file://$(find trainer)/meshes/visual/push_latch_handle.stl"/>
+      </geometry>
+      <material name="blue"/>
+    </visual>
+    <collision>
+      <origin xyz="0.0 0.0 0.0" rpy="0 0 0"/>
+      <geometry>
+        <mesh filename="file://$(find trainer)/meshes/collision/push_latch_handle.stl"/>
       </geometry>
       <material name="red"/>
@@ -176,5 +235,5 @@
   <joint name="${prefix}cabinet_3_joint" type="revolute">
     <axis xyz="0 0 1"/>
-    <limit effort="10.0" lower="0.0" upper="3.14" velocity="0.5"/>
+    <limit effort="10.0" lower="0.0" upper="${pi}" velocity="0.5"/>
     <parent link="${prefix}front_right_face"/>
     <child link="${prefix}cabinet_3"/>

File: trainer/urdf/trainer_side.xacro (robot description, xacro)
@@ -311,7 +311,7 @@
     </collision>
   </link>
-  <joint name="${prefix}recessed_latch_handle_joint" type="prismatic">
+  <joint name="${prefix}recessed_latch_handle_joint" type="revolute">
     <axis xyz="-1 0 0"/>
-    <limit effort="10.0" lower="0.0" upper="0.2921" velocity="0.5"/>
+    <limit effort="10.0" lower="0.0" upper="${pi/2}" velocity="0.5"/>
     <parent link="${prefix}recessed_latch_housing"/>
     <child link="${prefix}recessed_latch_handle"/>

Commit message: adjusting origin of round_latch_housing_joint

File: trainer/urdf/trainer_front_right_face.xacro (robot description, xacro)
@@ -65,5 +65,5 @@
     <parent link="${prefix}cabinet_1"/>
     <child link="${prefix}round_latch_housing"/>
-    <origin xyz="0.0032 -0.286 0.167" rpy="${pi} 0 0"/>
+    <origin xyz="-0.00547 -0.28855 0.16622" rpy="${pi} 0 0"/>
   </joint>
   <link name="${prefix}round_latch_housing">
