Commit message: Updating the side faces.

File: trainer/urdf/trainer_side.xacro (robot description, xacro)
@@ -8,12 +8,12 @@
     <joint name="${prefix}trainer_side_face_base_joint" type="fixed">
       <parent link="${parent}"/>
-      <child link="${prefix}side_face_lower"/>
+      <child link="${prefix}side_bottom_face"/>
       <xacro:insert_block name="origin"/>
     </joint>
-    <link name="${prefix}side_face_lower">
+    <link name="${prefix}side_bottom_face">
       <visual>
         <origin xyz="0.0 0.0 0.0" rpy="0 0 0"/>
           <geometry>
-            <mesh filename="file://$(find trainer)/meshes/visual/side_face_lower.stl"/>
+            <mesh filename="file://$(find trainer)/meshes/visual/side_bottom_face.stl"/>
           </geometry>
         <material name="red">
@@ -24,5 +24,5 @@
         <origin xyz="0.0 0.0 0.0" rpy="0 0 0"/>
           <geometry>
-            <mesh filename="file://$(find trainer)/meshes/collision/side_face_lower.stl"/>
+            <mesh filename="file://$(find trainer)/meshes/collision/side_bottom_face.stl"/>
           </geometry>
         <material name="red">
@@ -31,14 +31,14 @@
       </collision>
     </link>
-    <joint name="${prefix}side_face_plate_joint" type="fixed">
-      <parent link="${prefix}side_face_lower"/>
-      <child link="${prefix}side_face_plate"/>
+    <joint name="${prefix}side_top_face_joint" type="fixed">
+      <parent link="${prefix}side_bottom_face"/>
+      <child link="${prefix}side_top_face"/>
       <origin xyz="0.0 0.0 0.5084191" rpy="0 0 0"/>
     </joint>
-    <link name="${prefix}side_face_plate">
+    <link name="${prefix}side_top_face">
       <visual>
         <origin xyz="0.0 0.0 0.0" rpy="0 0 0"/>
           <geometry>
-            <mesh filename="file://$(find trainer)/meshes/visual/side_face_plate.stl"/>
+            <mesh filename="file://$(find trainer)/meshes/visual/side_top_face.stl"/>
           </geometry>
         <material name="red">
@@ -49,5 +49,5 @@
         <origin xyz="0.0 0.0 0.0" rpy="0 0 0"/>
           <geometry>
-            <mesh filename="file://$(find trainer)/meshes/collision/side_face_plate.stl"/>
+            <mesh filename="file://$(find trainer)/meshes/collision/side_top_face.stl"/>
           </geometry>
         <material name="red">

Commit message: Adding the side cabinet.

File: trainer/urdf/trainer_side.xacro (robot description, xacro)
@@ -56,4 +56,37 @@
       </collision>
     </link>
+  <joint name="${prefix}cabinet_4_joint" type="revolute">
+    <axis xyz="0 0 1"/>
+    <limit effort="10.0" lower="0.0" upper="3.14" velocity="0.5"/>
+    <parent link="${prefix}side_top_face"/>
+    <child link="${prefix}cabinet_4"/>
+    <origin xyz="0.004 0.006 0.484" rpy="0 0 0"/>
+  </joint>
+  <link name="${prefix}cabinet_4">
+    <!--TODO set proper inertia-->
+    <inertial>
+      <origin rpy="0 0 0" xyz="0.0 0.0 0.0"/>
+      <mass value="0.0"/>
+      <inertia ixx="0.0" ixy="0.0" ixz="0.0" iyy="0.0" iyz="0.0" izz="0.0"/>
+    </inertial>
+    <visual>
+      <origin xyz="0.0 0.0 0.0" rpy="0 0 0"/>
+      <geometry>
+        <mesh filename="file://$(find trainer)/meshes/visual/cabinet_door_4.stl"/>
+      </geometry>
+      <material name="blue">
+        <color rgba="0 0 1.0 0.75"/>
+      </material>
+    </visual>
+    <collision>
+      <origin xyz="0.0 0.0 0.0" rpy="0 0 0"/>
+      <geometry>
+        <mesh filename="file://$(find trainer)/meshes/collision/cabinet_door_4.stl"/>
+      </geometry>
+      <material name="blue">
+        <color rgba="0 0 1.0 0.75"/>
+      </material>
+    </collision>
+  </link>
   </xacro:macro>
 </robot>

Commit message: Adding drawers.

File: trainer/urdf/trainer_side.xacro (robot description, xacro)
@@ -89,4 +89,220 @@
     </collision>
   </link>
+  <joint name="${prefix}drawer_1_joint" type="prismatic">
+    <axis xyz="0 1 0"/>
+    <limit effort="10.0" lower="0.0" upper="0.305" velocity="0.5"/>
+    <parent link="${prefix}side_top_face"/>
+    <child link="${prefix}drawer_1_face"/>
+    <origin xyz="0.004 0.006 0.282" rpy="0 0 0"/>
+  </joint>
+  <link name="${prefix}drawer_1_face">
+    <!--TODO set proper inertia-->
+    <inertial>
+      <origin rpy="0 0 0" xyz="0.0 0.0 0.0"/>
+      <mass value="0.0"/>
+      <inertia ixx="0.0" ixy="0.0" ixz="0.0" iyy="0.0" iyz="0.0" izz="0.0"/>
+    </inertial>
+    <visual>
+      <origin xyz="0.0 0.0 0.0" rpy="0 0 0"/>
+      <geometry>
+        <mesh filename="file://$(find trainer)/meshes/visual/drawer_1_face.stl"/>
+      </geometry>
+      <material name="blue">
+        <color rgba="0 0 1.0 0.75"/>
+      </material>
+    </visual>
+    <collision>
+      <origin xyz="0.0 0.0 0.0" rpy="0 0 0"/>
+      <geometry>
+        <mesh filename="file://$(find trainer)/meshes/collision/drawer_1_face.stl"/>
+      </geometry>
+      <material name="blue">
+        <color rgba="0 0 1.0 0.75"/>
+      </material>
+    </collision>
+  </link>
+  <joint name="${prefix}drawer_1_left_joint" type="fixed">
+    <parent link="${prefix}drawer_1_face"/>
+    <child link="${prefix}drawer_1_left"/>
+    <origin xyz="0.293 -0.305 -0.007" rpy="0 0 0"/>
+  </joint>
+  <link name="${prefix}drawer_1_left">
+    <visual>
+      <origin xyz="${0.013/2} ${0.305/2} ${0.096/2}" rpy="0 0 0"/>
+      <geometry>
+        <box size="0.013 0.305 0.096"/>
+      </geometry>
+      <material name="blue">
+        <color rgba="0 0 1.0 0.75"/>
+      </material>
+    </visual>
+    <collision>
+      <origin xyz="${0.013/2} ${0.305/2} ${0.096/2}" rpy="0 0 0"/>
+      <geometry>
+        <box size="0.013 0.305 0.096"/>
+      </geometry>
+      <material name="blue">
+        <color rgba="0 0 1.0 0.75"/>
+      </material>
+    </collision>
+  </link>
+  <joint name="${prefix}drawer_1_right_joint" type="fixed">
+    <parent link="${prefix}drawer_1_face"/>
+    <child link="${prefix}drawer_1_right"/>
+    <origin xyz="0.0 -0.305 -0.007" rpy="0 0 0"/>
+  </joint>
+  <link name="${prefix}drawer_1_right">
+    <visual>
+      <origin xyz="${0.013/2} ${0.305/2} ${0.096/2}" rpy="0 0 0"/>
+      <geometry>
+        <box size="0.013 0.305 0.096"/>
+      </geometry>
+      <material name="blue">
+        <color rgba="0 0 1.0 0.75"/>
+      </material>
+    </visual>
+    <collision>
+      <origin xyz="${0.013/2} ${0.305/2} ${0.096/2}" rpy="0 0 0"/>
+      <geometry>
+        <box size="0.013 0.305 0.096"/>
+      </geometry>
+      <material name="blue">
+        <color rgba="0 0 1.0 0.75"/>
+      </material>
+    </collision>
+  </link>
+  <joint name="${prefix}drawer_1_bottom_joint" type="fixed">
+    <parent link="${prefix}drawer_1_face"/>
+    <child link="${prefix}drawer_1_bottom"/>
+    <origin xyz="0.0 -0.305 -0.007" rpy="0 0 0"/>
+  </joint>
+  <link name="${prefix}drawer_1_bottom">
+    <visual>
+      <origin xyz="${0.293/2} ${0.305/2} ${0.013/2}" rpy="0 0 0"/>
+      <geometry>
+        <box size="0.293 0.305 0.013"/>
+      </geometry>
+      <material name="blue">
+        <color rgba="0 0 1.0 0.75"/>
+      </material>
+    </visual>
+    <collision>
+      <origin xyz="${0.293/2} ${0.305/2} ${0.013/2}" rpy="0 0 0"/>
+      <geometry>
+        <box size="0.293 0.305 0.013"/>
+      </geometry>
+      <material name="blue">
+        <color rgba="0 0 1.0 0.75"/>
+      </material>
+    </collision>
+  </link>
+  <joint name="${prefix}drawer_2_joint" type="prismatic">
+    <axis xyz="0 1 0"/>
+    <limit effort="10.0" lower="0.0" upper="0.2921" velocity="0.5"/>
+    <parent link="${prefix}side_top_face"/>
+    <child link="${prefix}drawer_2_face"/>
+    <origin xyz="0.004 0.006 0.085" rpy="0 0 0"/>
+  </joint>
+  <link name="${prefix}drawer_2_face">
+    <!--TODO set proper inertia-->
+    <inertial>
+      <origin rpy="0 0 0" xyz="0.0 0.0 0.0"/>
+      <mass value="0.0"/>
+      <inertia ixx="0.0" ixy="0.0" ixz="0.0" iyy="0.0" iyz="0.0" izz="0.0"/>
+    </inertial>
+    <visual>
+      <origin xyz="0.0 0.0 0.0" rpy="0 0 0"/>
+      <geometry>
+        <mesh filename="file://$(find trainer)/meshes/visual/drawer_2_face.stl"/>
+      </geometry>
+      <material name="blue">
+        <color rgba="0 0 1.0 0.75"/>
+      </material>
+    </visual>
+    <collision>
+      <origin xyz="0.0 0.0 0.0" rpy="0 0 0"/>
+      <geometry>
+        <mesh filename="file://$(find trainer)/meshes/collision/drawer_2_face.stl"/>
+      </geometry>
+      <material name="blue">
+        <color rgba="0 0 1.0 0.75"/>
+      </material>
+    </collision>
+  </link>
+  <joint name="${prefix}drawer_2_left_joint" type="fixed">
+    <parent link="${prefix}drawer_2_face"/>
+    <child link="${prefix}drawer_2_left"/>
+    <origin xyz="0.293 -0.305 -0.007" rpy="0 0 0"/>
+  </joint>
+  <link name="${prefix}drawer_2_left">
+    <visual>
+      <origin xyz="${0.013/2} ${0.305/2} ${0.096/2}" rpy="0 0 0"/>
+      <geometry>
+        <box size="0.013 0.305 0.096"/>
+      </geometry>
+      <material name="blue">
+        <color rgba="0 0 1.0 0.75"/>
+      </material>
+    </visual>
+    <collision>
+      <origin xyz="${0.013/2} ${0.305/2} ${0.096/2}" rpy="0 0 0"/>
+      <geometry>
+        <box size="0.013 0.305 0.096"/>
+      </geometry>
+      <material name="blue">
+        <color rgba="0 0 1.0 0.75"/>
+      </material>
+    </collision>
+  </link>
+  <joint name="${prefix}drawer_2_right_joint" type="fixed">
+    <parent link="${prefix}drawer_2_face"/>
+    <child link="${prefix}drawer_2_right"/>
+    <origin xyz="0.0 -0.305 -0.007" rpy="0 0 0"/>
+  </joint>
+  <link name="${prefix}drawer_2_right">
+    <visual>
+      <origin xyz="${0.013/2} ${0.305/2} ${0.096/2}" rpy="0 0 0"/>
+      <geometry>
+        <box size="0.013 0.305 0.096"/>
+      </geometry>
+      <material name="blue">
+        <color rgba="0 0 1.0 0.75"/>
+      </material>
+    </visual>
+    <collision>
+      <origin xyz="${0.013/2} ${0.305/2} ${0.096/2}" rpy="0 0 0"/>
+      <geometry>
+        <box size="0.013 0.305 0.096"/>
+      </geometry>
+      <material name="blue">
+        <color rgba="0 0 1.0 0.75"/>
+      </material>
+    </collision>
+  </link>
+  <joint name="${prefix}drawer_2_bottom_joint" type="fixed">
+    <parent link="${prefix}drawer_2_face"/>
+    <child link="${prefix}drawer_2_bottom"/>
+    <origin xyz="0.0 -0.305 -0.007" rpy="0 0 0"/>
+  </joint>
+  <link name="${prefix}drawer_2_bottom">
+    <visual>
+      <origin xyz="${0.293/2} ${0.305/2} ${0.013/2}" rpy="0 0 0"/>
+      <geometry>
+        <box size="0.293 0.305 0.013"/>
+      </geometry>
+      <material name="blue">
+        <color rgba="0 0 1.0 0.75"/>
+      </material>
+    </visual>
+    <collision>
+      <origin xyz="${0.293/2} ${0.305/2} ${0.013/2}" rpy="0 0 0"/>
+      <geometry>
+        <box size="0.293 0.305 0.013"/>
+      </geometry>
+      <material name="blue">
+        <color rgba="0 0 1.0 0.75"/>
+      </material>
+    </collision>
+  </link>
   </xacro:macro>
 </robot>

Commit message: Updating cabinet 4 hinge.

File: trainer/urdf/trainer_side.xacro (robot description, xacro)
@@ -65,5 +65,5 @@
     <parent link="${prefix}side_top_face"/>
     <child link="${prefix}cabinet_4"/>
-    <origin xyz="0.004 0.006 0.484" rpy="0 0 0"/>
+    <origin xyz="0.0 0.017 0.484" rpy="0 0 0"/>
   </joint>
   <link name="${prefix}cabinet_4">
@@ -75,5 +75,5 @@
     </inertial>
     <visual>
-      <origin xyz="0.0 0.0 0.0" rpy="0 0 0"/>
+      <origin xyz="0.0048 -0.0106 0.0" rpy="0 0 0"/>
       <geometry>
         <mesh filename="file://$(find trainer)/meshes/visual/cabinet_door_4.stl"/>
@@ -82,5 +82,5 @@
     </visual>
     <collision>
-      <origin xyz="0.0 0.0 0.0" rpy="0 0 0"/>
+      <origin xyz="0.0048 -0.0106 0.0" rpy="0 0 0"/>
       <geometry>
         <mesh filename="file://$(find trainer)/meshes/collision/cabinet_door_4.stl"/>

Commit message: MR corrections.

File: trainer/urdf/trainer_side.xacro (robot description, xacro)
@@ -94,5 +94,5 @@
     <parent link="${prefix}side_top_face"/>
     <child link="${prefix}drawer_1_face"/>
-    <origin xyz="0.004 0.006 0.282" rpy="0 0 0"/>
+    <origin xyz="0.011 0.003 0.282" rpy="0 0 0"/>
   </joint>
   <link name="${prefix}drawer_1_face">
@@ -121,5 +121,5 @@
     <parent link="${prefix}drawer_1_face"/>
     <child link="${prefix}drawer_1_left"/>
-    <origin xyz="0.293 -0.305 -0.007" rpy="0 0 0"/>
+    <origin xyz="${0.293 - 0.013} -0.305 -0.007" rpy="0 0 0"/>
   </joint>
   <link name="${prefix}drawer_1_left">
@@ -204,5 +204,5 @@
     <parent link="${prefix}side_top_face"/>
     <child link="${prefix}drawer_2_face"/>
-    <origin xyz="0.004 0.006 0.085" rpy="0 0 0"/>
+    <origin xyz="0.011 0.003 0.085" rpy="0 0 0"/>
   </joint>
   <link name="${prefix}drawer_2_face">
@@ -231,5 +231,5 @@
     <parent link="${prefix}drawer_2_face"/>
     <child link="${prefix}drawer_2_left"/>
-    <origin xyz="0.293 -0.305 -0.007" rpy="0 0 0"/>
+    <origin xyz="${0.293 - 0.013} -0.305 -0.007" rpy="0 0 0"/>
   </joint>
   <link name="${prefix}drawer_2_left">

Commit message: Minor alteration.

File: trainer/urdf/trainer_side.xacro (robot description, xacro)
@@ -94,5 +94,5 @@
     <parent link="${prefix}side_top_face"/>
     <child link="${prefix}drawer_1_face"/>
-    <origin xyz="0.011 0.003 0.282" rpy="0 0 0"/>
+    <origin xyz="0.011 0.003 0.283" rpy="0 0 0"/>
   </joint>
   <link name="${prefix}drawer_1_face">
@@ -204,5 +204,5 @@
     <parent link="${prefix}side_top_face"/>
     <child link="${prefix}drawer_2_face"/>
-    <origin xyz="0.011 0.003 0.085" rpy="0 0 0"/>
+    <origin xyz="0.011 0.003 0.086" rpy="0 0 0"/>
   </joint>
   <link name="${prefix}drawer_2_face">

Commit message: adding x offset for hinge in cabinet 4

File: trainer/urdf/trainer_side.xacro (robot description, xacro)
@@ -65,5 +65,5 @@
     <parent link="${prefix}side_top_face"/>
     <child link="${prefix}cabinet_4"/>
-    <origin xyz="0.0 0.017 0.484" rpy="0 0 0"/>
+    <origin xyz="-0.0018 0.017 0.484" rpy="0 0 0"/>
   </joint>
   <link name="${prefix}cabinet_4">

Commit message: MR changes.

File: trainer/urdf/trainer_side.xacro (robot description, xacro)
@@ -121,5 +121,5 @@
     <parent link="${prefix}drawer_1_face"/>
     <child link="${prefix}drawer_1_left"/>
-    <origin xyz="${0.293 - 0.013} -0.305 -0.007" rpy="0 0 0"/>
+    <origin xyz="${0.293 - 0.013} -0.305 -0.00435" rpy="0 0 0"/>
   </joint>
   <link name="${prefix}drawer_1_left">
@@ -148,5 +148,5 @@
     <parent link="${prefix}drawer_1_face"/>
     <child link="${prefix}drawer_1_right"/>
-    <origin xyz="0.0 -0.305 -0.007" rpy="0 0 0"/>
+    <origin xyz="0.0 -0.305 -0.00435" rpy="0 0 0"/>
   </joint>
   <link name="${prefix}drawer_1_right">
@@ -175,5 +175,5 @@
     <parent link="${prefix}drawer_1_face"/>
     <child link="${prefix}drawer_1_bottom"/>
-    <origin xyz="0.0 -0.305 -0.007" rpy="0 0 0"/>
+    <origin xyz="0.0 -0.305 -0.00435" rpy="0 0 0"/>
   </joint>
   <link name="${prefix}drawer_1_bottom">
@@ -231,5 +231,5 @@
     <parent link="${prefix}drawer_2_face"/>
     <child link="${prefix}drawer_2_left"/>
-    <origin xyz="${0.293 - 0.013} -0.305 -0.007" rpy="0 0 0"/>
+    <origin xyz="${0.293 - 0.013} -0.305 -0.00435" rpy="0 0 0"/>
   </joint>
   <link name="${prefix}drawer_2_left">
@@ -258,5 +258,5 @@
     <parent link="${prefix}drawer_2_face"/>
     <child link="${prefix}drawer_2_right"/>
-    <origin xyz="0.0 -0.305 -0.007" rpy="0 0 0"/>
+    <origin xyz="0.0 -0.305 -0.00435" rpy="0 0 0"/>
   </joint>
   <link name="${prefix}drawer_2_right">
@@ -285,5 +285,5 @@
     <parent link="${prefix}drawer_2_face"/>
     <child link="${prefix}drawer_2_bottom"/>
-    <origin xyz="0.0 -0.305 -0.007" rpy="0 0 0"/>
+    <origin xyz="0.0 -0.305 -0.00435" rpy="0 0 0"/>
   </joint>
   <link name="${prefix}drawer_2_bottom">

Commit message: Adding the paddle latch handle.

File: trainer/urdf/trainer_side.xacro (robot description, xacro)
@@ -75,5 +75,5 @@
     </inertial>
     <visual>
-      <origin xyz="0.0048 -0.0106 0.0" rpy="0 0 0"/>
+      <origin xyz="0.00305 -0.0106 0.0" rpy="0 0 0"/>
       <geometry>
         <mesh filename="file://$(find trainer)/meshes/visual/cabinet_door_4.stl"/>
@@ -82,7 +82,63 @@
     </visual>
     <collision>
-      <origin xyz="0.0048 -0.0106 0.0" rpy="0 0 0"/>
+      <origin xyz="0.00305 -0.0106 0.0" rpy="0 0 0"/>
       <geometry>
         <mesh filename="file://$(find trainer)/meshes/collision/cabinet_door_4.stl"/>
+      </geometry>
+      <material name="red"/>
+    </collision>
+  </link>
+  <joint name="${prefix}paddle_latch_housing_joint" type="fixed">
+    <parent link="${prefix}cabinet_4"/>
+    <child link="${prefix}paddle_latch_housing"/>
+    <origin xyz="0.2043 -0.007 0.1313" rpy="0 0 0"/>
+  </joint>
+  <link name="${prefix}paddle_latch_housing">
+    <!--TODO set proper inertia-->
+    <inertial>
+      <origin rpy="0 0 0" xyz="0.0 0.0 0.0"/>
+      <mass value="0.0"/>
+      <inertia ixx="0.0" ixy="0.0" ixz="0.0" iyy="0.0" iyz="0.0" izz="0.0"/>
+    </inertial>
+    <visual>
+      <origin xyz="0.00305 0.0 0.00305" rpy="0 0 0"/>
+      <geometry>
+        <mesh filename="file://$(find trainer)/meshes/visual/paddle_latch_housing.stl"/>
+      </geometry>
+      <material name="gray"/>
+    </visual>
+    <collision>
+      <origin xyz="0.00305 0.0 0.00305" rpy="0 0 0"/>
+      <geometry>
+        <mesh filename="file://$(find trainer)/meshes/collision/paddle_latch_housing.stl"/>
+      </geometry>
+      <material name="red"/>
+    </collision>
+  </link>
+  <joint name="${prefix}paddle_latch_handle_joint" type="revolute">
+    <axis xyz="0 0 -1"/>
+    <limit effort="10.0" lower="0.0" upper="0.785375" velocity="0.5"/>
+    <parent link="${prefix}paddle_latch_housing"/>
+    <child link="${prefix}paddle_latch_handle"/>
+    <origin xyz="0.06693 -0.0047 0.0107" rpy="0 0 0"/>
+  </joint>
+  <link name="${prefix}paddle_latch_handle">
+    <!--TODO set proper inertia-->
+    <inertial>
+      <origin rpy="0 0 0" xyz="0.0 0.0 0.0"/>
+      <mass value="0.0"/>
+      <inertia ixx="0.0" ixy="0.0" ixz="0.0" iyy="0.0" iyz="0.0" izz="0.0"/>
+    </inertial>
+    <visual>
+      <origin xyz="0.0 0.0 0.0" rpy="0 0 0"/>
+      <geometry>
+        <mesh filename="file://$(find trainer)/meshes/visual/paddle_latch_handle.stl"/>
+      </geometry>
+      <material name="blue"/>
+    </visual>
+    <collision>
+      <origin xyz="0.0 0.0 0.0" rpy="0 0 0"/>
+      <geometry>
+        <mesh filename="file://$(find trainer)/meshes/collision/paddle_latch_handle.stl"/>
       </geometry>
       <material name="red"/>

Commit message: Adding recessed handle.

File: trainer/urdf/trainer_side.xacro (robot description, xacro)
@@ -284,4 +284,60 @@
     </collision>
   </link>
+  <joint name="${prefix}recessed_latch_housing_joint" type="fixed">
+    <parent link="${prefix}drawer_2_face"/>
+    <child link="${prefix}recessed_latch_housing"/>
+    <origin xyz="0.1148 0.004 0.0165" rpy="0 0 0"/>
+  </joint>
+  <link name="${prefix}recessed_latch_housing">
+    <!--TODO set proper inertia-->
+    <inertial>
+      <origin rpy="0 0 0" xyz="0.0 0.0 0.0"/>
+      <mass value="0.0"/>
+      <inertia ixx="0.0" ixy="0.0" ixz="0.0" iyy="0.0" iyz="0.0" izz="0.0"/>
+    </inertial>
+    <visual>
+      <origin xyz="0.0 0.0 0.0" rpy="0 0 0"/>
+      <geometry>
+        <mesh filename="file://$(find trainer)/meshes/visual/recessed_latch_housing.stl"/>
+      </geometry>
+      <material name="gray"/>
+    </visual>
+    <collision>
+      <origin xyz="0.0 0.0 0.0" rpy="0 0 0"/>
+      <geometry>
+        <mesh filename="file://$(find trainer)/meshes/collision/recessed_latch_housing.stl"/>
+      </geometry>
+      <material name="red"/>
+    </collision>
+  </link>
+  <joint name="${prefix}recessed_latch_handle_joint" type="prismatic">
+    <axis xyz="-1 0 0"/>
+    <limit effort="10.0" lower="0.0" upper="0.2921" velocity="0.5"/>
+    <parent link="${prefix}recessed_latch_housing"/>
+    <child link="${prefix}recessed_latch_handle"/>
+    <origin xyz="0.0508 -0.0028 0.00665" rpy="0 0 0"/>
+  </joint>
+  <link name="${prefix}recessed_latch_handle">
+    <!--TODO set proper inertia-->
+    <inertial>
+      <origin rpy="0 0 0" xyz="0.0 0.0 0.0"/>
+      <mass value="0.0"/>
+      <inertia ixx="0.0" ixy="0.0" ixz="0.0" iyy="0.0" iyz="0.0" izz="0.0"/>
+    </inertial>
+    <visual>
+      <origin xyz="0.0 0.0 0.0" rpy="0 0 0"/>
+      <geometry>
+        <mesh filename="file://$(find trainer)/meshes/visual/recessed_latch_handle.stl"/>
+      </geometry>
+      <material name="blue"/>
+    </visual>
+    <collision>
+      <origin xyz="0.0 0.0 0.0" rpy="0 0 0"/>
+      <geometry>
+        <mesh filename="file://$(find trainer)/meshes/collision/recessed_latch_handle.stl"/>
+      </geometry>
+      <material name="red"/>
+    </collision>
+  </link>
   <joint name="${prefix}drawer_2_left_joint" type="fixed">
     <parent link="${prefix}drawer_2_face"/>

Commit message: adjusting y value for paddle_latch_housing to be from the back of the housing

File: trainer/urdf/trainer_side.xacro (robot description, xacro)
@@ -121,5 +121,5 @@
     <parent link="${prefix}paddle_latch_housing"/>
     <child link="${prefix}paddle_latch_handle"/>
-    <origin xyz="0.06693 -0.0047 0.0107" rpy="0 0 0"/>
+    <origin xyz="0.06693 -0.003531 0.0107" rpy="0 0 0"/>
   </joint>
   <link name="${prefix}paddle_latch_handle">

Commit message: updating recessed_latch_housing and recessed_latch_housing_handle origins

File: trainer/urdf/trainer_side.xacro (robot description, xacro)
@@ -287,5 +287,5 @@
     <parent link="${prefix}drawer_2_face"/>
     <child link="${prefix}recessed_latch_housing"/>
-    <origin xyz="0.1148 0.004 0.0165" rpy="0 0 0"/>
+    <origin xyz="0.1148 0.003175 0.0165" rpy="0 0 0"/>
   </joint>
   <link name="${prefix}recessed_latch_housing">
@@ -316,5 +316,5 @@
     <parent link="${prefix}recessed_latch_housing"/>
     <child link="${prefix}recessed_latch_handle"/>
-    <origin xyz="0.0508 -0.0028 0.00665" rpy="0 0 0"/>
+    <origin xyz="0.0508 -0.001778 0.006477" rpy="0 0 0"/>
   </joint>
   <link name="${prefix}recessed_latch_handle">
