Commit message: Fixing the origin and units.

File: trainer/urdf/trainer_frame.xacro (robot description, xacro)
@@ -3,5 +3,5 @@
     <link name="trainer">
       <visual>
-        <origin xyz="2.246 1.504 0.565" rpy="0 0 0"/>
+        <origin xyz="0.0 0.0 0.0" rpy="0 0 0"/>
           <geometry>
             <mesh filename="file://$(find trainer)/meshes/visual/ivr_tasktrainer_frame.stl"/>
@@ -12,5 +12,5 @@
       </visual>
       <collision>
-        <origin xyz="2.246 1.504 0.565" rpy="0 0 0"/>
+        <origin xyz="0.0 0.0 0.0" rpy="0 0 0"/>
           <geometry>
             <mesh filename="file://$(find trainer)/meshes/collision/ivr_tasktrainer_frame.stl"/>

Commit message: Changing to xacro macro.

File: trainer/urdf/trainer_frame.xacro (robot description, xacro)
@@ -1,5 +1,15 @@
 <?xml version="1.0"?>
-<robot xmlns:xacro="http://wiki.ros.org/xacro" name="trainer_frame">
-    <link name="trainer">
+<robot xmlns:xacro="http://wiki.ros.org/xacro">
+  <xacro:macro name="trainer_frame" params="
+    name:=''
+    prefix:=''
+    parent:=''
+    *origin">
+    <joint name="${prefix}trainer_frame_base_joint" type="fixed">
+      <parent link="${parent}"/>
+      <child link="${prefix}trainer_frame"/>
+      <xacro:insert_block name="origin"/>
+    </joint>
+    <link name="${prefix}trainer_frame">
       <visual>
         <origin xyz="0.0 0.0 0.0" rpy="0 0 0"/>
@@ -8,5 +18,5 @@
           </geometry>
         <material name="red">
-          <color rgba="1.0 0 0 0.5"/>
+          <color rgba="1.0 0 0 0.75"/>
         </material>
       </visual>
@@ -17,7 +27,8 @@
           </geometry>
         <material name="red">
-          <color rgba="1.0 0 0 0.5"/>
+          <color rgba="1.0 0 0 0.75"/>
         </material>
       </collision>
     </link>
+  </xacro:macro>
 </robot>

Commit message: Finishing collision boxes and adding inertial TODO.

File: trainer/urdf/trainer_frame.xacro (robot description, xacro)
@@ -21,11 +21,104 @@
         </material>
       </visual>
+    </link>
+    <joint name="trainer_box_joint" type="fixed">
+      <parent link="trainer_frame"/>
+      <child link="trainer_box"/>
+      <origin xyz="0.0 0.0 0.0" rpy="0 0 0"/>
+    </joint>
+    <link name="trainer_box">
+    <!--TODO: set proper inertia-->
+      <inertial>
+        <origin rpy="0 0 0" xyz="0.0 0.0 0.0"/>
+        <mass value="0.0"/>
+        <inertia ixx="0.0" ixy="0.0" ixz="0.0" iyy="0.0" iyz="0.0" izz="0.0"/>
+      </inertial>
       <collision>
-        <origin xyz="0.0 0.0 0.0" rpy="0 0 0"/>
-          <geometry>
-            <mesh filename="file://$(find trainer)/meshes/collision/ivr_tasktrainer_frame.stl"/>
-          </geometry>
+        <origin xyz="${1.27/2} 0.48 ${0.452/2}" rpy="0 0 0"/>
+        <geometry>
+          <box size="1.27 0.816 0.452"/>
+        </geometry>
         <material name="red">
-          <color rgba="1.0 0 0 0.75"/>
+          <color rgba="1.0 0 0 0.5"/>
+        </material>
+      </collision>
+    </link>
+    <joint name="trainer_top_joint" type="fixed">
+      <parent link="trainer_frame"/>
+      <child link="trainer_top"/>
+      <origin xyz="0.0 0.0 1.52" rpy="0 0 0"/>
+    </joint>
+    <link name="trainer_top">
+      <collision>
+        <origin xyz="${1.27/2} 0.48 ${0.08/2}" rpy="0 0 0"/>
+        <geometry>
+          <box size="1.27 0.816 0.08"/>
+        </geometry>
+        <material name="red">
+          <color rgba="1.0 0 0 1.0"/>
+        </material>
+      </collision>
+    </link>
+    <joint name="trainer_plane_left_joint" type="fixed">
+      <parent link="trainer_frame"/>
+      <child link="trainer_plane_left"/>
+      <origin xyz="0.0 0.0 0.0" rpy="0 0 0"/>
+    </joint>
+    <link name="trainer_plane_left">
+      <collision>
+        <origin xyz="${1.27/2} 0.04 ${1.60/2}" rpy="0 0 0"/>
+        <geometry>
+          <box size="1.27 0.08 1.60"/>
+        </geometry>
+        <material name="red">
+          <color rgba="1.0 0 0 0.5"/>
+        </material>
+      </collision>
+    </link>
+    <joint name="trainer_plane_middle_joint" type="fixed">
+      <parent link="trainer_frame"/>
+      <child link="trainer_plane_middle"/>
+      <origin xyz="0.0 0.428 0.0" rpy="0 0 0"/>
+    </joint>
+    <link name="trainer_plane_middle">
+      <collision>
+        <origin xyz="${1.27/2} 0.02 ${1.60/2}" rpy="0 0 0"/>
+        <geometry>
+          <box size="1.27 0.04 1.60"/>
+        </geometry>
+        <material name="red">
+          <color rgba="1.0 0 0 0.5"/>
+        </material>
+      </collision>
+    </link>
+    <joint name="trainer_plane_right_1_joint" type="fixed">
+      <parent link="trainer_frame"/>
+      <child link="trainer_plane_right_1"/>
+      <origin xyz="0.0 0.816 0.0" rpy="0 0 0"/>
+    </joint>
+    <link name="trainer_plane_right_1">
+      <collision>
+        <origin xyz="${0.810/2} 0.04 ${1.60/2}" rpy="0 0 0"/>
+        <geometry>
+          <box size="0.810 0.08 1.60"/>
+        </geometry>
+        <material name="red">
+          <color rgba="1.0 0 0 0.5"/>
+        </material>
+      </collision>
+    </link>
+    <joint name="trainer_plane_right_2_joint" type="fixed">
+      <parent link="trainer_frame"/>
+      <child link="trainer_plane_right_2"/>
+      <origin xyz="1.129 0.816 0.0" rpy="0 0 0"/>
+    </joint>
+    <link name="trainer_plane_right_2">
+      <collision>
+        <origin xyz="${0.13335/2} 0.04 ${1.60/2}" rpy="0 0 0"/>
+        <geometry>
+          <box size="0.13335 0.08 1.60"/>
+        </geometry>
+        <material name="red">
+          <color rgba="1.0 0 0 0.5"/>
         </material>
       </collision>

Commit message: Adding some extra collision volume around the extrusions.

File: trainer/urdf/trainer_frame.xacro (robot description, xacro)
@@ -35,7 +35,7 @@
       </inertial>
       <collision>
-        <origin xyz="${1.27/2} 0.48 ${0.452/2}" rpy="0 0 0"/>
+        <origin xyz="${1.27/2} 0.48 ${0.47/2}" rpy="0 0 0"/>
         <geometry>
-          <box size="1.27 0.816 0.452"/>
+          <box size="1.27 0.816 0.47"/>
         </geometry>
         <material name="red">
@@ -51,7 +51,7 @@
     <link name="trainer_top">
       <collision>
-        <origin xyz="${1.27/2} 0.48 ${0.08/2}" rpy="0 0 0"/>
+        <origin xyz="${1.27/2} 0.48 ${0.1/2}" rpy="0 0 0"/>
         <geometry>
-          <box size="1.27 0.816 0.08"/>
+          <box size="1.27 0.816 0.1"/>
         </geometry>
         <material name="red">
@@ -67,7 +67,7 @@
     <link name="trainer_plane_left">
       <collision>
-        <origin xyz="${1.27/2} 0.04 ${1.60/2}" rpy="0 0 0"/>
+        <origin xyz="${1.27/2} ${0.1/2} ${1.60/2}" rpy="0 0 0"/>
         <geometry>
-          <box size="1.27 0.08 1.60"/>
+          <box size="1.27 0.1 1.60"/>
         </geometry>
         <material name="red">
@@ -79,11 +79,11 @@
       <parent link="trainer_frame"/>
       <child link="trainer_plane_middle"/>
-      <origin xyz="0.0 0.428 0.0" rpy="0 0 0"/>
+      <origin xyz="0.0 0.42 0.0" rpy="0 0 0"/>
     </joint>
     <link name="trainer_plane_middle">
       <collision>
-        <origin xyz="${1.27/2} 0.02 ${1.60/2}" rpy="0 0 0"/>
+        <origin xyz="${1.27/2} ${0.05/2} ${1.60/2}" rpy="0 0 0"/>
         <geometry>
-          <box size="1.27 0.04 1.60"/>
+          <box size="1.27 0.05 1.60"/>
         </geometry>
         <material name="red">
@@ -95,11 +95,11 @@
       <parent link="trainer_frame"/>
       <child link="trainer_plane_right_1"/>
-      <origin xyz="0.0 0.816 0.0" rpy="0 0 0"/>
+      <origin xyz="0.0 0.8 0.0" rpy="0 0 0"/>
     </joint>
     <link name="trainer_plane_right_1">
       <collision>
-        <origin xyz="${0.810/2} 0.04 ${1.60/2}" rpy="0 0 0"/>
+        <origin xyz="${0.810/2} ${0.1/2} ${1.60/2}" rpy="0 0 0"/>
         <geometry>
-          <box size="0.810 0.08 1.60"/>
+          <box size="0.810 0.1 1.60"/>
         </geometry>
         <material name="red">
@@ -111,11 +111,11 @@
       <parent link="trainer_frame"/>
       <child link="trainer_plane_right_2"/>
-      <origin xyz="1.129 0.816 0.0" rpy="0 0 0"/>
+      <origin xyz="1.129 0.8 0.0" rpy="0 0 0"/>
     </joint>
     <link name="trainer_plane_right_2">
       <collision>
-        <origin xyz="${0.13335/2} 0.04 ${1.60/2}" rpy="0 0 0"/>
+        <origin xyz="${0.13335/2} ${0.1/2} ${1.60/2}" rpy="0 0 0"/>
         <geometry>
-          <box size="0.13335 0.08 1.60"/>
+          <box size="0.13335 0.1 1.60"/>
         </geometry>
         <material name="red">

Commit message: Cleaning up.

File: trainer/urdf/trainer_frame.xacro (robot description, xacro)
@@ -28,5 +28,5 @@
     </joint>
     <link name="trainer_box">
-    <!--TODO set proper inertia-->
+      <!--TODO set proper inertia-->
       <inertial>
         <origin rpy="0 0 0" xyz="0.0 0.0 0.0"/>

File: trainer/urdf/trainer_front_left_face.xacro (robot description, xacro)
@@ -13,4 +13,10 @@
   </joint>
   <link name="${prefix}front_face_plate">
+    <!--TODO set proper inertia-->
+    <inertial>
+      <origin rpy="0 0 0" xyz="0.0 0.0 0.0"/>
+      <mass value="0.0"/>
+      <inertia ixx="0.0" ixy="0.0" ixz="0.0" iyy="0.0" iyz="0.0" izz="0.0"/>
+    </inertial>
     <visual>
       <origin xyz="0.0 0.0 0.0" rpy="0 0 0"/>
@@ -32,12 +38,66 @@
     </collision>
   </link>
-  <xacro:include filename="$(find trainer)/urdf/trainer_cubby_1.xacro"/>
-  <xacro:cubby_1 name="$(arg name)" prefix="${prefix}" parent="${prefix}front_face_plate">
+  <joint name="${prefix}cubby_1_joint" type="fixed">
+    <parent link="${prefix}front_face_plate"/>
+    <child link="${prefix}cubby_1"/>
     <origin xyz="0.0 0.002 0.525" rpy="0 0 0"/>
-  </xacro:cubby_1>
-  <xacro:include filename="$(find trainer)/urdf/trainer_cubby_2.xacro"/>
-  <xacro:cubby_2 name="$(arg name)" prefix="${prefix}" parent="${prefix}front_face_plate">
+  </joint>
+  <link name="${prefix}cubby_1">
+    <!--TODO set proper inertia-->
+    <inertial>
+      <origin rpy="0 0 0" xyz="0.0 0.0 0.0"/>
+      <mass value="0.0"/>
+      <inertia ixx="0.0" ixy="0.0" ixz="0.0" iyy="0.0" iyz="0.0" izz="0.0"/>
+    </inertial>
+    <visual>
+      <origin xyz="0.0 0.0 0.0" rpy="0 0 0"/>
+        <geometry>
+          <mesh filename="file://$(find trainer)/meshes/visual/cubby_1.stl"/>
+        </geometry>
+      <material name="red">
+        <color rgba="1.0 0 0 0.75"/>
+      </material>
+    </visual>
+    <collision>
+      <origin xyz="0.0 0.0 0.0" rpy="0 0 0"/>
+        <geometry>
+          <mesh filename="file://$(find trainer)/meshes/collision/cubby_1.stl"/>
+        </geometry>
+      <material name="red">
+        <color rgba="1.0 0 0 0.75"/>
+      </material>
+    </collision>
+  </link>
+  <joint name="${prefix}cubby_2_joint" type="fixed">
+    <parent link="${prefix}front_face_plate"/>
+    <child link="${prefix}cubby_2"/>
     <origin xyz="0.0 0.002 0.875" rpy="0 0 0"/>
-  </xacro:cubby_2>
+  </joint>
+  <link name="${prefix}cubby_2">
+    <!--TODO set proper inertia-->
+    <inertial>
+      <origin rpy="0 0 0" xyz="0.0 0.0 0.0"/>
+      <mass value="0.0"/>
+      <inertia ixx="0.0" ixy="0.0" ixz="0.0" iyy="0.0" iyz="0.0" izz="0.0"/>
+    </inertial>
+    <visual>
+      <origin xyz="0.0 0.0 0.0" rpy="0 0 0"/>
+        <geometry>
+          <mesh filename="file://$(find trainer)/meshes/visual/cubby_2.stl"/>
+        </geometry>
+      <material name="red">
+        <color rgba="1.0 0 0 0.75"/>
+      </material>
+    </visual>
+    <collision>
+      <origin xyz="0.0 0.0 0.0" rpy="0 0 0"/>
+        <geometry>
+          <mesh filename="file://$(find trainer)/meshes/collision/cubby_2.stl"/>
+        </geometry>
+      <material name="red">
+        <color rgba="1.0 0 0 0.75"/>
+      </material>
+    </collision>
+  </link>
   <xacro:if value="${shelf}">
     <joint name="${prefix}trainer_cubby_shelf_joint" type="fixed">
@@ -47,4 +107,10 @@
     </joint>
     <link name="${prefix}cubby_shelf">
+      <!--TODO set proper inertia-->
+      <inertial>
+        <origin rpy="0 0 0" xyz="0.0 0.0 0.0"/>
+        <mass value="0.0"/>
+        <inertia ixx="0.0" ixy="0.0" ixz="0.0" iyy="0.0" iyz="0.0" izz="0.0"/>
+      </inertial>
       <visual>
         <origin xyz="${0.173/2} ${0.428/2} ${0.02/2}" rpy="0 0 0"/>

Commit message: Minor collision changes.

File: trainer/urdf/trainer_frame.xacro (robot description, xacro)
@@ -13,5 +13,6 @@
     <link name="${prefix}trainer_frame">
       <visual>
-        <origin xyz="0.0 0.0 0.0" rpy="0 0 0"/>
+        <!--Offset is to adjust for the radius on the extrusion-->
+        <origin xyz="0.0 0.004 0.0" rpy="0 0 0"/>
           <geometry>
             <mesh filename="file://$(find trainer)/meshes/visual/ivr_tasktrainer_frame.stl"/>
@@ -35,7 +36,7 @@
       </inertial>
       <collision>
-        <origin xyz="${1.27/2} 0.48 ${0.47/2}" rpy="0 0 0"/>
+        <origin xyz="${1.27/2} ${0.896/2} ${0.47/2}" rpy="0 0 0"/>
         <geometry>
-          <box size="1.27 0.816 0.47"/>
+          <box size="1.27 0.896 0.47"/>
         </geometry>
         <material name="red">
@@ -51,7 +52,7 @@
     <link name="trainer_top">
       <collision>
-        <origin xyz="${1.27/2} 0.48 ${0.1/2}" rpy="0 0 0"/>
+        <origin xyz="${1.27/2} ${0.896/2} ${0.1/2}" rpy="0 0 0"/>
         <geometry>
-          <box size="1.27 0.816 0.1"/>
+          <box size="1.27 0.896 0.1"/>
         </geometry>
         <material name="red">

Commit message: Updating collision primitives.

File: trainer/urdf/trainer_frame.xacro (robot description, xacro)
@@ -112,11 +112,11 @@
       <parent link="trainer_frame"/>
       <child link="trainer_plane_right_2"/>
-      <origin xyz="1.129 0.8 0.0" rpy="0 0 0"/>
+      <origin xyz="1.124 0.81 0.0" rpy="0 0 0"/>
     </joint>
     <link name="trainer_plane_right_2">
       <collision>
-        <origin xyz="${0.13335/2} ${0.1/2} ${1.60/2}" rpy="0 0 0"/>
+        <origin xyz="${0.14/2} ${0.1/2} ${1.60/2}" rpy="0 0 0"/>
         <geometry>
-          <box size="0.13335 0.1 1.60"/>
+          <box size="0.14 0.1 1.60"/>
         </geometry>
         <material name="red">

Commit message: added the missing prefixes

File: trainer/urdf/trainer_frame.xacro (robot description, xacro)
@@ -21,10 +21,10 @@
       </visual>
     </link>
-    <joint name="trainer_box_joint" type="fixed">
-      <parent link="trainer_frame"/>
-      <child link="trainer_box"/>
+    <joint name="${prefix}trainer_box_joint" type="fixed">
+      <parent link="${prefix}trainer_frame"/>
+      <child link="${prefix}trainer_box"/>
       <origin xyz="0.0 0.0 0.0" rpy="0 0 0"/>
     </joint>
-    <link name="trainer_box">
+    <link name="${prefix}trainer_box">
       <!--TODO set proper inertia-->
       <inertial>
@@ -41,10 +41,10 @@
       </collision>
     </link>
-    <joint name="trainer_top_joint" type="fixed">
-      <parent link="trainer_frame"/>
-      <child link="trainer_top"/>
+    <joint name="${prefix}trainer_top_joint" type="fixed">
+      <parent link="${prefix}trainer_frame"/>
+      <child link="${prefix}trainer_top"/>
       <origin xyz="0.0 0.0 1.52" rpy="0 0 0"/>
     </joint>
-    <link name="trainer_top">
+    <link name="${prefix}trainer_top">
       <collision>
         <origin xyz="${1.27/2} ${0.896/2} ${0.1/2}" rpy="0 0 0"/>
@@ -55,10 +55,10 @@
       </collision>
     </link>
-    <joint name="trainer_plane_left_joint" type="fixed">
-      <parent link="trainer_frame"/>
-      <child link="trainer_plane_left"/>
+    <joint name="${prefix}trainer_plane_left_joint" type="fixed">
+      <parent link="${prefix}trainer_frame"/>
+      <child link="${prefix}trainer_plane_left"/>
       <origin xyz="0.0 0.0 0.0" rpy="0 0 0"/>
     </joint>
-    <link name="trainer_plane_left">
+    <link name="${prefix}trainer_plane_left">
       <collision>
         <origin xyz="${1.27/2} ${0.1/2} ${1.60/2}" rpy="0 0 0"/>
@@ -69,10 +69,10 @@
       </collision>
     </link>
-    <joint name="trainer_plane_middle_joint" type="fixed">
-      <parent link="trainer_frame"/>
-      <child link="trainer_plane_middle"/>
+    <joint name="${prefix}trainer_plane_middle_joint" type="fixed">
+      <parent link="${prefix}trainer_frame"/>
+      <child link="${prefix}trainer_plane_middle"/>
       <origin xyz="0.0 0.42 0.0" rpy="0 0 0"/>
     </joint>
-    <link name="trainer_plane_middle">
+    <link name="${prefix}trainer_plane_middle">
       <collision>
         <origin xyz="${1.27/2} ${0.05/2} ${1.60/2}" rpy="0 0 0"/>
@@ -83,10 +83,10 @@
       </collision>
     </link>
-    <joint name="trainer_plane_right_1_joint" type="fixed">
-      <parent link="trainer_frame"/>
-      <child link="trainer_plane_right_1"/>
+    <joint name="${prefix}trainer_plane_right_1_joint" type="fixed">
+      <parent link="${prefix}trainer_frame"/>
+      <child link="${prefix}trainer_plane_right_1"/>
       <origin xyz="0.0 0.8 0.0" rpy="0 0 0"/>
     </joint>
-    <link name="trainer_plane_right_1">
+    <link name="${prefix}trainer_plane_right_1">
       <collision>
         <origin xyz="${0.810/2} ${0.1/2} ${1.60/2}" rpy="0 0 0"/>
@@ -97,10 +97,10 @@
       </collision>
     </link>
-    <joint name="trainer_plane_right_2_joint" type="fixed">
-      <parent link="trainer_frame"/>
-      <child link="trainer_plane_right_2"/>
+    <joint name="${prefix}trainer_plane_right_2_joint" type="fixed">
+      <parent link="${prefix}trainer_frame"/>
+      <child link="${prefix}trainer_plane_right_2"/>
       <origin xyz="1.124 0.81 0.0" rpy="0 0 0"/>
     </joint>
-    <link name="trainer_plane_right_2">
+    <link name="${prefix}trainer_plane_right_2">
       <collision>
         <origin xyz="${0.14/2} ${0.1/2} ${1.60/2}" rpy="0 0 0"/>
