Commit message: Updating colors.

File: trainer/urdf/bench_seat.xacro (robot description, xacro)
@@ -23,6 +23,6 @@
           <box size="0.127 0.895 0.05"/>
         </geometry>
-        <material name="green">
-          <color rgba="0.0 1.0 0 0.5"/>
+        <material name="gray">
+          <color rgba="0.85 0.85 0.85 0.75"/>
         </material>
       </visual>
@@ -32,6 +32,6 @@
           <box size="0.127 0.895 0.05"/>
         </geometry>
-        <material name="green">
-          <color rgba="0.0 1.0 0 0.5"/>
+        <material name="red">
+          <color rgba="1.0 0.0 0.0 0.75"/>
         </material>
       </collision>
@@ -48,6 +48,6 @@
           <box size="0.708 0.05 0.05"/>
         </geometry>
-        <material name="green">
-          <color rgba="0.0 1.0 0 0.5"/>
+        <material name="gray">
+          <color rgba="0.85 0.85 0.85 0.75"/>
         </material>
       </visual>
@@ -57,6 +57,6 @@
           <box size="0.708 0.05 0.05"/>
         </geometry>
-        <material name="green">
-          <color rgba="0.0 1.0 0 0.5"/>
+        <material name="red">
+          <color rgba="1.0 0.0 0.0 0.75"/>
         </material>
       </collision>
@@ -73,6 +73,6 @@
           <box size="0.708 0.05 0.05"/>
         </geometry>
-        <material name="green">
-          <color rgba="0.0 1.0 0 0.5"/>
+        <material name="gray">
+          <color rgba="0.85 0.85 0.85 0.75"/>
         </material>
       </visual>
@@ -82,6 +82,6 @@
           <box size="0.708 0.05 0.05"/>
         </geometry>
-        <material name="green">
-          <color rgba="0.0 1.0 0 0.5"/>
+        <material name="red">
+          <color rgba="1.0 0.0 0.0 0.75"/>
         </material>
       </collision>
@@ -98,6 +98,6 @@
           <box size="0.05 0.895 0.05"/>
         </geometry>
-        <material name="green">
-          <color rgba="0.0 1.0 0 0.5"/>
+        <material name="gray">
+          <color rgba="0.85 0.85 0.85 0.75"/>
         </material>
       </visual>
@@ -107,6 +107,6 @@
           <box size="0.05 0.895 0.05"/>
         </geometry>
-        <material name="green">
-          <color rgba="0.0 1.0 0 0.5"/>
+        <material name="red">
+          <color rgba="1.0 0.0 0.0 0.75"/>
         </material>
       </collision>

File: trainer/urdf/ceiling.xacro (robot description, xacro)
@@ -17,6 +17,6 @@
           <box size="1.901 1.4694 0.05"/>
         </geometry>
-        <material name="red">
-          <color rgba="1.0 0.0 0.0 0.75"/>
+        <material name="gray">
+          <color rgba="0.85 0.85 0.85 0.75"/>
         </material>
       </visual>

File: trainer/urdf/trainer_frame.xacro (robot description, xacro)
@@ -14,9 +14,9 @@
       <visual>
         <origin xyz="0.0 0.0 0.0" rpy="0 0 0"/>
-          <geometry>
-            <mesh filename="file://$(find trainer)/meshes/visual/ivr_tasktrainer_frame.stl"/>
-          </geometry>
-        <material name="red">
-          <color rgba="1.0 0 0 0.75"/>
+        <geometry>
+          <mesh filename="file://$(find trainer)/meshes/visual/ivr_tasktrainer_frame.stl"/>
+        </geometry>
+        <material name="gray">
+          <color rgba="0.85 0.85 0.85 0.75"/>
         </material>
       </visual>

File: trainer/urdf/trainer_front_left_face.xacro (robot description, xacro)
@@ -24,6 +24,6 @@
         <mesh filename="file://$(find trainer)/meshes/visual/front_left_face.stl"/>
       </geometry>
-      <material name="red">
-        <color rgba="1.0 0 0 0.75"/>
+      <material name="gray">
+        <color rgba="0.85 0.85 0.85 0.75"/>
       </material>
     </visual>
@@ -52,16 +52,16 @@
     <visual>
       <origin xyz="0.0 0.0 0.0" rpy="0 0 0"/>
-        <geometry>
-          <mesh filename="file://$(find trainer)/meshes/visual/cubby_1.stl"/>
-        </geometry>
-      <material name="red">
-        <color rgba="1.0 0 0 0.75"/>
+      <geometry>
+        <mesh filename="file://$(find trainer)/meshes/visual/cubby_1.stl"/>
+      </geometry>
+      <material name="gray">
+        <color rgba="0.85 0.85 0.85 0.75"/>
       </material>
     </visual>
     <collision>
       <origin xyz="0.0 0.0 0.0" rpy="0 0 0"/>
-        <geometry>
-          <mesh filename="file://$(find trainer)/meshes/collision/cubby_1.stl"/>
-        </geometry>
+      <geometry>
+        <mesh filename="file://$(find trainer)/meshes/collision/cubby_1.stl"/>
+      </geometry>
       <material name="red">
         <color rgba="1.0 0 0 0.75"/>
@@ -83,16 +83,16 @@
     <visual>
       <origin xyz="0.0 0.0 0.0" rpy="0 0 0"/>
-        <geometry>
-          <mesh filename="file://$(find trainer)/meshes/visual/cubby_2.stl"/>
-        </geometry>
-      <material name="red">
-        <color rgba="1.0 0 0 0.75"/>
+      <geometry>
+        <mesh filename="file://$(find trainer)/meshes/visual/cubby_2.stl"/>
+      </geometry>
+      <material name="gray">
+        <color rgba="0.85 0.85 0.85 0.75"/>
       </material>
     </visual>
     <collision>
       <origin xyz="0.0 0.0 0.0" rpy="0 0 0"/>
-        <geometry>
-          <mesh filename="file://$(find trainer)/meshes/collision/cubby_2.stl"/>
-        </geometry>
+      <geometry>
+        <mesh filename="file://$(find trainer)/meshes/collision/cubby_2.stl"/>
+      </geometry>
       <material name="red">
         <color rgba="1.0 0 0 0.75"/>
@@ -118,6 +118,6 @@
           <box size="0.173 0.428 0.02"/>
         </geometry>
-        <material name="red">
-          <color rgba="1.0 0.0 0 0.75"/>
+        <material name="gray">
+          <color rgba="0.85 0.85 0.85 0.75"/>
         </material>
       </visual>

File: trainer/urdf/trainer_front_right_face.xacro (robot description, xacro)
@@ -23,6 +23,6 @@
         <mesh filename="file://$(find trainer)/meshes/visual/front_right_face.stl"/>
       </geometry>
-      <material name="red">
-        <color rgba="1.0 0 0 0.75"/>
+      <material name="gray">
+        <color rgba="0.85 0.85 0.85 0.75"/>
       </material>
     </visual>
@@ -65,6 +65,6 @@
         <mesh filename="file://$(find trainer)/meshes/collision/cabinet_door_1.stl"/>
       </geometry>
-      <material name="blue">
-        <color rgba="0 0 1.0 0.75"/>
+      <material name="red">
+        <color rgba="1.0 0 0 0.75"/>
       </material>
     </collision>
@@ -98,6 +98,6 @@
         <mesh filename="file://$(find trainer)/meshes/collision/cabinet_door_2.stl"/>
       </geometry>
-      <material name="blue">
-        <color rgba="0 0 1.0 0.75"/>
+      <material name="red">
+        <color rgba="1.0 0 0 0.75"/>
       </material>
     </collision>
@@ -131,6 +131,6 @@
         <mesh filename="file://$(find trainer)/meshes/collision/cabinet_door_3.stl"/>
       </geometry>
-      <material name="blue">
-        <color rgba="0 0 1.0 0.75"/>
+      <material name="red">
+        <color rgba="1.0 0 0 0.75"/>
       </material>
     </collision>

File: trainer/urdf/trainer_side.xacro (robot description, xacro)
@@ -12,11 +12,17 @@
     </joint>
     <link name="${prefix}side_bottom_face">
+      <!--TODO set proper inertia-->
+      <inertial>
+        <origin rpy="0 0 0" xyz="0.0 0.0 0.0"/>
+        <mass value="0.0"/>
+        <inertia ixx="0.0" ixy="0.0" ixz="0.0" iyy="0.0" iyz="0.0" izz="0.0"/>
+      </inertial>
       <visual>
         <origin xyz="0.0 0.0 0.0" rpy="0 0 0"/>
-          <geometry>
-            <mesh filename="file://$(find trainer)/meshes/visual/side_bottom_face.stl"/>
-          </geometry>
-        <material name="red">
-          <color rgba="1.0 0 0 0.75"/>
+        <geometry>
+          <mesh filename="file://$(find trainer)/meshes/visual/side_bottom_face.stl"/>
+        </geometry>
+        <material name="gray">
+          <color rgba="0.85 0.85 0.85 0.75"/>
         </material>
       </visual>
@@ -37,11 +43,17 @@
     </joint>
     <link name="${prefix}side_top_face">
+      <!--TODO set proper inertia-->
+      <inertial>
+        <origin rpy="0 0 0" xyz="0.0 0.0 0.0"/>
+        <mass value="0.0"/>
+        <inertia ixx="0.0" ixy="0.0" ixz="0.0" iyy="0.0" iyz="0.0" izz="0.0"/>
+      </inertial>
       <visual>
         <origin xyz="0.0 0.0 0.0" rpy="0 0 0"/>
-          <geometry>
-            <mesh filename="file://$(find trainer)/meshes/visual/side_top_face.stl"/>
-          </geometry>
-        <material name="red">
-          <color rgba="1.0 0 0 0.75"/>
+        <geometry>
+          <mesh filename="file://$(find trainer)/meshes/visual/side_top_face.stl"/>
+        </geometry>
+        <material name="gray">
+          <color rgba="0.85 0.85 0.85 0.75"/>
         </material>
       </visual>
@@ -84,6 +96,6 @@
         <mesh filename="file://$(find trainer)/meshes/collision/cabinet_door_4.stl"/>
       </geometry>
-      <material name="blue">
-        <color rgba="0 0 1.0 0.75"/>
+      <material name="red">
+        <color rgba="1.0 0 0 0.75"/>
       </material>
     </collision>
@@ -117,6 +129,6 @@
         <mesh filename="file://$(find trainer)/meshes/collision/drawer_1_face.stl"/>
       </geometry>
-      <material name="blue">
-        <color rgba="0 0 1.0 0.75"/>
+      <material name="red">
+        <color rgba="1.0 0 0 0.75"/>
       </material>
     </collision>
@@ -128,20 +140,26 @@
   </joint>
   <link name="${prefix}drawer_1_left">
-    <visual>
-      <origin xyz="${0.013/2} ${0.305/2} ${0.096/2}" rpy="0 0 0"/>
-      <geometry>
-        <box size="0.013 0.305 0.096"/>
-      </geometry>
-      <material name="blue">
-        <color rgba="0 0 1.0 0.75"/>
-      </material>
-    </visual>
-    <collision>
-      <origin xyz="${0.013/2} ${0.305/2} ${0.096/2}" rpy="0 0 0"/>
-      <geometry>
-        <box size="0.013 0.305 0.096"/>
-      </geometry>
-      <material name="blue">
-        <color rgba="0 0 1.0 0.75"/>
+    <!--TODO set proper inertia-->
+    <inertial>
+      <origin rpy="0 0 0" xyz="0.0 0.0 0.0"/>
+      <mass value="0.0"/>
+      <inertia ixx="0.0" ixy="0.0" ixz="0.0" iyy="0.0" iyz="0.0" izz="0.0"/>
+    </inertial>
+    <visual>
+      <origin xyz="${0.013/2} ${0.305/2} ${0.096/2}" rpy="0 0 0"/>
+      <geometry>
+        <box size="0.013 0.305 0.096"/>
+      </geometry>
+      <material name="blue">
+        <color rgba="0 0 1.0 0.75"/>
+      </material>
+    </visual>
+    <collision>
+      <origin xyz="${0.013/2} ${0.305/2} ${0.096/2}" rpy="0 0 0"/>
+      <geometry>
+        <box size="0.013 0.305 0.096"/>
+      </geometry>
+      <material name="red">
+        <color rgba="1.0 0 0 0.75"/>
       </material>
     </collision>
@@ -153,20 +171,26 @@
   </joint>
   <link name="${prefix}drawer_1_right">
-    <visual>
-      <origin xyz="${0.013/2} ${0.305/2} ${0.096/2}" rpy="0 0 0"/>
-      <geometry>
-        <box size="0.013 0.305 0.096"/>
-      </geometry>
-      <material name="blue">
-        <color rgba="0 0 1.0 0.75"/>
-      </material>
-    </visual>
-    <collision>
-      <origin xyz="${0.013/2} ${0.305/2} ${0.096/2}" rpy="0 0 0"/>
-      <geometry>
-        <box size="0.013 0.305 0.096"/>
-      </geometry>
-      <material name="blue">
-        <color rgba="0 0 1.0 0.75"/>
+    <!--TODO set proper inertia-->
+    <inertial>
+      <origin rpy="0 0 0" xyz="0.0 0.0 0.0"/>
+      <mass value="0.0"/>
+      <inertia ixx="0.0" ixy="0.0" ixz="0.0" iyy="0.0" iyz="0.0" izz="0.0"/>
+    </inertial>
+    <visual>
+      <origin xyz="${0.013/2} ${0.305/2} ${0.096/2}" rpy="0 0 0"/>
+      <geometry>
+        <box size="0.013 0.305 0.096"/>
+      </geometry>
+      <material name="blue">
+        <color rgba="0 0 1.0 0.75"/>
+      </material>
+    </visual>
+    <collision>
+      <origin xyz="${0.013/2} ${0.305/2} ${0.096/2}" rpy="0 0 0"/>
+      <geometry>
+        <box size="0.013 0.305 0.096"/>
+      </geometry>
+      <material name="red">
+        <color rgba="1.0 0 0 0.75"/>
       </material>
     </collision>
@@ -178,4 +202,10 @@
   </joint>
   <link name="${prefix}drawer_1_bottom">
+    <!--TODO set proper inertia-->
+    <inertial>
+      <origin rpy="0 0 0" xyz="0.0 0.0 0.0"/>
+      <mass value="0.0"/>
+      <inertia ixx="0.0" ixy="0.0" ixz="0.0" iyy="0.0" iyz="0.0" izz="0.0"/>
+    </inertial>
     <visual>
       <origin xyz="${0.293/2} ${0.305/2} ${0.013/2}" rpy="0 0 0"/>
@@ -192,6 +222,6 @@
         <box size="0.293 0.305 0.013"/>
       </geometry>
-      <material name="blue">
-        <color rgba="0 0 1.0 0.75"/>
+      <material name="red">
+        <color rgba="1.0 0 0 0.75"/>
       </material>
     </collision>
@@ -225,6 +255,6 @@
         <mesh filename="file://$(find trainer)/meshes/collision/drawer_2_face.stl"/>
       </geometry>
-      <material name="blue">
-        <color rgba="0 0 1.0 0.75"/>
+      <material name="red">
+        <color rgba="1.0 0 0 0.75"/>
       </material>
     </collision>
@@ -236,20 +266,26 @@
   </joint>
   <link name="${prefix}drawer_2_left">
-    <visual>
-      <origin xyz="${0.013/2} ${0.305/2} ${0.096/2}" rpy="0 0 0"/>
-      <geometry>
-        <box size="0.013 0.305 0.096"/>
-      </geometry>
-      <material name="blue">
-        <color rgba="0 0 1.0 0.75"/>
-      </material>
-    </visual>
-    <collision>
-      <origin xyz="${0.013/2} ${0.305/2} ${0.096/2}" rpy="0 0 0"/>
-      <geometry>
-        <box size="0.013 0.305 0.096"/>
-      </geometry>
-      <material name="blue">
-        <color rgba="0 0 1.0 0.75"/>
+    <!--TODO set proper inertia-->
+    <inertial>
+      <origin rpy="0 0 0" xyz="0.0 0.0 0.0"/>
+      <mass value="0.0"/>
+      <inertia ixx="0.0" ixy="0.0" ixz="0.0" iyy="0.0" iyz="0.0" izz="0.0"/>
+    </inertial>
+    <visual>
+      <origin xyz="${0.013/2} ${0.305/2} ${0.096/2}" rpy="0 0 0"/>
+      <geometry>
+        <box size="0.013 0.305 0.096"/>
+      </geometry>
+      <material name="blue">
+        <color rgba="0 0 1.0 0.75"/>
+      </material>
+    </visual>
+    <collision>
+      <origin xyz="${0.013/2} ${0.305/2} ${0.096/2}" rpy="0 0 0"/>
+      <geometry>
+        <box size="0.013 0.305 0.096"/>
+      </geometry>
+      <material name="red">
+        <color rgba="1.0 0 0 0.75"/>
       </material>
     </collision>
@@ -261,20 +297,26 @@
   </joint>
   <link name="${prefix}drawer_2_right">
-    <visual>
-      <origin xyz="${0.013/2} ${0.305/2} ${0.096/2}" rpy="0 0 0"/>
-      <geometry>
-        <box size="0.013 0.305 0.096"/>
-      </geometry>
-      <material name="blue">
-        <color rgba="0 0 1.0 0.75"/>
-      </material>
-    </visual>
-    <collision>
-      <origin xyz="${0.013/2} ${0.305/2} ${0.096/2}" rpy="0 0 0"/>
-      <geometry>
-        <box size="0.013 0.305 0.096"/>
-      </geometry>
-      <material name="blue">
-        <color rgba="0 0 1.0 0.75"/>
+    <!--TODO set proper inertia-->
+    <inertial>
+      <origin rpy="0 0 0" xyz="0.0 0.0 0.0"/>
+      <mass value="0.0"/>
+      <inertia ixx="0.0" ixy="0.0" ixz="0.0" iyy="0.0" iyz="0.0" izz="0.0"/>
+    </inertial>
+    <visual>
+      <origin xyz="${0.013/2} ${0.305/2} ${0.096/2}" rpy="0 0 0"/>
+      <geometry>
+        <box size="0.013 0.305 0.096"/>
+      </geometry>
+      <material name="blue">
+        <color rgba="0 0 1.0 0.75"/>
+      </material>
+    </visual>
+    <collision>
+      <origin xyz="${0.013/2} ${0.305/2} ${0.096/2}" rpy="0 0 0"/>
+      <geometry>
+        <box size="0.013 0.305 0.096"/>
+      </geometry>
+      <material name="red">
+        <color rgba="1.0 0 0 0.75"/>
       </material>
     </collision>
@@ -286,4 +328,10 @@
   </joint>
   <link name="${prefix}drawer_2_bottom">
+    <!--TODO set proper inertia-->
+    <inertial>
+      <origin rpy="0 0 0" xyz="0.0 0.0 0.0"/>
+      <mass value="0.0"/>
+      <inertia ixx="0.0" ixy="0.0" ixz="0.0" iyy="0.0" iyz="0.0" izz="0.0"/>
+    </inertial>
     <visual>
       <origin xyz="${0.293/2} ${0.305/2} ${0.013/2}" rpy="0 0 0"/>
@@ -300,6 +348,6 @@
         <box size="0.293 0.305 0.013"/>
       </geometry>
-      <material name="blue">
-        <color rgba="0 0 1.0 0.75"/>
+      <material name="red">
+        <color rgba="1.0 0 0 0.75"/>
       </material>
     </collision>

Commit message: One branch to rule them all.

File: trainer/urdf/bench_seat.xacro (robot description, xacro)
@@ -19,7 +19,7 @@
       </inertial>
       <visual>
-        <origin xyz="${0.127/2} ${0.895/2} ${0.05/2}" rpy="0 0 0"/>
+        <origin xyz="${0.127/2} ${0.895/2} ${0.04/2}" rpy="0 0 0"/>
         <geometry>
-          <box size="0.127 0.895 0.05"/>
+          <box size="0.127 0.895 0.04"/>
         </geometry>
         <material name="gray"/>
@@ -40,7 +40,7 @@
     <link name="${prefix}bench_left">
       <visual>
-        <origin xyz="${0.708/2} ${0.05/2} ${0.05/2}" rpy="0 0 0"/>
+        <origin xyz="${0.708/2} ${0.04/2} ${0.04/2}" rpy="0 0 0"/>
         <geometry>
-          <box size="0.708 0.05 0.05"/>
+          <box size="0.708 0.04 0.04"/>
         </geometry>
         <material name="gray"/>
@@ -61,7 +61,7 @@
     <link name="${prefix}bench_right">
       <visual>
-        <origin xyz="${0.708/2} ${0.05/2} ${0.05/2}" rpy="0 0 0"/>
+        <origin xyz="${0.708/2} ${0.05/2} ${0.04/2}" rpy="0 0 0"/>
         <geometry>
-          <box size="0.708 0.05 0.05"/>
+          <box size="0.708 0.04 0.04"/>
         </geometry>
         <material name="gray"/>
@@ -82,7 +82,7 @@
     <link name="${prefix}bench_front">
       <visual>
-        <origin xyz="${0.05/2} ${0.895/2} ${0.05/2}" rpy="0 0 0"/>
+        <origin xyz="${0.05/2} ${0.895/2} ${0.04/2}" rpy="0 0 0"/>
         <geometry>
-          <box size="0.05 0.895 0.05"/>
+          <box size="0.04 0.895 0.04"/>
         </geometry>
         <material name="gray"/>
@@ -101,5 +101,5 @@
       <parent link="${prefix}bench_back"/>
       <child link="${prefix}bench_lid"/>
-      <origin xyz="0.127 0.0 0.05" rpy="0 0 0"/>
+      <origin xyz="0.127 0.0 0.0475" rpy="0 0 0"/>
     </joint>
     <link name="${prefix}bench_lid">
@@ -111,14 +111,16 @@
       </inertial>
       <visual>
-        <origin xyz="${0.603/2} ${0.895/2} ${0.05/2}" rpy="0 0 0"/>
+        <!--0.0075 is the radius of the hinge-->
+        <origin xyz="${0.603/2 + 0.0075} ${0.920/2} ${0.065/2 - 0.0075}" rpy="0 0 0"/>
         <geometry>
-          <box size="0.603 0.895 0.05"/>
+          <box size="0.603 0.920 0.065"/>
         </geometry>
         <material name="blue"/>
       </visual>
       <collision>
-        <origin xyz="${0.603/2} ${0.895/2} ${0.05/2}" rpy="0 0 0"/>
+        <!--0.0075 is the radius of the hinge-->
+        <origin xyz="${0.603/2 + 0.0075} ${0.920/2} ${0.065/2 - 0.0075}" rpy="0 0 0"/>
         <geometry>
-          <box size="0.603 0.895 0.05"/>
+          <box size="0.603 0.920 ${0.065/2}"/>
         </geometry>
         <material name="blue"/>

File: trainer/urdf/trainer_frame.xacro (robot description, xacro)
@@ -13,5 +13,6 @@
     <link name="${prefix}trainer_frame">
       <visual>
-        <origin xyz="0.0 0.0 0.0" rpy="0 0 0"/>
+        <!--Offset is to adjust for the radius on the extrusion-->
+        <origin xyz="0.0 0.004 0.0" rpy="0 0 0"/>
         <geometry>
           <mesh filename="file://$(find trainer)/meshes/visual/ivr_tasktrainer_frame.stl"/>

Commit message: Adding calibration frames for the trainer and bench.

File: trainer/urdf/bench_seat.xacro (robot description, xacro)
@@ -127,4 +127,16 @@
       </collision>
     </link>
+    <joint name="${prefix}bench_left_cal_joint" type="fixed">
+      <parent link="${prefix}bench_front"/>
+      <child link="${prefix}bench_left_cal_frame"/>
+      <origin xyz="0.045 0.0 0.0" rpy="0 0 0"/>
+    </joint>
+    <link name="${prefix}bench_left_cal_frame"/>
+    <joint name="${prefix}bench_right_cal_joint" type="fixed">
+      <parent link="${prefix}bench_right"/>
+      <child link="${prefix}bench_right_cal_frame"/>
+      <origin xyz="0.7062 0.05 0.0" rpy="0 0 0"/>
+    </joint>
+    <link name="${prefix}bench_right_cal_frame"/>
   </xacro:macro>
 </robot>

Commit message: updating bench seat angle to 95 degrees max

File: trainer/urdf/bench_seat.xacro (robot description, xacro)
@@ -98,5 +98,6 @@
     <joint name="${prefix}bench_lid_joint" type="revolute">
       <axis xyz="0 -1 0"/>
-      <limit effort="10.0" lower="0.0" upper="1.57" velocity="0.5"/>
+      <!-- upper is 95 degrees -->
+      <limit effort="10.0" lower="0.0" upper="1.65806" velocity="0.5"/>
       <parent link="${prefix}bench_back"/>
       <child link="${prefix}bench_lid"/>

Commit message: Fixing collision box on the bench seat lid.

File: trainer/urdf/bench_seat.xacro (robot description, xacro)
@@ -136,5 +136,5 @@
         <origin xyz="${0.603/2 + 0.0075} ${0.920/2} ${0.065/2 - 0.0075}" rpy="0 0 0"/>
         <geometry>
-          <box size="0.603 0.920 ${0.065/2}"/>
+          <box size="0.603 0.920 0.065"/>
         </geometry>
         <material name="blue"/>

Commit message: Replaced bench collision box with mesh.

File: trainer/urdf/bench_seat.xacro (robot description, xacro)
@@ -134,7 +134,7 @@
       <collision>
         <!--0.0075 is the radius of the hinge-->
-        <origin xyz="${0.603/2 + 0.0075} ${0.920/2} ${0.065/2 - 0.0075}" rpy="0 0 0"/>
+        <origin xyz="0.0 0.0 0.0" rpy="0 0 0"/>
         <geometry>
-          <box size="0.603 0.920 0.065"/>
+          <mesh filename="package://trainer/meshes/visual/bench_lid.stl"/>
         </geometry>
         <material name="blue"/>

Commit message: fix bench collision geometry

File: trainer/urdf/bench_seat.xacro (robot description, xacro)
@@ -25,7 +25,7 @@
       </visual>
       <collision>
-        <origin xyz="${0.127/2} ${0.895/2} ${0.05/2}" rpy="0 0 0"/>
+        <origin xyz="${0.127/2} ${0.895/2} ${0.04/2}" rpy="0 0 0"/>
         <geometry>
-          <box size="0.127 0.895 0.05"/>
+          <box size="0.127 0.895 0.04"/>
         </geometry>
         <material name="red"/>
@@ -51,7 +51,7 @@
       </visual>
       <collision>
-        <origin xyz="${0.708/2} ${0.05/2} ${0.05/2}" rpy="0 0 0"/>
+        <origin xyz="${0.708/2} ${0.04/2} ${0.04/2}" rpy="0 0 0"/>
         <geometry>
-          <box size="0.708 0.05 0.05"/>
+          <box size="0.708 0.04 0.04"/>
         </geometry>
         <material name="red"/>
@@ -77,7 +77,7 @@
       </visual>
       <collision>
-        <origin xyz="${0.708/2} ${0.05/2} ${0.05/2}" rpy="0 0 0"/>
+        <origin xyz="${0.708/2} ${0.05/2} ${0.04/2}" rpy="0 0 0"/>
         <geometry>
-          <box size="0.708 0.05 0.05"/>
+          <box size="0.708 0.04 0.04"/>
         </geometry>
         <material name="red"/>
@@ -103,7 +103,7 @@
       </visual>
       <collision>
-        <origin xyz="${0.05/2} ${0.895/2} ${0.05/2}" rpy="0 0 0"/>
+        <origin xyz="${0.05/2} ${0.895/2} ${0.04/2}" rpy="0 0 0"/>
         <geometry>
-          <box size="0.05 0.895 0.05"/>
+          <box size="0.04 0.895 0.04"/>
         </geometry>
         <material name="red"/>
