Commit message: added red tape texture to trainer bench_lid

File: trainer/urdf/bench_seat.xacro (robot description, xacro)
@@ -129,7 +129,9 @@
         <origin xyz="0.0 0.0 0.0" rpy="0 0 0"/>
         <geometry>
-          <mesh filename="package://trainer/meshes/visual/bench_lid.stl"/>
+          <mesh filename="package://trainer/meshes/visual/imetro_bench_lid.dae"/>
         </geometry>
-        <material name="blue"/>
+        <material name="${prefix}bench_lid_texture">
+          <texture filename="package://trainer/meshes/visual/bench_lid_texture.png"/>
+        </material>
       </visual>
       <collision>

Commit message: updated bench seat mass to match real weighed mass

File: trainer/urdf/bench_seat.xacro (robot description, xacro)
@@ -123,5 +123,5 @@
       <inertial>
         <origin xyz="0.2652256 0.46 0.03190335" rpy="0 0 0"/>
-        <mass value="9.07185"/>
+        <mass value="11.5"/>
         <inertia ixx="0.643167" ixy="0.0" ixz="0.002867943" iyy="0.2210995" iyz="0.0" izz="0.8576681"/>
       </inertial>
