Commit message: Fixed the hatch rotation and added parts for the handles.

File: hatch_4040/urdf/colors.xacro (robot description, xacro)
@@ -11,5 +11,5 @@
   </material>
   <material name="gray">
-    <color rgba="0.85 0.85 0.85 0.75"/>
+    <color rgba="0.85 0.85 0.85 1.0"/>
   </material>
 </robot>

File: hatch_4040/urdf/hatch_4040.xacro (robot description, xacro)
@@ -38,5 +38,5 @@
       <parent link="${prefix}hatch_4040_frame"/>
       <child link="${prefix}hatch_4040_face"/>
-      <origin xyz="0.083 1.22 0.0982" rpy="0 0 0"/>
+      <origin xyz="0.083 1.215 0.103" rpy="0 0 0"/>
     </joint>
     <link name="${prefix}hatch_4040_face">
