Commit message: Updates for the MR.

File: hatch_4040/urdf/crank_wheel.xacro (robot description, xacro)
@@ -42,5 +42,5 @@
       <parent link="${prefix}rotary_wheel"/>
       <child link="${prefix}rotary_handle"/>
-      <origin xyz="0.053975 0.0 0.0190500" rpy="0 0 0"/>
+      <origin xyz="0.053975 0.0 0.0155" rpy="0 0 0"/>
     </joint>
     <link name="${prefix}rotary_handle">
@@ -52,5 +52,5 @@
       </inertial>
       <visual>
-        <origin xyz="0.0 0.0 0.0" rpy="0 0 0"/>
+        <origin xyz="0.0 0.0 0.00355" rpy="0 0 0"/>
         <geometry>
           <mesh filename="file://$(find hatch_4040)/meshes/visual/crank_handle.stl"/>
@@ -59,5 +59,5 @@
       </visual>
       <collision>
-        <origin xyz="0.0 0.0 0.0" rpy="0 0 0"/>
+        <origin xyz="0.0 0.0 0.00355" rpy="0 0 0"/>
         <geometry>
           <mesh filename="file://$(find hatch_4040)/meshes/collision/crank_handle.stl"/>

File: hatch_4040/urdf/grab_handle.xacro (robot description, xacro)
@@ -20,7 +20,7 @@
       <visual>
         <!--This transform is for the stl file origin-->
-        <origin xyz="-0.92001848 0.1492 0.0403" rpy="0 0 0"/>
+        <origin xyz="0.0 0.0 0.0" rpy="0 0 0"/>
         <geometry>
-          <mesh filename="file://$(find hatch_4040)/meshes/visual/grab_handle.stl" scale="0.254 0.254 0.254"/>
+          <mesh filename="file://$(find hatch_4040)/meshes/visual/grab_handle.stl"/>
         </geometry>
         <material name="gray"/>
@@ -30,5 +30,5 @@
         <origin xyz="0.0 0.0 0.0" rpy="0 0 0"/>
         <geometry>
-          <mesh filename="file://$(find hatch_4040)/meshes/collision/grab_handle.stl" scale="0.254 0.254 0.254"/>
+          <mesh filename="file://$(find hatch_4040)/meshes/collision/grab_handle.stl"/>
         </geometry>
         <material name="red"/>

File: hatch_4040/urdf/hatch_4040.xacro (robot description, xacro)
@@ -64,12 +64,12 @@
     <xacro:include filename="$(find hatch_4040)/urdf/crank_wheel.xacro"/>
     <xacro:crank_wheel name="$(arg name)" prefix="$(arg prefix)external_" parent="${prefix}hatch_4040_face">
-      <origin xyz="0.0522475 -0.473371 0.606772" rpy="0 ${pi/2} 0"/>
+      <origin xyz="0.0522475 -0.473371 0.604" rpy="0 ${pi/2} 0"/>
     </xacro:crank_wheel>
     <xacro:crank_wheel name="$(arg name)" prefix="$(arg prefix)internal_" parent="${prefix}hatch_4040_face">
-      <origin xyz="-0.1795475 -0.473371 0.606772" rpy="0 -${pi/2} 0"/>
+      <origin xyz="-0.1795475 -0.473371 0.604" rpy="0 -${pi/2} 0"/>
     </xacro:crank_wheel>
     <xacro:include filename="$(find hatch_4040)/urdf/grab_handle.xacro"/>
     <xacro:grab_handle name="$(arg name)" prefix="$(arg prefix)external_" parent="${prefix}hatch_4040_face">
-      <origin xyz="-0.0497 -0.788394 0.3147147" rpy="0 0 0"/>
+      <origin xyz="-0.0497 -0.788394 0.3147147" rpy="-0.436332 0 0"/>
     </xacro:grab_handle>
     <xacro:grab_handle name="$(arg name)" prefix="$(arg prefix)internal_" parent="${prefix}hatch_4040_face">

File: hatch_frame/urdf/hatch_frame.xacro (robot description, xacro)
@@ -57,5 +57,5 @@
       <parent link="hatch_bottom"/>
       <child link="hatch_front"/>
-      <origin xyz="0.589 0.0 0.0" rpy="0 0 0"/>
+      <origin xyz="0.578 0.0 0.0" rpy="0 0 0"/>
     </joint>
     <link name="hatch_front">
