Commit message: Adding the hatch frame, still needs a simplified collision hatch face.

File: hatch_4040/urdf/hatch_4040.urdf.xacro (robot description, xacro)
@@ -3,9 +3,13 @@
   <xacro:arg name="name" default=""/>
   <xacro:arg name="prefix" default=""/>
+  <xacro:include filename="$(find hatch_frame)/urdf/hatch_frame.xacro"/>
   <xacro:include filename="$(find hatch_4040)/urdf/colors.xacro"/>
   <xacro:include filename="$(find hatch_4040)/urdf/hatch_4040.xacro"/>
   <link name="world"/>
-  <xacro:hatch_4040 name="$(arg name)" prefix="$(arg prefix)" parent="world">
+  <xacro:hatch_frame name="$(arg name)" prefix="$(arg prefix)" parent="world">
     <origin xyz="0 0 0" rpy="0 0 0"/>
+  </xacro:hatch_frame>
+  <xacro:hatch_4040 name="$(arg name)" prefix="$(arg prefix)" parent="hatch_frame">
+    <origin xyz="0.668 0.02 0.657" rpy="0 0 0"/>
   </xacro:hatch_4040>
 </robot>

File: hatch_4040/urdf/hatch_4040.xacro (robot description, xacro)
@@ -6,24 +6,10 @@
     parent:=''
     *origin">
-    <joint name="${prefix}hatch_4040_base_joint" type="fixed">
-      <parent link="${parent}"/>
-      <child link="${prefix}hatch_4040"/>
+    <joint name="${prefix}hatch_4040_frame_joint" type="fixed">
+      <parent link="${prefix}${parent}"/>
+      <child link="${prefix}hatch_4040_frame"/>
       <xacro:insert_block name="origin"/>
     </joint>
-    <link name="${prefix}hatch_4040">
-      <visual>
-        <origin xyz="0.0 0.0 0.0" rpy="0 0 0"/>
-          <geometry>
-            <mesh filename="file://$(find hatch_4040)/meshes/visual/hatch_4040.stl"/>
-          </geometry>
-        <material name="gray"/>
-      </visual>
-    </link>
-    <joint name="hatch_4040_joint" type="fixed">
-      <parent link="hatch_4040"/>
-      <child link="hatch_bottom"/>
-      <origin xyz="0.0 0.0 0.0" rpy="0 0 0"/>
-    </joint>
-    <link name="hatch_bottom">
+    <link name="${prefix}hatch_4040_frame">
       <!--TODO set proper inertia-->
       <inertial>
@@ -32,78 +18,38 @@
         <inertia ixx="0.0" ixy="0.0" ixz="0.0" iyy="0.0" iyz="0.0" izz="0.0"/>
       </inertial>
+      <visual>
+        <origin xyz="0.0 0.0 0.0" rpy="0 0 0"/>
+        <geometry>
+          <mesh filename="file://$(find hatch_4040)/meshes/visual/hatch_4040_frame.stl"/>
+        </geometry>
+        <material name="gray"/>
+      </visual>
       <collision>
-        <origin xyz="${0.675/2} ${1.307/2} ${0.04/2}" rpy="0 0 0"/>
+        <origin xyz="0.0 0.0 0.0" rpy="0 0 0"/>
         <geometry>
-          <box size="0.675 1.307 0.04"/>
+          <mesh filename="file://$(find hatch_4040)/meshes/visual/hatch_4040_frame.stl"/>
         </geometry>
         <material name="red"/>
       </collision>
     </link>
-    <joint name="hatch_bottom_back" type="fixed">
-      <parent link="hatch_bottom"/>
-      <child link="hatch_back"/>
-      <origin xyz="0.0 0.0 0.0" rpy="0 0 0"/>
+    <joint name="${prefix}hatch_4040_frame_face_joint" type="revolute">
+      <axis xyz="0 0 1"/>
+      <limit effort="10.0" lower="0.0" upper="3.14" velocity="0.5"/>
+      <parent link="${prefix}hatch_4040_frame"/>
+      <child link="${prefix}hatch_4040_face"/>
+      <origin xyz="0.083 1.22 0.0982" rpy="0 0 0"/>
     </joint>
-    <link name="hatch_back">
+    <link name="${prefix}hatch_4040_face">
+      <visual>
+        <origin xyz="0.0 0.0 0.0" rpy="0 0 0"/>
+        <geometry>
+          <mesh filename="file://$(find hatch_4040)/meshes/visual/hatch_4040_face.stl"/>
+        </geometry>
+        <material name="gray"/>
+      </visual>
       <collision>
-        <origin xyz="${0.1/2} ${1.307/2} ${0.610/2}" rpy="0 0 0"/>
+        <origin xyz="0.0 0.0 0.0" rpy="0 0 0"/>
         <geometry>
-          <box size="0.1 1.307 0.610"/>
-        </geometry>
-        <material name="red"/>
-      </collision>
-    </link>
-    <joint name="hatch_bottom_front" type="fixed">
-      <parent link="hatch_bottom"/>
-      <child link="hatch_front"/>
-      <origin xyz="0.589 0.0 0.0" rpy="0 0 0"/>
-    </joint>
-    <link name="hatch_front">
-      <collision>
-        <origin xyz="${0.1/2} ${1.307/2} ${0.610/2}" rpy="0 0 0"/>
-        <geometry>
-          <box size="0.1 1.307 0.610"/>
-        </geometry>
-        <material name="red"/>
-      </collision>
-    </link>
-    <joint name="hatch_bottom_left" type="fixed">
-      <parent link="hatch_bottom"/>
-      <child link="hatch_left"/>
-      <origin xyz="0.0 -0.01 0.0" rpy="0 0 0"/>
-    </joint>
-    <link name="hatch_left">
-      <collision>
-        <origin xyz="${0.675/2} ${0.1/2} ${2.1082/2}" rpy="0 0 0"/>
-        <geometry>
-          <box size="0.675 0.1 2.1082"/>
-        </geometry>
-        <material name="red"/>
-      </collision>
-    </link>
-    <joint name="hatch_bottom_right" type="fixed">
-      <parent link="hatch_bottom"/>
-      <child link="hatch_right"/>
-      <origin xyz="0.0 1.22 0.0" rpy="0 0 0"/>
-    </joint>
-    <link name="hatch_right">
-      <collision>
-        <origin xyz="${0.675/2} ${0.1/2} ${2.108/2}" rpy="0 0 0"/>
-        <geometry>
-          <box size="0.675 0.1 2.1082"/>
-        </geometry>
-        <material name="red"/>
-      </collision>
-    </link>
-    <joint name="hatch_bottom_top" type="fixed">
-      <parent link="hatch_bottom"/>
-      <child link="hatch_top"/>
-      <origin xyz="0.589 0.0 1.913" rpy="0 0 0"/>
-    </joint>
-    <link name="hatch_top">
-      <collision>
-        <origin xyz="${0.1/2} ${1.307/2} ${0.197/2}" rpy="0 0 0"/>
-        <geometry>
-          <box size="0.1 1.307 0.197"/>
+          <mesh filename="file://$(find hatch_4040)/meshes/collision/hatch_4040_face.stl"/>
         </geometry>
         <material name="red"/>

File: hatch_frame/urdf/hatch_frame.urdf.xacro (robot description, xacro)
@@ -4,4 +4,5 @@
   <xacro:arg name="prefix" default=""/>
   <xacro:include filename="$(find hatch_frame)/urdf/hatch_frame.xacro"/>
+  <xacro:include filename="$(find hatch_frame)/urdf/colors.xacro"/>
   <link name="world"/>
   <xacro:hatch_frame name="$(arg name)" prefix="$(arg prefix)" parent="world">

File: hatch_frame/urdf/hatch_frame.xacro (robot description, xacro)
@@ -14,19 +14,15 @@
       <visual>
         <origin xyz="0.0 0.0 0.0" rpy="0 0 0"/>
-          <geometry>
-            <mesh filename="file://$(find hatch_frame)/meshes/visual/ivr_hatch_frame.stl"/>
-          </geometry>
-        <material name="red">
-          <color rgba="1.0 0 0 0.75"/>
-        </material>
+        <geometry>
+          <mesh filename="file://$(find hatch_frame)/meshes/visual/ivr_hatch_frame.stl"/>
+        </geometry>
+        <material name="gray"/>
       </visual>
       <collision>
         <origin xyz="0.0 0.0 0.0" rpy="0 0 0"/>
-          <geometry>
-            <mesh filename="file://$(find hatch_frame)/meshes/collision/ivr_hatch_frame.stl"/>
-          </geometry>
-        <material name="red">
-          <color rgba="1.0 0 0 0.75"/>
-        </material>
+        <geometry>
+          <mesh filename="file://$(find hatch_frame)/meshes/collision/ivr_hatch_frame.stl"/>
+        </geometry>
+        <material name="red"/>
       </collision>
     </link>

Commit message: Fixing minor misalignment.

File: hatch_4040/urdf/hatch_4040.urdf.xacro (robot description, xacro)
@@ -11,5 +11,5 @@
   </xacro:hatch_frame>
   <xacro:hatch_4040 name="$(arg name)" prefix="$(arg prefix)" parent="hatch_frame">
-    <origin xyz="0.668 0.02 0.657" rpy="0 0 0"/>
+    <origin xyz="0.668 0.06 0.657" rpy="0 0 0"/>
   </xacro:hatch_4040>
 </robot>

Commit message: Adding todos and siwtching to hatch_accessories.

File: hatch_4040/urdf/hatch_4040.urdf.xacro (robot description, xacro)
@@ -3,6 +3,6 @@
   <xacro:arg name="name" default=""/>
   <xacro:arg name="prefix" default=""/>
-  <xacro:include filename="$(find hatch_frame)/urdf/hatch_frame.xacro"/>
-  <xacro:include filename="$(find hatch_frame)/urdf/colors.xacro"/>
+  <xacro:include filename="$(find hatch_accessories)/urdf/hatch_frame.xacro"/>
+  <xacro:include filename="$(find hatch_accessories)/urdf/colors.xacro"/>
   <xacro:include filename="$(find hatch_4040)/urdf/hatch_4040.xacro"/>
   <link name="world"/>

File: hatch_4040/urdf/hatch_4040.xacro (robot description, xacro)
@@ -62,5 +62,5 @@
       </collision>
     </link>
-    <xacro:include filename="$(find hatch_frame)/urdf/crank_wheel.xacro"/>
+    <xacro:include filename="$(find hatch_accessories)/urdf/crank_wheel.xacro"/>
     <xacro:crank_wheel name="$(arg name)" prefix="$(arg prefix)external_" parent="${prefix}hatch_4040_face">
       <origin xyz="0.04431 -0.473371 0.604" rpy="0 ${pi/2} 0"/>
@@ -69,5 +69,5 @@
       <origin xyz="-0.1716 -0.473371 0.604" rpy="0 -${pi/2} 0"/>
     </xacro:crank_wheel>
-    <xacro:include filename="$(find hatch_frame)/urdf/grab_handle.xacro"/>
+    <xacro:include filename="$(find hatch_accessories)/urdf/grab_handle.xacro"/>
     <xacro:grab_handle name="$(arg name)" prefix="$(arg prefix)external_" parent="${prefix}hatch_4040_face">
       <origin xyz="-0.0497 -0.788394 0.3147147" rpy="-0.3926991 0 0"/>

File: hatch_4060/urdf/hatch_4060.urdf.xacro (robot description, xacro)
@@ -3,10 +3,11 @@
   <xacro:arg name="name" default=""/>
   <xacro:arg name="prefix" default=""/>
+  <!--TODO which handles are mounted?-->
   <xacro:property name="external_handle_1" default="true"/>
   <xacro:property name="external_handle_2" default="false"/>
   <xacro:property name="internal_handle_1" default="true"/>
   <xacro:property name="internal_handle_2" default="false"/>
-  <xacro:include filename="$(find hatch_frame)/urdf/hatch_frame.xacro"/>
-  <xacro:include filename="$(find hatch_frame)/urdf/colors.xacro"/>
+  <xacro:include filename="$(find hatch_accessories)/urdf/hatch_frame.xacro"/>
+  <xacro:include filename="$(find hatch_accessories)/urdf/colors.xacro"/>
   <xacro:include filename="$(find hatch_4060)/urdf/hatch_4060.xacro"/>
   <link name="world"/>

File: hatch_4060/urdf/hatch_4060.xacro (robot description, xacro)
@@ -51,4 +51,5 @@
         <inertia ixx="0.0" ixy="0.0" ixz="0.0" iyy="0.0" iyz="0.0" izz="0.0"/>
       </inertial>
+      <!--TODO check the orientation of the hinges, up or down-->
       <visual>
         <origin xyz="0.0 0.0 0.0" rpy="0 0 0"/>
@@ -66,5 +67,6 @@
       </collision>
     </link>
-    <xacro:include filename="$(find hatch_frame)/urdf/crank_wheel.xacro"/>
+    <xacro:include filename="$(find hatch_accessories)/urdf/crank_wheel.xacro"/>
+    <!--TODO are the centers located properly?-->
     <xacro:crank_wheel name="$(arg name)" prefix="$(arg prefix)external_" parent="${prefix}hatch_4060_face">
       <origin xyz="0.0522475 -0.9474 0.4295" rpy="0 ${pi/2} 0"/>
@@ -73,5 +75,6 @@
       <origin xyz="-0.1795475 -0.9474 0.4295" rpy="0 -${pi/2} 0"/>
     </xacro:crank_wheel>
-    <xacro:include filename="$(find hatch_frame)/urdf/grab_handle.xacro"/>
+    <xacro:include filename="$(find hatch_accessories)/urdf/grab_handle.xacro"/>
+    <!--TODO which handles are mounted?-->
     <xacro:if value="${external_handle_1}">
       <xacro:grab_handle name="$(arg name)" prefix="$(arg prefix)external_1_" parent="${prefix}hatch_4060_face">

File: hatch_accessories/urdf/crank_wheel.xacro (robot description, xacro)
@@ -24,12 +24,12 @@
         <origin xyz="0.0 0.0 0.0" rpy="0 0 0"/>
         <geometry>
-          <mesh filename="file://$(find hatch_frame)/meshes/visual/crank_wheel.stl"/>
+          <mesh filename="file://$(find hatch_accessories)/meshes/visual/crank_wheel.stl"/>
         </geometry>
-        <material name="gray"/>
+        <material name="blue"/>
       </visual>
       <collision>
         <origin xyz="0.0 0.0 0.0" rpy="0 0 0"/>
         <geometry>
-          <mesh filename="file://$(find hatch_frame)/meshes/collision/crank_wheel.stl"/>
+          <mesh filename="file://$(find hatch_accessories)/meshes/collision/crank_wheel.stl"/>
         </geometry>
         <material name="red"/>
@@ -54,12 +54,12 @@
         <origin xyz="0.0 0.0 0.00355" rpy="0 0 0"/>
         <geometry>
-          <mesh filename="file://$(find hatch_frame)/meshes/visual/crank_handle.stl"/>
+          <mesh filename="file://$(find hatch_accessories)/meshes/visual/crank_handle.stl"/>
         </geometry>
-        <material name="gray"/>
+        <material name="blue"/>
       </visual>
       <collision>
         <origin xyz="0.0 0.0 0.00355" rpy="0 0 0"/>
         <geometry>
-          <mesh filename="file://$(find hatch_frame)/meshes/collision/crank_handle.stl"/>
+          <mesh filename="file://$(find hatch_accessories)/meshes/collision/crank_handle.stl"/>
         </geometry>
         <material name="red"/>

File: hatch_accessories/urdf/grab_handle.xacro (robot description, xacro)
@@ -22,7 +22,7 @@
         <origin xyz="0.0 0.0 0.0" rpy="0 0 0"/>
         <geometry>
-          <mesh filename="file://$(find hatch_frame)/meshes/visual/grab_handle.stl"/>
+          <mesh filename="file://$(find hatch_accessories)/meshes/visual/grab_handle.stl"/>
         </geometry>
-        <material name="gray"/>
+        <material name="blue"/>
       </visual>
       <collision>
@@ -30,5 +30,5 @@
         <origin xyz="0.0 0.0 0.0" rpy="0 0 0"/>
         <geometry>
-          <mesh filename="file://$(find hatch_frame)/meshes/collision/grab_handle.stl"/>
+          <mesh filename="file://$(find hatch_accessories)/meshes/collision/grab_handle.stl"/>
         </geometry>
         <material name="red"/>

File: hatch_accessories/urdf/hatch_frame.urdf.xacro (robot description, xacro)
@@ -3,6 +3,6 @@
   <xacro:arg name="name" default=""/>
   <xacro:arg name="prefix" default=""/>
-  <xacro:include filename="$(find hatch_frame)/urdf/colors.xacro"/>
-  <xacro:include filename="$(find hatch_frame)/urdf/hatch_frame.xacro"/>
+  <xacro:include filename="$(find hatch_accessories)/urdf/colors.xacro"/>
+  <xacro:include filename="$(find hatch_accessories)/urdf/hatch_frame.xacro"/>
   <link name="world"/>
   <xacro:hatch_frame name="$(arg name)" prefix="$(arg prefix)" parent="world">

File: hatch_accessories/urdf/hatch_frame.xacro (robot description, xacro)
@@ -15,5 +15,5 @@
         <origin xyz="0.0 0.0 0.0" rpy="0 0 0"/>
         <geometry>
-          <mesh filename="file://$(find hatch_frame)/meshes/visual/ivr_hatch_frame.stl"/>
+          <mesh filename="file://$(find hatch_accessories)/meshes/visual/ivr_hatch_frame.stl"/>
         </geometry>
         <material name="gray"/>

Commit message: Updating 4040 hatch to keep joint names consistent between hatches.

File: hatch_4040/urdf/hatch_4040.urdf.xacro (robot description, xacro)
@@ -10,6 +10,6 @@
     <origin xyz="0 0 0" rpy="0 0 0"/>
   </xacro:hatch_frame>
-  <xacro:hatch_4040 name="$(arg name)" prefix="$(arg prefix)" parent="hatch_frame">
+  <xacro:hatch name="$(arg name)" prefix="$(arg prefix)" parent="hatch_frame">
     <origin xyz="0.668 0.06 0.657" rpy="0 0 0"/>
-  </xacro:hatch_4040>
+  </xacro:hatch>
 </robot>

File: hatch_4040/urdf/hatch_4040.xacro (robot description, xacro)
@@ -1,15 +1,15 @@
 <?xml version="1.0"?>
 <robot xmlns:xacro="http://wiki.ros.org/xacro">
-  <xacro:macro name="hatch_4040" params="
+  <xacro:macro name="hatch" params="
     name:=''
     prefix:=''
     parent:=''
     *origin">
-    <joint name="${prefix}hatch_4040_frame_joint" type="fixed">
+    <joint name="${prefix}hatch_outer_frame_joint" type="fixed">
       <parent link="${prefix}${parent}"/>
-      <child link="${prefix}hatch_4040_frame"/>
+      <child link="${prefix}hatch_outer_frame"/>
       <xacro:insert_block name="origin"/>
     </joint>
-    <link name="${prefix}hatch_4040_frame">
+    <link name="${prefix}hatch_outer_frame">
       <!--TODO set proper inertia-->
       <inertial>
@@ -33,12 +33,12 @@
       </collision>
     </link>
-    <joint name="${prefix}hatch_4040_frame_face_joint" type="revolute">
+    <joint name="${prefix}hatch_outer_frame_face_joint" type="revolute">
       <axis xyz="0 0 1"/>
       <limit effort="10.0" lower="0.0" upper="3.14" velocity="0.5"/>
-      <parent link="${prefix}hatch_4040_frame"/>
-      <child link="${prefix}hatch_4040_face"/>
+      <parent link="${prefix}hatch_outer_frame"/>
+      <child link="${prefix}hatch_face"/>
       <origin xyz="0.083 1.215 0.103" rpy="0 0 0"/>
     </joint>
-    <link name="${prefix}hatch_4040_face">
+    <link name="${prefix}hatch_face">
       <!--TODO set proper inertia-->
       <inertial>
@@ -63,5 +63,5 @@
     </link>
     <joint name="${prefix}right_cal_1_joint" type="fixed">
-      <parent link="${prefix}hatch_4040_face"/>
+      <parent link="${prefix}hatch_face"/>
       <child link="${prefix}right_cal_1_frame"/>
       <origin xyz="0.0167 0.0 0.0" rpy="0 0 0"/>
@@ -69,5 +69,5 @@
     <link name="${prefix}right_cal_1_frame"/>
     <joint name="${prefix}right_cal_2_joint" type="fixed">
-      <parent link="${prefix}hatch_4040_face"/>
+      <parent link="${prefix}hatch_face"/>
       <child link="${prefix}right_cal_2_frame"/>
       <origin xyz="0.0 0.0167 0.0" rpy="0 0 0"/>
@@ -75,15 +75,15 @@
     <link name="${prefix}right_cal_2_frame"/>
     <xacro:include filename="$(find hatch_accessories)/urdf/crank_wheel.xacro"/>
-    <xacro:crank_wheel name="$(arg name)" prefix="$(arg prefix)external_" parent="${prefix}hatch_4040_face">
+    <xacro:crank_wheel name="$(arg name)" prefix="$(arg prefix)external_" parent="${prefix}hatch_face">
       <origin xyz="0.04431 -0.475371 0.602" rpy="0 ${pi/2} 0"/>
     </xacro:crank_wheel>
-    <xacro:crank_wheel name="$(arg name)" prefix="$(arg prefix)internal_" parent="${prefix}hatch_4040_face">
+    <xacro:crank_wheel name="$(arg name)" prefix="$(arg prefix)internal_" parent="${prefix}hatch_face">
       <origin xyz="-0.1716 -0.475371 0.602" rpy="0 -${pi/2} 0"/>
     </xacro:crank_wheel>
     <xacro:include filename="$(find hatch_accessories)/urdf/grab_handle.xacro"/>
-    <xacro:grab_handle name="$(arg name)" prefix="$(arg prefix)external_" parent="${prefix}hatch_4040_face">
+    <xacro:grab_handle name="$(arg name)" prefix="$(arg prefix)external_" parent="${prefix}hatch_face">
       <origin xyz="-0.0597 -0.788394 0.3147147" rpy="-0.3926991 0 0"/>
     </xacro:grab_handle>
-    <xacro:grab_handle name="$(arg name)" prefix="$(arg prefix)internal_" parent="${prefix}hatch_4040_face">
+    <xacro:grab_handle name="$(arg name)" prefix="$(arg prefix)internal_" parent="${prefix}hatch_face">
       <origin xyz="-0.0776 -0.851588 0.3093442" rpy="0 ${pi} 0"/>
     </xacro:grab_handle>
