Commit message: Adding the rotary wheels.

File: hatch_4040/urdf/hatch_4040.xacro (robot description, xacro)
@@ -41,4 +41,10 @@
     </joint>
     <link name="${prefix}hatch_4040_face">
+      <!--TODO set proper inertia-->
+      <inertial>
+        <origin rpy="0 0 0" xyz="0.0 0.0 0.0"/>
+        <mass value="0.0"/>
+        <inertia ixx="0.0" ixy="0.0" ixz="0.0" iyy="0.0" iyz="0.0" izz="0.0"/>
+      </inertial>
       <visual>
         <origin xyz="0.0 0.0 0.0" rpy="0 0 0"/>
@@ -56,4 +62,12 @@
       </collision>
     </link>
+    <xacro:include filename="$(find trainer)/urdf/crank_wheel.xacro"/>
+    <xacro:crank_wheel name="$(arg name)" prefix="$(arg prefix)external_" parent="${prefix}hatch_4040_face">
+      <origin xyz="0.0522475 -0.473371 0.606772" rpy="0 ${pi/2} 0"/>
+    </xacro:crank_wheel>
+    <xacro:include filename="$(find trainer)/urdf/crank_wheel.xacro"/>
+    <xacro:crank_wheel name="$(arg name)" prefix="$(arg prefix)internal_" parent="${prefix}hatch_4040_face">
+      <origin xyz="-0.1795475 -0.473371 0.606772" rpy="0 -${pi/2} 0"/>
+    </xacro:crank_wheel>
   </xacro:macro>
 </robot>

File: trainer/urdf/trainer_frame.xacro (robot description, xacro)
@@ -13,5 +13,6 @@
     <link name="${prefix}trainer_frame">
       <visual>
-        <origin xyz="0.0 0.0 0.0" rpy="0 0 0"/>
+        <!--Offset is to adjust for the radius on the extrusion-->
+        <origin xyz="0.0 0.004 0.0" rpy="0 0 0"/>
         <geometry>
           <mesh filename="file://$(find trainer)/meshes/visual/ivr_tasktrainer_frame.stl"/>

Commit message: Adding the grab handles but still need updated stl with the proper origin.

File: hatch_4040/urdf/hatch_4040.xacro (robot description, xacro)
@@ -62,12 +62,18 @@
       </collision>
     </link>
-    <xacro:include filename="$(find trainer)/urdf/crank_wheel.xacro"/>
+    <xacro:include filename="$(find hatch_4040)/urdf/crank_wheel.xacro"/>
     <xacro:crank_wheel name="$(arg name)" prefix="$(arg prefix)external_" parent="${prefix}hatch_4040_face">
       <origin xyz="0.0522475 -0.473371 0.606772" rpy="0 ${pi/2} 0"/>
     </xacro:crank_wheel>
-    <xacro:include filename="$(find trainer)/urdf/crank_wheel.xacro"/>
     <xacro:crank_wheel name="$(arg name)" prefix="$(arg prefix)internal_" parent="${prefix}hatch_4040_face">
       <origin xyz="-0.1795475 -0.473371 0.606772" rpy="0 -${pi/2} 0"/>
     </xacro:crank_wheel>
+    <xacro:include filename="$(find hatch_4040)/urdf/grab_handle.xacro"/>
+    <xacro:grab_handle name="$(arg name)" prefix="$(arg prefix)external_" parent="${prefix}hatch_4040_face">
+      <origin xyz="-0.0497 -0.788394 0.3147147" rpy="0 0 0"/>
+    </xacro:grab_handle>
+    <xacro:grab_handle name="$(arg name)" prefix="$(arg prefix)internal_" parent="${prefix}hatch_4040_face">
+      <origin xyz="-0.0776 -0.851588 0.3093442" rpy="0 ${pi} 0"/>
+    </xacro:grab_handle>
   </xacro:macro>
 </robot>

Commit message: Adding a better mesh for collision checking.

File: hatch_4040/urdf/hatch_4040.xacro (robot description, xacro)
@@ -57,5 +57,5 @@
         <origin xyz="0.0 0.0 0.0" rpy="0 0 0"/>
         <geometry>
-          <mesh filename="file://$(find hatch_4040)/meshes/collision/hatch_4040_face.stl"/>
+          <mesh filename="file://$(find hatch_4040)/meshes/collision/hatch_4040_collision.stl"/>
         </geometry>
         <material name="red"/>

Commit message: updating angle of grab handle to 22.5 degrees

File: hatch_4040/urdf/hatch_4040.xacro (robot description, xacro)
@@ -71,5 +71,5 @@
     <xacro:include filename="$(find hatch_4040)/urdf/grab_handle.xacro"/>
     <xacro:grab_handle name="$(arg name)" prefix="$(arg prefix)external_" parent="${prefix}hatch_4040_face">
-      <origin xyz="-0.0497 -0.788394 0.3147147" rpy="-0.436332 0 0"/>
+      <origin xyz="-0.0497 -0.788394 0.3147147" rpy="-0.3926991 0 0"/>
     </xacro:grab_handle>
     <xacro:grab_handle name="$(arg name)" prefix="$(arg prefix)internal_" parent="${prefix}hatch_4040_face">

Commit message: Changing the crank wheel and cleaning up some files.

File: hatch_4040/urdf/hatch_4040.xacro (robot description, xacro)
@@ -64,8 +64,8 @@
     <xacro:include filename="$(find hatch_frame)/urdf/crank_wheel.xacro"/>
     <xacro:crank_wheel name="$(arg name)" prefix="$(arg prefix)external_" parent="${prefix}hatch_4040_face">
-      <origin xyz="0.0522475 -0.473371 0.604" rpy="0 ${pi/2} 0"/>
+      <origin xyz="0.04431 -0.473371 0.604" rpy="0 ${pi/2} 0"/>
     </xacro:crank_wheel>
     <xacro:crank_wheel name="$(arg name)" prefix="$(arg prefix)internal_" parent="${prefix}hatch_4040_face">
-      <origin xyz="-0.1795475 -0.473371 0.604" rpy="0 -${pi/2} 0"/>
+      <origin xyz="-0.1716 -0.473371 0.604" rpy="0 -${pi/2} 0"/>
     </xacro:crank_wheel>
     <xacro:include filename="$(find hatch_frame)/urdf/grab_handle.xacro"/>

File: hatch_frame/urdf/crank_wheel.xacro (robot description, xacro)
@@ -24,5 +24,5 @@
         <origin xyz="0.0 0.0 0.0" rpy="0 0 0"/>
         <geometry>
-          <mesh filename="file://$(find hatch_4040)/meshes/visual/crank_wheel.stl"/>
+          <mesh filename="file://$(find hatch_frame)/meshes/visual/crank_wheel.stl"/>
         </geometry>
         <material name="gray"/>
@@ -31,5 +31,5 @@
         <origin xyz="0.0 0.0 0.0" rpy="0 0 0"/>
         <geometry>
-          <mesh filename="file://$(find hatch_4040)/meshes/collision/crank_wheel.stl"/>
+          <mesh filename="file://$(find hatch_frame)/meshes/collision/crank_wheel.stl"/>
         </geometry>
         <material name="red"/>
@@ -42,5 +42,5 @@
       <parent link="${prefix}rotary_wheel"/>
       <child link="${prefix}rotary_handle"/>
-      <origin xyz="0.053975 0.0 0.0155" rpy="0 0 0"/>
+      <origin xyz="0.0 0.053975 0.0155" rpy="0 0 0"/>
     </joint>
     <link name="${prefix}rotary_handle">
@@ -54,5 +54,5 @@
         <origin xyz="0.0 0.0 0.00355" rpy="0 0 0"/>
         <geometry>
-          <mesh filename="file://$(find hatch_4040)/meshes/visual/crank_handle.stl"/>
+          <mesh filename="file://$(find hatch_frame)/meshes/visual/crank_handle.stl"/>
         </geometry>
         <material name="gray"/>
@@ -61,5 +61,5 @@
         <origin xyz="0.0 0.0 0.00355" rpy="0 0 0"/>
         <geometry>
-          <mesh filename="file://$(find hatch_4040)/meshes/collision/crank_handle.stl"/>
+          <mesh filename="file://$(find hatch_frame)/meshes/collision/crank_handle.stl"/>
         </geometry>
         <material name="red"/>

File: hatch_frame/urdf/grab_handle.xacro (robot description, xacro)
@@ -22,5 +22,5 @@
         <origin xyz="0.0 0.0 0.0" rpy="0 0 0"/>
         <geometry>
-          <mesh filename="file://$(find hatch_4040)/meshes/visual/grab_handle.stl"/>
+          <mesh filename="file://$(find hatch_frame)/meshes/visual/grab_handle.stl"/>
         </geometry>
         <material name="gray"/>
@@ -30,5 +30,5 @@
         <origin xyz="0.0 0.0 0.0" rpy="0 0 0"/>
         <geometry>
-          <mesh filename="file://$(find hatch_4040)/meshes/collision/grab_handle.stl"/>
+          <mesh filename="file://$(find hatch_frame)/meshes/collision/grab_handle.stl"/>
         </geometry>
         <material name="red"/>
