Commit message: switched file to package

File: hatch_4040/urdf/hatch_4040.xacro (robot description, xacro)
@@ -21,5 +21,5 @@
         <origin xyz="0.0 0.0 0.0" rpy="0 0 0"/>
         <geometry>
-          <mesh filename="file://$(find hatch_4040)/meshes/visual/hatch_4040_frame.stl"/>
+          <mesh filename="package://hatch_4040/meshes/visual/hatch_4040_frame.stl"/>
         </geometry>
         <material name="gray"/>
@@ -28,5 +28,5 @@
         <origin xyz="0.0 0.0 0.0" rpy="0 0 0"/>
         <geometry>
-          <mesh filename="file://$(find hatch_4040)/meshes/collision/hatch_4040_frame_no_latches.stl"/>
+          <mesh filename="package://hatch_4040/meshes/collision/hatch_4040_frame_no_latches.stl"/>
         </geometry>
         <material name="red"/>
@@ -50,5 +50,5 @@
         <origin xyz="0.0 0.0 0.0" rpy="0 0 0"/>
         <geometry>
-          <mesh filename="file://$(find hatch_4040)/meshes/visual/hatch_4040_face.stl"/>
+          <mesh filename="package://hatch_4040/meshes/visual/hatch_4040_face.stl"/>
         </geometry>
         <material name="gray"/>
@@ -57,5 +57,5 @@
         <origin xyz="0.0 0.0 0.0" rpy="0 0 0"/>
         <geometry>
-          <mesh filename="file://$(find hatch_4040)/meshes/collision/hatch_4040_collision.stl"/>
+          <mesh filename="package://hatch_4040/meshes/collision/hatch_4040_collision.stl"/>
         </geometry>
         <material name="red"/>

File: hatch_4060/urdf/hatch_4060.xacro (robot description, xacro)
@@ -25,5 +25,5 @@
         <origin xyz="0.0 0.0 0.0" rpy="0 0 0"/>
         <geometry>
-          <mesh filename="file://$(find hatch_4060)/meshes/visual/hatch_4060_frame.stl"/>
+          <mesh filename="package://hatch_4060/meshes/visual/hatch_4060_frame.stl"/>
         </geometry>
         <material name="gray"/>
@@ -32,5 +32,5 @@
         <origin xyz="0.0 0.0 0.0" rpy="0 0 0"/>
         <geometry>
-          <mesh filename="file://$(find hatch_4060)/meshes/collision/hatch_4060_frame.stl"/>
+          <mesh filename="package://hatch_4060/meshes/collision/hatch_4060_frame.stl"/>
         </geometry>
         <material name="red"/>
@@ -55,5 +55,5 @@
         <origin xyz="0.0 0.0 0.0" rpy="0 0 0"/>
         <geometry>
-          <mesh filename="file://$(find hatch_4060)/meshes/visual/hatch_4060_face.stl"/>
+          <mesh filename="package://hatch_4060/meshes/visual/hatch_4060_face.stl"/>
         </geometry>
         <material name="gray"/>
@@ -62,5 +62,5 @@
         <origin xyz="0.0 0.0 0.0" rpy="0 0 0"/>
         <geometry>
-          <mesh filename="file://$(find hatch_4060)/meshes/collision/hatch_4060_collision.stl"/>
+          <mesh filename="package://hatch_4060/meshes/collision/hatch_4060_collision.stl"/>
         </geometry>
         <material name="red"/>

File: hatch_accessories/urdf/crank_wheel.xacro (robot description, xacro)
@@ -24,5 +24,5 @@
         <origin xyz="0.0 0.0 0.0" rpy="0 0 0"/>
         <geometry>
-          <mesh filename="file://$(find hatch_accessories)/meshes/visual/crank_wheel.stl"/>
+          <mesh filename="package://hatch_accessories/meshes/visual/crank_wheel.stl"/>
         </geometry>
         <material name="blue"/>
@@ -31,5 +31,5 @@
         <origin xyz="0.0 0.0 0.0" rpy="0 0 0"/>
         <geometry>
-          <mesh filename="file://$(find hatch_accessories)/meshes/collision/crank_wheel.stl"/>
+          <mesh filename="package://hatch_accessories/meshes/collision/crank_wheel.stl"/>
         </geometry>
         <material name="red"/>
@@ -54,5 +54,5 @@
         <origin xyz="0.0 0.0 0.00355" rpy="0 0 0"/>
         <geometry>
-          <mesh filename="file://$(find hatch_accessories)/meshes/visual/crank_handle.stl"/>
+          <mesh filename="package://hatch_accessories/meshes/visual/crank_handle.stl"/>
         </geometry>
         <material name="blue"/>
@@ -61,5 +61,5 @@
         <origin xyz="0.0 0.0 0.00355" rpy="0 0 0"/>
         <geometry>
-          <mesh filename="file://$(find hatch_accessories)/meshes/collision/crank_handle.stl"/>
+          <mesh filename="package://hatch_accessories/meshes/collision/crank_handle.stl"/>
         </geometry>
         <material name="red"/>

File: hatch_accessories/urdf/grab_handle.xacro (robot description, xacro)
@@ -22,5 +22,5 @@
         <origin xyz="0.0 0.0 0.0" rpy="0 0 0"/>
         <geometry>
-          <mesh filename="file://$(find hatch_accessories)/meshes/visual/grab_handle.stl"/>
+          <mesh filename="package://hatch_accessories/meshes/visual/grab_handle.stl"/>
         </geometry>
         <material name="blue"/>
@@ -30,5 +30,5 @@
         <origin xyz="0.0 0.0 0.0" rpy="0 0 0"/>
         <geometry>
-          <mesh filename="file://$(find hatch_accessories)/meshes/collision/grab_handle.stl"/>
+          <mesh filename="package://hatch_accessories/meshes/collision/grab_handle.stl"/>
         </geometry>
         <material name="red"/>

File: hatch_accessories/urdf/hatch_frame.xacro (robot description, xacro)
@@ -15,5 +15,5 @@
         <origin xyz="0.0 0.0 0.0" rpy="0 0 0"/>
         <geometry>
-          <mesh filename="file://$(find hatch_accessories)/meshes/visual/ivr_hatch_frame.stl"/>
+          <mesh filename="package://hatch_accessories/meshes/visual/ivr_hatch_frame.stl"/>
         </geometry>
         <material name="gray"/>

File: trainer/urdf/trainer_frame.xacro (robot description, xacro)
@@ -16,5 +16,5 @@
         <origin xyz="0.0 0.004 0.0" rpy="0 0 0"/>
         <geometry>
-          <mesh filename="file://$(find trainer)/meshes/visual/ivr_tasktrainer_frame.stl"/>
+          <mesh filename="package://trainer/meshes/visual/ivr_tasktrainer_frame.stl"/>
         </geometry>
         <material name="gray"/>

File: trainer/urdf/trainer_front_left_face.xacro (robot description, xacro)
@@ -22,5 +22,5 @@
       <origin xyz="0.0 0.0 0.0" rpy="0 0 0"/>
       <geometry>
-        <mesh filename="file://$(find trainer)/meshes/visual/front_left_face.stl"/>
+        <mesh filename="package://trainer/meshes/visual/front_left_face.stl"/>
       </geometry>
       <material name="gray"/>
@@ -29,5 +29,5 @@
       <origin xyz="0.0 0.0 0.0" rpy="0 0 0"/>
       <geometry>
-        <mesh filename="file://$(find trainer)/meshes/collision/front_left_face.stl"/>
+        <mesh filename="package://trainer/meshes/collision/front_left_face.stl"/>
       </geometry>
       <material name="red"/>
@@ -49,5 +49,5 @@
       <origin xyz="0.0 0.0 0.0" rpy="0 0 0"/>
       <geometry>
-        <mesh filename="file://$(find trainer)/meshes/visual/cubby_1.stl"/>
+        <mesh filename="package://trainer/meshes/visual/cubby_1.stl"/>
       </geometry>
       <material name="gray"/>
@@ -56,5 +56,5 @@
       <origin xyz="0.0 0.0 0.0" rpy="0 0 0"/>
       <geometry>
-        <mesh filename="file://$(find trainer)/meshes/collision/cubby_1.stl"/>
+        <mesh filename="package://trainer/meshes/collision/cubby_1.stl"/>
       </geometry>
       <material name="red"/>
@@ -76,5 +76,5 @@
       <origin xyz="0.0 0.0 0.0" rpy="0 0 0"/>
       <geometry>
-        <mesh filename="file://$(find trainer)/meshes/visual/cubby_2.stl"/>
+        <mesh filename="package://trainer/meshes/visual/cubby_2.stl"/>
       </geometry>
       <material name="gray"/>
@@ -83,5 +83,5 @@
       <origin xyz="0.0 0.0 0.0" rpy="0 0 0"/>
       <geometry>
-        <mesh filename="file://$(find trainer)/meshes/collision/cubby_2.stl"/>
+        <mesh filename="package://trainer/meshes/collision/cubby_2.stl"/>
       </geometry>
       <material name="red"/>

File: trainer/urdf/trainer_front_right_face.xacro (robot description, xacro)
@@ -21,5 +21,5 @@
       <origin xyz="0.0 0.0 0.0" rpy="0 0 0"/>
       <geometry>
-        <mesh filename="file://$(find trainer)/meshes/visual/front_right_face.stl"/>
+        <mesh filename="package://trainer/meshes/visual/front_right_face.stl"/>
       </geometry>
       <material name="gray"/>
@@ -28,5 +28,5 @@
       <origin xyz="0.0 0.0 0.0" rpy="0 0 0"/>
       <geometry>
-        <mesh filename="file://$(find trainer)/meshes/collision/front_right_face.stl"/>
+        <mesh filename="package://trainer/meshes/collision/front_right_face.stl"/>
       </geometry>
       <material name="red"/>
@@ -50,12 +50,12 @@
       <origin xyz="${-0.0075 - 0.003175} -0.00366 0.0" rpy="0 0 0"/>
       <geometry>
-        <mesh filename="file://$(find trainer)/meshes/visual/cabinet_door_1.stl"/>
-      </geometry>
-      <material name="blue"/>
-    </visual>
-    <collision>
-      <origin xyz="${-0.0075 - 0.003175} -0.00366 0.0" rpy="0 0 0"/>
-      <geometry>
-        <mesh filename="file://$(find trainer)/meshes/collision/cabinet_door_1.stl"/>
+        <mesh filename="package://trainer/meshes/visual/cabinet_door_1.stl"/>
+      </geometry>
+      <material name="blue"/>
+    </visual>
+    <collision>
+      <origin xyz="${-0.0075 - 0.003175} -0.00366 0.0" rpy="0 0 0"/>
+      <geometry>
+        <mesh filename="package://trainer/meshes/collision/cabinet_door_1.stl"/>
       </geometry>
       <material name="red"/>
@@ -77,5 +77,5 @@
       <origin xyz="0.0 0.0 0.0" rpy="0 0 0"/>
       <geometry>
-        <mesh filename="file://$(find trainer)/meshes/visual/round_latch_housing.stl"/>
+        <mesh filename="package://trainer/meshes/visual/round_latch_housing.stl"/>
       </geometry>
       <material name="gray"/>
@@ -84,5 +84,5 @@
       <origin xyz="0.0 0.0 0.0" rpy="0 0 0"/>
       <geometry>
-        <mesh filename="file://$(find trainer)/meshes/collision/round_latch_housing.stl"/>
+        <mesh filename="package://trainer/meshes/collision/round_latch_housing.stl"/>
       </geometry>
       <material name="red"/>
@@ -106,12 +106,12 @@
       <origin xyz="0.0 0.0 0.0" rpy="0 0 0"/>
       <geometry>
-        <mesh filename="file://$(find trainer)/meshes/visual/round_latch_handle.stl"/>
-      </geometry>
-      <material name="blue"/>
-    </visual>
-    <collision>
-      <origin xyz="0.0 0.0 0.0" rpy="0 0 0"/>
-      <geometry>
-        <mesh filename="file://$(find trainer)/meshes/collision/round_latch_handle.stl"/>
+        <mesh filename="package://trainer/meshes/visual/round_latch_handle.stl"/>
+      </geometry>
+      <material name="blue"/>
+    </visual>
+    <collision>
+      <origin xyz="0.0 0.0 0.0" rpy="0 0 0"/>
+      <geometry>
+        <mesh filename="package://trainer/meshes/collision/round_latch_handle.stl"/>
       </geometry>
       <material name="red"/>
@@ -135,5 +135,5 @@
       <origin xyz="${-0.0075 - 0.003175} 0.00366 0.0" rpy="0 0 0"/>
       <geometry>
-        <mesh filename="file://$(find trainer)/meshes/visual/cabinet_door_2.stl"/>
+        <mesh filename="package://trainer/meshes/visual/cabinet_door_2.stl"/>
       </geometry>
       <material name="blue"/>
@@ -142,5 +142,5 @@
       <origin xyz="${-0.0075 - 0.003175} 0.00366 0.0" rpy="0 0 0"/>
       <geometry>
-        <mesh filename="file://$(find trainer)/meshes/collision/cabinet_door_2.stl"/>
+        <mesh filename="package://trainer/meshes/collision/cabinet_door_2.stl"/>
       </geometry>
       <material name="red"/>
@@ -162,5 +162,5 @@
       <origin xyz="0.0 0.0 0.0" rpy="0 0 0"/>
       <geometry>
-        <mesh filename="file://$(find trainer)/meshes/visual/push_latch_housing.stl"/>
+        <mesh filename="package://trainer/meshes/visual/push_latch_housing.stl"/>
       </geometry>
       <material name="gray"/>
@@ -169,5 +169,5 @@
       <origin xyz="0.0 0.0 0.0" rpy="0 0 0"/>
       <geometry>
-        <mesh filename="file://$(find trainer)/meshes/collision/push_latch_housing.stl"/>
+        <mesh filename="package://trainer/meshes/collision/push_latch_housing.stl"/>
       </geometry>
       <material name="red"/>
@@ -192,12 +192,12 @@
       <origin xyz="0.0 0.0 0.0" rpy="0 0 0"/>
       <geometry>
-        <mesh filename="file://$(find trainer)/meshes/visual/push_latch_button.stl"/>
-      </geometry>
-      <material name="blue"/>
-    </visual>
-    <collision>
-      <origin xyz="0.0 0.0 0.0" rpy="0 0 0"/>
-      <geometry>
-        <mesh filename="file://$(find trainer)/meshes/collision/push_latch_button.stl"/>
+        <mesh filename="package://trainer/meshes/visual/push_latch_button.stl"/>
+      </geometry>
+      <material name="blue"/>
+    </visual>
+    <collision>
+      <origin xyz="0.0 0.0 0.0" rpy="0 0 0"/>
+      <geometry>
+        <mesh filename="package://trainer/meshes/collision/push_latch_button.stl"/>
       </geometry>
       <material name="red"/>
@@ -221,12 +221,12 @@
       <origin xyz="0.0 0.0 0.0" rpy="0 0 0"/>
       <geometry>
-        <mesh filename="file://$(find trainer)/meshes/visual/push_latch_handle.stl"/>
-      </geometry>
-      <material name="blue"/>
-    </visual>
-    <collision>
-      <origin xyz="0.0 0.0 0.0" rpy="0 0 0"/>
-      <geometry>
-        <mesh filename="file://$(find trainer)/meshes/collision/push_latch_handle.stl"/>
+        <mesh filename="package://trainer/meshes/visual/push_latch_handle.stl"/>
+      </geometry>
+      <material name="blue"/>
+    </visual>
+    <collision>
+      <origin xyz="0.0 0.0 0.0" rpy="0 0 0"/>
+      <geometry>
+        <mesh filename="package://trainer/meshes/collision/push_latch_handle.stl"/>
       </geometry>
       <material name="red"/>
@@ -250,12 +250,12 @@
       <origin xyz="${-0.0075 - 0.003175} -0.00366 0.0" rpy="0 0 0"/>
       <geometry>
-        <mesh filename="file://$(find trainer)/meshes/visual/cabinet_door_3.stl"/>
-      </geometry>
-      <material name="blue"/>
-    </visual>
-    <collision>
-      <origin xyz="${-0.0075 - 0.003175} -0.00366 0.0" rpy="0 0 0"/>
-      <geometry>
-        <mesh filename="file://$(find trainer)/meshes/collision/cabinet_door_3.stl"/>
+        <mesh filename="package://trainer/meshes/visual/cabinet_door_3.stl"/>
+      </geometry>
+      <material name="blue"/>
+    </visual>
+    <collision>
+      <origin xyz="${-0.0075 - 0.003175} -0.00366 0.0" rpy="0 0 0"/>
+      <geometry>
+        <mesh filename="package://trainer/meshes/collision/cabinet_door_3.stl"/>
       </geometry>
       <material name="red"/>

File: trainer/urdf/trainer_side.xacro (robot description, xacro)
@@ -21,5 +21,5 @@
         <origin xyz="0.0 0.0 0.0" rpy="0 0 0"/>
         <geometry>
-          <mesh filename="file://$(find trainer)/meshes/visual/side_bottom_face.stl"/>
+          <mesh filename="package://trainer/meshes/visual/side_bottom_face.stl"/>
         </geometry>
         <material name="gray"/>
@@ -28,5 +28,5 @@
         <origin xyz="0.0 0.0 0.0" rpy="0 0 0"/>
           <geometry>
-            <mesh filename="file://$(find trainer)/meshes/collision/side_bottom_face.stl"/>
+            <mesh filename="package://trainer/meshes/collision/side_bottom_face.stl"/>
           </geometry>
         <material name="red"/>
@@ -48,5 +48,5 @@
         <origin xyz="0.0 0.0 0.0" rpy="0 0 0"/>
         <geometry>
-          <mesh filename="file://$(find trainer)/meshes/visual/side_top_face.stl"/>
+          <mesh filename="package://trainer/meshes/visual/side_top_face.stl"/>
         </geometry>
         <material name="gray"/>
@@ -55,5 +55,5 @@
         <origin xyz="0.0 0.0 0.0" rpy="0 0 0"/>
           <geometry>
-            <mesh filename="file://$(find trainer)/meshes/collision/side_top_face.stl"/>
+            <mesh filename="package://trainer/meshes/collision/side_top_face.stl"/>
           </geometry>
         <material name="red"/>
@@ -77,5 +77,5 @@
       <origin xyz="0.00305 -0.0106 0.0" rpy="0 0 0"/>
       <geometry>
-        <mesh filename="file://$(find trainer)/meshes/visual/cabinet_door_4.stl"/>
+        <mesh filename="package://trainer/meshes/visual/cabinet_door_4.stl"/>
       </geometry>
       <material name="blue"/>
@@ -84,5 +84,5 @@
       <origin xyz="0.00305 -0.0106 0.0" rpy="0 0 0"/>
       <geometry>
-        <mesh filename="file://$(find trainer)/meshes/collision/cabinet_door_4.stl"/>
+        <mesh filename="package://trainer/meshes/collision/cabinet_door_4.stl"/>
       </geometry>
       <material name="red"/>
@@ -104,5 +104,5 @@
       <origin xyz="0.00305 0.0 0.00305" rpy="0 0 0"/>
       <geometry>
-        <mesh filename="file://$(find trainer)/meshes/visual/paddle_latch_housing.stl"/>
+        <mesh filename="package://trainer/meshes/visual/paddle_latch_housing.stl"/>
       </geometry>
       <material name="gray"/>
@@ -111,5 +111,5 @@
       <origin xyz="0.00305 0.0 0.00305" rpy="0 0 0"/>
       <geometry>
-        <mesh filename="file://$(find trainer)/meshes/collision/paddle_latch_housing.stl"/>
+        <mesh filename="package://trainer/meshes/collision/paddle_latch_housing.stl"/>
       </geometry>
       <material name="red"/>
@@ -133,12 +133,12 @@
       <origin xyz="0.0 0.0 0.0" rpy="0 0 0"/>
       <geometry>
-        <mesh filename="file://$(find trainer)/meshes/visual/paddle_latch_handle.stl"/>
-      </geometry>
-      <material name="blue"/>
-    </visual>
-    <collision>
-      <origin xyz="0.0 0.0 0.0" rpy="0 0 0"/>
-      <geometry>
-        <mesh filename="file://$(find trainer)/meshes/collision/paddle_latch_handle.stl"/>
+        <mesh filename="package://trainer/meshes/visual/paddle_latch_handle.stl"/>
+      </geometry>
+      <material name="blue"/>
+    </visual>
+    <collision>
+      <origin xyz="0.0 0.0 0.0" rpy="0 0 0"/>
+      <geometry>
+        <mesh filename="package://trainer/meshes/collision/paddle_latch_handle.stl"/>
       </geometry>
       <material name="red"/>
@@ -162,12 +162,12 @@
       <origin xyz="0.0 0.0 0.0" rpy="0 0 0"/>
       <geometry>
-        <mesh filename="file://$(find trainer)/meshes/visual/drawer_1_face.stl"/>
-      </geometry>
-      <material name="blue"/>
-    </visual>
-    <collision>
-      <origin xyz="0.0 0.0 0.0" rpy="0 0 0"/>
-      <geometry>
-        <mesh filename="file://$(find trainer)/meshes/collision/drawer_1_face.stl"/>
+        <mesh filename="package://trainer/meshes/visual/drawer_1_face.stl"/>
+      </geometry>
+      <material name="blue"/>
+    </visual>
+    <collision>
+      <origin xyz="0.0 0.0 0.0" rpy="0 0 0"/>
+      <geometry>
+        <mesh filename="package://trainer/meshes/collision/drawer_1_face.stl"/>
       </geometry>
       <material name="red"/>
@@ -272,12 +272,12 @@
       <origin xyz="0.0 0.0 0.0" rpy="0 0 0"/>
       <geometry>
-        <mesh filename="file://$(find trainer)/meshes/visual/drawer_2_face.stl"/>
-      </geometry>
-      <material name="blue"/>
-    </visual>
-    <collision>
-      <origin xyz="0.0 0.0 0.0" rpy="0 0 0"/>
-      <geometry>
-        <mesh filename="file://$(find trainer)/meshes/collision/drawer_2_face.stl"/>
+        <mesh filename="package://trainer/meshes/visual/drawer_2_face.stl"/>
+      </geometry>
+      <material name="blue"/>
+    </visual>
+    <collision>
+      <origin xyz="0.0 0.0 0.0" rpy="0 0 0"/>
+      <geometry>
+        <mesh filename="package://trainer/meshes/collision/drawer_2_face.stl"/>
       </geometry>
       <material name="red"/>
@@ -299,5 +299,5 @@
       <origin xyz="0.0 0.0 0.0" rpy="0 0 0"/>
       <geometry>
-        <mesh filename="file://$(find trainer)/meshes/visual/recessed_latch_housing.stl"/>
+        <mesh filename="package://trainer/meshes/visual/recessed_latch_housing.stl"/>
       </geometry>
       <material name="gray"/>
@@ -306,5 +306,5 @@
       <origin xyz="0.0 0.0 0.0" rpy="0 0 0"/>
       <geometry>
-        <mesh filename="file://$(find trainer)/meshes/collision/recessed_latch_housing.stl"/>
+        <mesh filename="package://trainer/meshes/collision/recessed_latch_housing.stl"/>
       </geometry>
       <material name="red"/>
@@ -328,12 +328,12 @@
       <origin xyz="0.0 0.0 0.0" rpy="0 0 0"/>
       <geometry>
-        <mesh filename="file://$(find trainer)/meshes/visual/recessed_latch_handle.stl"/>
-      </geometry>
-      <material name="blue"/>
-    </visual>
-    <collision>
-      <origin xyz="0.0 0.0 0.0" rpy="0 0 0"/>
-      <geometry>
-        <mesh filename="file://$(find trainer)/meshes/collision/recessed_latch_handle.stl"/>
+        <mesh filename="package://trainer/meshes/visual/recessed_latch_handle.stl"/>
+      </geometry>
+      <material name="blue"/>
+    </visual>
+    <collision>
+      <origin xyz="0.0 0.0 0.0" rpy="0 0 0"/>
+      <geometry>
+        <mesh filename="package://trainer/meshes/collision/recessed_latch_handle.stl"/>
       </geometry>
       <material name="red"/>

Commit message: Adding calibration frames on the hatch axis.

File: hatch_4040/urdf/hatch_4040.xacro (robot description, xacro)
@@ -62,4 +62,16 @@
       </collision>
     </link>
+    <joint name="${prefix}right_cal_1_joint" type="fixed">
+      <parent link="${prefix}hatch_4040_face"/>
+      <child link="${prefix}right_cal_1_frame"/>
+      <origin xyz="0.0167 0.0 0.0" rpy="0 0 0"/>
+    </joint>
+    <link name="${prefix}right_cal_1_frame"/>
+    <joint name="${prefix}right_cal_2_joint" type="fixed">
+      <parent link="${prefix}hatch_4040_face"/>
+      <child link="${prefix}right_cal_2_frame"/>
+      <origin xyz="0.0 0.0167 0.0" rpy="0 0 0"/>
+    </joint>
+    <link name="${prefix}right_cal_2_frame"/>
     <xacro:include filename="$(find hatch_accessories)/urdf/crank_wheel.xacro"/>
     <xacro:crank_wheel name="$(arg name)" prefix="$(arg prefix)external_" parent="${prefix}hatch_4040_face">

File: hatch_4060/urdf/hatch_4060.xacro (robot description, xacro)
@@ -67,4 +67,16 @@
       </collision>
     </link>
+    <joint name="${prefix}right_cal_1_joint" type="fixed">
+      <parent link="${prefix}hatch_4060_face"/>
+      <child link="${prefix}right_cal_1_frame"/>
+      <origin xyz="0.0167 0.0 0.0" rpy="0 0 0"/>
+    </joint>
+    <link name="${prefix}right_cal_1_frame"/>
+    <joint name="${prefix}right_cal_2_joint" type="fixed">
+      <parent link="${prefix}hatch_4060_face"/>
+      <child link="${prefix}right_cal_2_frame"/>
+      <origin xyz="0.0 0.0167 0.0" rpy="0 0 0"/>
+    </joint>
+    <link name="${prefix}right_cal_2_frame"/>
     <xacro:include filename="$(find hatch_accessories)/urdf/crank_wheel.xacro"/>
     <!--TODO are the centers located properly?-->
