Commit message: finishing calibration for the 4040 hatch

File: hatch_4040/urdf/hatch_4040.xacro (robot description, xacro)
@@ -76,12 +76,12 @@
     <xacro:include filename="$(find hatch_accessories)/urdf/crank_wheel.xacro"/>
     <xacro:crank_wheel name="$(arg name)" prefix="$(arg prefix)external_" parent="${prefix}hatch_4040_face">
-      <origin xyz="0.04431 -0.473371 0.604" rpy="0 ${pi/2} 0"/>
+      <origin xyz="0.04431 -0.475371 0.602" rpy="0 ${pi/2} 0"/>
     </xacro:crank_wheel>
     <xacro:crank_wheel name="$(arg name)" prefix="$(arg prefix)internal_" parent="${prefix}hatch_4040_face">
-      <origin xyz="-0.1716 -0.473371 0.604" rpy="0 -${pi/2} 0"/>
+      <origin xyz="-0.1716 -0.475371 0.602" rpy="0 -${pi/2} 0"/>
     </xacro:crank_wheel>
     <xacro:include filename="$(find hatch_accessories)/urdf/grab_handle.xacro"/>
     <xacro:grab_handle name="$(arg name)" prefix="$(arg prefix)external_" parent="${prefix}hatch_4040_face">
-      <origin xyz="-0.0497 -0.788394 0.3147147" rpy="-0.3926991 0 0"/>
+      <origin xyz="-0.0597 -0.788394 0.3147147" rpy="-0.3926991 0 0"/>
     </xacro:grab_handle>
     <xacro:grab_handle name="$(arg name)" prefix="$(arg prefix)internal_" parent="${prefix}hatch_4040_face">

Commit message: Changing the hatch maximum angles to 95 degrees.

File: hatch_4040/urdf/hatch_4040.xacro (robot description, xacro)
@@ -35,5 +35,5 @@
     <joint name="${prefix}hatch_4040_frame_face_joint" type="revolute">
       <axis xyz="0 0 1"/>
-      <limit effort="10.0" lower="0.0" upper="3.14" velocity="0.5"/>
+      <limit effort="10.0" lower="0.0" upper="1.65806" velocity="0.5"/> <!-- 95 degrees -->
       <parent link="${prefix}hatch_4040_frame"/>
       <child link="${prefix}hatch_4040_face"/>

File: hatch_4060/urdf/hatch_4060.xacro (robot description, xacro)
@@ -39,5 +39,5 @@
     <joint name="${prefix}hatch_4060_frame_face_joint" type="revolute">
       <axis xyz="0 0 1"/>
-      <limit effort="10.0" lower="0.0" upper="3.14" velocity="0.5"/>
+      <limit effort="10.0" lower="0.0" upper="1.65806" velocity="0.5"/> <!-- 95 degrees -->
       <parent link="${prefix}hatch_4060_frame"/>
       <child link="${prefix}hatch_4060_face"/>

Commit message: Switching internal/external to reflect a real system.

File: hatch_4040/urdf/hatch_4040.xacro (robot description, xacro)
@@ -76,15 +76,15 @@
     <xacro:include filename="$(find hatch_accessories)/urdf/crank_wheel.xacro"/>
     <xacro:crank_wheel name="$(arg name)" prefix="$(arg prefix)external_" parent="${prefix}hatch_face">
-      <origin xyz="0.04431 -0.475371 0.602" rpy="0 ${pi/2} 0"/>
+      <origin xyz="-0.1716 -0.475371 0.602" rpy="0 -${pi/2} 0"/>
     </xacro:crank_wheel>
     <xacro:crank_wheel name="$(arg name)" prefix="$(arg prefix)internal_" parent="${prefix}hatch_face">
-      <origin xyz="-0.1716 -0.475371 0.602" rpy="0 -${pi/2} 0"/>
+      <origin xyz="0.04431 -0.475371 0.602" rpy="0 ${pi/2} 0"/>
     </xacro:crank_wheel>
     <xacro:include filename="$(find hatch_accessories)/urdf/grab_handle.xacro"/>
     <xacro:grab_handle name="$(arg name)" prefix="$(arg prefix)external_" parent="${prefix}hatch_face">
-      <origin xyz="-0.0597 -0.788394 0.3147147" rpy="-0.3926991 0 0"/>
+      <origin xyz="-0.0776 -0.851588 0.3093442" rpy="0 ${pi} 0"/>
     </xacro:grab_handle>
     <xacro:grab_handle name="$(arg name)" prefix="$(arg prefix)internal_" parent="${prefix}hatch_face">
-      <origin xyz="-0.0776 -0.851588 0.3093442" rpy="0 ${pi} 0"/>
+      <origin xyz="-0.0597 -0.788394 0.3147147" rpy="-0.3926991 0 0"/>
     </xacro:grab_handle>
   </xacro:macro>

File: hatch_4060/urdf/hatch_4060.xacro (robot description, xacro)
@@ -82,8 +82,8 @@
     <!--TODO are the centers located properly?-->
     <xacro:crank_wheel name="$(arg name)" prefix="$(arg prefix)external_" parent="${prefix}hatch_face">
-      <origin xyz="0.04431 -0.9474 0.4295" rpy="0 ${pi/2} 0"/>
+      <origin xyz="-0.17161 -0.9474 0.4295" rpy="0 -${pi/2} 0"/>
     </xacro:crank_wheel>
     <xacro:crank_wheel name="$(arg name)" prefix="$(arg prefix)internal_" parent="${prefix}hatch_face">
-      <origin xyz="-0.17161 -0.9474 0.4295" rpy="0 -${pi/2} 0"/>
+      <origin xyz="0.04431 -0.9474 0.4295" rpy="0 ${pi/2} 0"/>
     </xacro:crank_wheel>
     <xacro:include filename="$(find hatch_accessories)/urdf/grab_handle.xacro"/>
@@ -91,20 +91,20 @@
     <xacro:if value="${external_handle_1}">
       <xacro:grab_handle name="$(arg name)" prefix="$(arg prefix)external_1_" parent="${prefix}hatch_face">
-        <origin xyz="-0.0573 -0.9016 0.7357" rpy="0 0 0"/>
+        <origin xyz="-0.07 -0.9016 0.7957" rpy="0 ${pi} 0"/>
       </xacro:grab_handle>
     </xacro:if>
     <xacro:if value="${external_handle_2}">
       <xacro:grab_handle name="$(arg name)" prefix="$(arg prefix)external_2_" parent="${prefix}hatch_face">
-        <origin xyz="-0.0497 -1.078 0.6957" rpy="${pi/2} 0 0"/>
+        <origin xyz="-0.0776 -1.0293 0.6957" rpy="${-pi/2} ${pi} 0"/>
       </xacro:grab_handle>
     </xacro:if>
     <xacro:if value="${internal_handle_1}">
       <xacro:grab_handle name="$(arg name)" prefix="$(arg prefix)internal_1_" parent="${prefix}hatch_face">
-        <origin xyz="-0.07 -0.9016 0.7957" rpy="0 ${pi} 0"/>
+        <origin xyz="-0.0573 -0.9016 0.7357" rpy="0 0 0"/>
       </xacro:grab_handle>
     </xacro:if>
     <xacro:if value="${internal_handle_2}">
       <xacro:grab_handle name="$(arg name)" prefix="$(arg prefix)internal_2_" parent="${prefix}hatch_face">
-        <origin xyz="-0.0776 -1.0293 0.6957" rpy="${-pi/2} ${pi} 0"/>
+        <origin xyz="-0.0497 -1.078 0.6957" rpy="${pi/2} 0 0"/>
       </xacro:grab_handle>
     </xacro:if>

Commit message: fixing namespacing issues for 4040 and 4060, and allowing manager to handle prefix

File: hatch_4040/urdf/hatch_4040.xacro (robot description, xacro)
@@ -1,5 +1,5 @@
 <?xml version="1.0"?>
 <robot xmlns:xacro="http://wiki.ros.org/xacro">
-  <xacro:macro name="hatch" params="
+  <xacro:macro name="hatch_4040" params="
     name:=''
     prefix:=''
@@ -7,5 +7,5 @@
     *origin">
     <joint name="${prefix}hatch_outer_frame_joint" type="fixed">
-      <parent link="${prefix}${parent}"/>
+      <parent link="${parent}"/>
       <child link="${prefix}hatch_outer_frame"/>
       <xacro:insert_block name="origin"/>
@@ -75,15 +75,15 @@
     <link name="${prefix}right_cal_2_frame"/>
     <xacro:include filename="$(find hatch_accessories)/urdf/crank_wheel.xacro"/>
-    <xacro:crank_wheel name="$(arg name)" prefix="$(arg prefix)external_" parent="${prefix}hatch_face">
+    <xacro:crank_wheel name="$(arg name)" prefix="${prefix}external_" parent="${prefix}hatch_face">
       <origin xyz="-0.1716 -0.475371 0.602" rpy="0 -${pi/2} 0"/>
     </xacro:crank_wheel>
-    <xacro:crank_wheel name="$(arg name)" prefix="$(arg prefix)internal_" parent="${prefix}hatch_face">
+    <xacro:crank_wheel name="$(arg name)" prefix="${prefix}internal_" parent="${prefix}hatch_face">
       <origin xyz="0.04431 -0.475371 0.602" rpy="0 ${pi/2} 0"/>
     </xacro:crank_wheel>
     <xacro:include filename="$(find hatch_accessories)/urdf/grab_handle.xacro"/>
-    <xacro:grab_handle name="$(arg name)" prefix="$(arg prefix)external_" parent="${prefix}hatch_face">
+    <xacro:grab_handle name="$(arg name)" prefix="${prefix}external_" parent="${prefix}hatch_face">
       <origin xyz="-0.0776 -0.851588 0.3093442" rpy="0 ${pi} 0"/>
     </xacro:grab_handle>
-    <xacro:grab_handle name="$(arg name)" prefix="$(arg prefix)internal_" parent="${prefix}hatch_face">
+    <xacro:grab_handle name="$(arg name)" prefix="${prefix}internal_" parent="${prefix}hatch_face">
       <origin xyz="-0.0597 -0.788394 0.3147147" rpy="-0.3926991 0 0"/>
     </xacro:grab_handle>

File: hatch_4060/urdf/hatch_4060.xacro (robot description, xacro)
@@ -1,5 +1,5 @@
 <?xml version="1.0"?>
 <robot xmlns:xacro="http://wiki.ros.org/xacro">
-  <xacro:macro name="hatch" params="
+  <xacro:macro name="hatch_4060" params="
     name:=''
     prefix:=''
@@ -12,5 +12,5 @@
     internal_handle_2:='false'">
     <joint name="${prefix}hatch_inner_frame_joint" type="fixed">
-      <parent link="${prefix}${parent}"/>
+      <parent link="${parent}"/>
       <child link="${prefix}hatch_inner_frame"/>
       <origin xyz="0.584329 1.245 0.7113" rpy="0 0 ${pi}"/>
@@ -39,5 +39,5 @@
     </link>
     <joint name="${prefix}hatch_outer_frame_joint" type="fixed">
-      <parent link="${prefix}${parent}"/>
+      <parent link="${parent}"/>
       <child link="${prefix}hatch_outer_frame"/>
       <xacro:insert_block name="origin"/>
@@ -109,8 +109,8 @@
     <xacro:include filename="$(find hatch_accessories)/urdf/crank_wheel.xacro"/>
     <!--TODO are the centers located properly?-->
-    <xacro:crank_wheel name="$(arg name)" prefix="$(arg prefix)external_" parent="${prefix}hatch_face">
+    <xacro:crank_wheel name="$(arg name)" prefix="${prefix}external_" parent="${prefix}hatch_face">
       <origin xyz="-0.17161 -0.9474 0.4325" rpy="0 -${pi/2} 0"/>
     </xacro:crank_wheel>
-    <xacro:crank_wheel name="$(arg name)" prefix="$(arg prefix)internal_" parent="${prefix}hatch_face">
+    <xacro:crank_wheel name="$(arg name)" prefix="${prefix}internal_" parent="${prefix}hatch_face">
       <origin xyz="0.04431 -0.9474 0.4265" rpy="0 ${pi/2} 0"/>
     </xacro:crank_wheel>
@@ -118,25 +118,25 @@
     <!--TODO which handles are mounted?-->
     <xacro:if value="${external_handle_1}">
-      <xacro:grab_handle name="$(arg name)" prefix="$(arg prefix)external_1_" parent="${prefix}hatch_face">
+      <xacro:grab_handle name="$(arg name)" prefix="${prefix}external_1_" parent="${prefix}hatch_face">
         <origin xyz="-0.07 -0.9016 ${0.7971+0.005}" rpy="0 ${pi} 0"/>
       </xacro:grab_handle>
     </xacro:if>
     <xacro:if value="${external_handle_2}">
-      <xacro:grab_handle name="$(arg name)" prefix="$(arg prefix)external_2_" parent="${prefix}hatch_face">
+      <xacro:grab_handle name="$(arg name)" prefix="${prefix}external_2_" parent="${prefix}hatch_face">
         <origin xyz="-0.07 ${-1.0223-0.005} ${0.6957 - 0.007}" rpy="${-pi/2} ${pi} 0"/>
       </xacro:grab_handle>
     </xacro:if>
     <xacro:if value="${external_handle_3}">
-      <xacro:grab_handle name="$(arg name)" prefix="$(arg prefix)external_3_" parent="${prefix}hatch_face">
+      <xacro:grab_handle name="$(arg name)" prefix="${prefix}external_3_" parent="${prefix}hatch_face">
         <origin xyz="${-0.07-0.005} ${-0.145+0.0195 - 0.004} 0.6957" rpy="${-pi/2} ${pi} 0"/>
       </xacro:grab_handle>
     </xacro:if>
     <xacro:if value="${internal_handle_1}">
-      <xacro:grab_handle name="$(arg name)" prefix="$(arg prefix)internal_1_" parent="${prefix}hatch_face">
+      <xacro:grab_handle name="$(arg name)" prefix="${prefix}internal_1_" parent="${prefix}hatch_face">
         <origin xyz="-0.058 -0.9016 0.7971" rpy="0 0 0"/>
       </xacro:grab_handle>
     </xacro:if>
     <xacro:if value="${internal_handle_2}">
-      <xacro:grab_handle name="$(arg name)" prefix="$(arg prefix)internal_2_" parent="${prefix}hatch_face">
+      <xacro:grab_handle name="$(arg name)" prefix="${prefix}internal_2_" parent="${prefix}hatch_face">
         <origin xyz="-0.058 -1.078 0.6957" rpy="${pi/2} 0 0"/>
       </xacro:grab_handle>
