Commit message: added hinge side handle to 4040

File: hatch_4040/urdf/hatch_4040.xacro (robot description, xacro)
@@ -85,4 +85,7 @@
       <origin xyz="-0.0776 -0.851588 0.3093442" rpy="0 ${pi} 0"/>
     </xacro:grab_handle>
+    <xacro:grab_handle prefix="${prefix}external_hinge_" parent="${prefix}hatch_face">
+      <origin xyz="-0.0776 -0.251588 0.3093442" rpy="0 ${pi} 0"/>
+    </xacro:grab_handle>
     <xacro:grab_handle prefix="${prefix}internal_" parent="${prefix}hatch_face">
       <origin xyz="-0.0597 -0.788394 0.3147147" rpy="-0.3926991 0 0"/>

Commit message: Update handle macro in hatch_4040

File: hatch_4040/urdf/hatch_4040.xacro (robot description, xacro)
@@ -92,7 +92,11 @@
     </xacro:grab_handle>
   </xacro:macro>
-  <xacro:macro name="hatch_4040_mj_processed_inputs">
+  <xacro:macro name="hatch_4040_mj_processed_inputs" params="
+    prefix:=''
+    ">
     <xacro:include filename="$(find hatch_accessories)/urdf/grab_handle.xacro"/>
-    <xacro:grab_handle_mj_processed_inputs/>
+    <xacro:grab_handle_mj_processed_inputs prefix="${prefix}external_"/>
+    <xacro:grab_handle_mj_processed_inputs prefix="${prefix}external_hinge_"/>
+    <xacro:grab_handle_mj_processed_inputs prefix="${prefix}internal_"/>
     <decompose_mesh mesh_name="hatch_4040_frame" threshold="0.01"/>
     <decompose_mesh mesh_name="hatch_4040_face" threshold="0.01"/>
