Commit message: Adding grasping frames for the grab handle and rotary handle.

File: hatch_accessories/urdf/crank_wheel.xacro (robot description, xacro)
@@ -66,4 +66,10 @@
       </collision>
     </link>
+    <joint name="${prefix}rotary_handle_grasp_joint" type="fixed">
+      <parent link="${prefix}rotary_handle"/>
+      <child link="${prefix}rotary_handle_grasp"/>
+      <origin xyz="0.0 0.0 0.04" rpy="0 0 0"/>
+    </joint>
+    <link name="${prefix}rotary_handle_grasp"/>
   </xacro:macro>
 </robot>

File: hatch_accessories/urdf/grab_handle.xacro (robot description, xacro)
@@ -8,8 +8,8 @@
     <joint name="${prefix}grab_handle_joint" type="fixed">
       <parent link="${parent}"/>
-      <child link="${prefix}exterior_grab_handle"/>
+      <child link="${prefix}grab_handle"/>
       <xacro:insert_block name="origin"/>
     </joint>
-    <link name="${prefix}exterior_grab_handle">
+    <link name="${prefix}grab_handle">
       <!--TODO set proper inertia-->
       <inertial>
@@ -35,4 +35,10 @@
       </collision>
     </link>
+    <joint name="${prefix}grab_center_joint" type="fixed">
+      <parent link="${prefix}grab_handle"/>
+      <child link="${prefix}grab_center"/>
+      <origin xyz="0.082 -0.0935 0.0" rpy="0 0 0"/>
+    </joint>
+    <link name="${prefix}grab_center"/>
   </xacro:macro>
 </robot>
