Commit message: adjusted hatch walls

File: hatch_accessories/urdf/hatch_frame.xacro (robot description, xacro)
@@ -47,7 +47,7 @@
     <link name="${prefix}hatch_back">
       <collision>
-        <origin xyz="${0.1/2} ${1.307/2} ${0.610/2}" rpy="0 0 0"/>
+        <origin xyz="${0.1/2} ${1.307/2} ${0.4953/2}" rpy="0 0 0"/>
         <geometry>
-          <box size="0.1 1.307 0.610"/>
+          <box size="0.1 1.307 0.4953"/>
         </geometry>
         <material name="red"/>
@@ -61,7 +61,7 @@
     <link name="${prefix}hatch_front">
       <collision>
-        <origin xyz="${0.1/2} ${1.307/2} ${0.610/2}" rpy="0 0 0"/>
+        <origin xyz="${0.1/2} ${1.307/2} ${0.4953/2}" rpy="0 0 0"/>
         <geometry>
-          <box size="0.1 1.307 0.610"/>
+          <box size="0.1 1.307 0.4953"/>
         </geometry>
         <material name="red"/>
@@ -95,7 +95,7 @@
     <link name="${prefix}hatch_right">
       <collision>
-        <origin xyz="${0.675/2} ${0.1/2} ${2.108/2}" rpy="0 0 0"/>
+        <origin xyz="${0.675/2} ${0.1/2} ${0.4953/2}" rpy="0 0 0"/>
         <geometry>
-          <box size="0.675 0.1 2.1082"/>
+          <box size="0.675 0.1 0.4953"/>
         </geometry>
         <material name="red"/>

Commit message: fixed left side collision

File: hatch_accessories/urdf/hatch_frame.xacro (robot description, xacro)
@@ -101,4 +101,11 @@
         <material name="red"/>
       </collision>
+      <collision>
+        <origin xyz="${1.307/2 - 0.1/4} ${0.1/2} ${2.1082/2}" rpy="0 0 0"/>
+        <geometry>
+          <box size="0.1 0.1 2.1082"/>
+        </geometry>
+        <material name="red"/>
+      </collision>
     </link>
     <joint name="${prefix}hatch_bottom_top" type="fixed">

Commit message: added no left stl

File: hatch_accessories/urdf/hatch_frame.xacro (robot description, xacro)
@@ -15,5 +15,6 @@
         <origin xyz="0.0 0.0 0.0" rpy="0 0 0"/>
         <geometry>
-          <mesh filename="package://hatch_accessories/meshes/visual/ivr_hatch_frame.stl"/>
+          <!-- <mesh filename="package://hatch_accessories/meshes/visual/ivr_hatch_frame.stl"/> -->
+          <mesh filename="package://hatch_accessories/meshes/visual/ivr_hatch_frame_no_left.stl"/>
         </geometry>
         <material name="gray"/>

Commit message: calibrated bench height

File: hatch_accessories/urdf/hatch_frame.xacro (robot description, xacro)
@@ -139,5 +139,5 @@
     <link name="${prefix}hatch_bench">
       <visual>
-        <origin xyz="${0.675/2} ${1.307/2} ${0.4953/2}" rpy="0 0 0"/>
+        <origin xyz="${0.675/2} ${1.307/2} ${0.4953/2 + 0.01}" rpy="0 0 0"/>
         <geometry>
           <box size="0.675 1.307 0.4953"/>
@@ -146,5 +146,5 @@
       </visual>
       <collision>
-        <origin xyz="${0.675/2} ${1.307/2} ${0.4953/2}" rpy="0 0 0"/>
+        <origin xyz="${0.675/2} ${1.307/2} ${0.4953/2 + 0.01}" rpy="0 0 0"/>
         <geometry>
           <box size="0.675 1.307 0.4953"/>
