Commit message: Adding additional grasp and calibration frames.

File: hatch_accessories/urdf/grab_handle.xacro (robot description, xacro)
@@ -38,7 +38,13 @@
       <parent link="${prefix}grab_handle"/>
       <child link="${prefix}grab_center"/>
-      <origin xyz="0.082 -0.0935 0.0" rpy="0 0 0"/>
+      <origin xyz="0.0807 -0.0889 0.0" rpy="0 0 0"/>
     </joint>
     <link name="${prefix}grab_center"/>
+    <joint name="${prefix}grab_touch_joint" type="fixed">
+      <parent link="${prefix}grab_handle"/>
+      <child link="${prefix}grab_touch"/>
+      <origin xyz="0.0934 -0.0889 0.0" rpy="0 0 0"/>
+    </joint>
+    <link name="${prefix}grab_touch"/>
   </xacro:macro>
 </robot>

File: hatch_accessories/urdf/hatch_frame.xacro (robot description, xacro)
@@ -20,10 +20,10 @@
       </visual>
     </link>
-    <joint name="hatch_frame_joint" type="fixed">
-      <parent link="hatch_frame"/>
-      <child link="hatch_bottom"/>
+    <joint name="${prefix}hatch_frame_joint" type="fixed">
+      <parent link="${prefix}hatch_frame"/>
+      <child link="${prefix}hatch_bottom"/>
       <origin xyz="0.0 0.0 0.0" rpy="0 0 0"/>
     </joint>
-    <link name="hatch_bottom">
+    <link name="${prefix}hatch_bottom">
       <!--TODO set proper inertia-->
       <inertial>
@@ -40,10 +40,10 @@
       </collision>
     </link>
-    <joint name="hatch_bottom_back" type="fixed">
-      <parent link="hatch_bottom"/>
-      <child link="hatch_back"/>
+    <joint name="${prefix}hatch_bottom_back" type="fixed">
+      <parent link="${prefix}hatch_bottom"/>
+      <child link="${prefix}hatch_back"/>
       <origin xyz="0.0 0.0 0.0" rpy="0 0 0"/>
     </joint>
-    <link name="hatch_back">
+    <link name="${prefix}hatch_back">
       <collision>
         <origin xyz="${0.1/2} ${1.307/2} ${0.610/2}" rpy="0 0 0"/>
@@ -54,10 +54,10 @@
       </collision>
     </link>
-    <joint name="hatch_bottom_front" type="fixed">
-      <parent link="hatch_bottom"/>
-      <child link="hatch_front"/>
+    <joint name="${prefix}hatch_bottom_front" type="fixed">
+      <parent link="${prefix}hatch_bottom"/>
+      <child link="${prefix}hatch_front"/>
       <origin xyz="0.578 0.0 0.0" rpy="0 0 0"/>
     </joint>
-    <link name="hatch_front">
+    <link name="${prefix}hatch_front">
       <collision>
         <origin xyz="${0.1/2} ${1.307/2} ${0.610/2}" rpy="0 0 0"/>
@@ -68,10 +68,16 @@
       </collision>
     </link>
-    <joint name="hatch_bottom_left" type="fixed">
-      <parent link="hatch_bottom"/>
-      <child link="hatch_left"/>
+    <joint name="${prefix}hatch_frame_front_bottom_joint" type="fixed">
+      <parent link="${prefix}hatch_frame"/>
+      <child link="${prefix}hatch_frame_front_bottom"/>
+      <origin xyz="0.67 0.0 0.0" rpy="0 0 0"/>
+    </joint>
+    <link name="${prefix}hatch_frame_front_bottom"/>
+    <joint name="${prefix}hatch_bottom_left" type="fixed">
+      <parent link="${prefix}hatch_bottom"/>
+      <child link="${prefix}hatch_left"/>
       <origin xyz="0.0 -0.01 0.0" rpy="0 0 0"/>
     </joint>
-    <link name="hatch_left">
+    <link name="${prefix}hatch_left">
       <collision>
         <origin xyz="${0.675/2} ${0.1/2} ${2.1082/2}" rpy="0 0 0"/>
@@ -82,10 +88,10 @@
       </collision>
     </link>
-    <joint name="hatch_bottom_right" type="fixed">
-      <parent link="hatch_bottom"/>
-      <child link="hatch_right"/>
+    <joint name="${prefix}hatch_bottom_right" type="fixed">
+      <parent link="${prefix}hatch_bottom"/>
+      <child link="${prefix}hatch_right"/>
       <origin xyz="0.0 1.22 0.0" rpy="0 0 0"/>
     </joint>
-    <link name="hatch_right">
+    <link name="${prefix}hatch_right">
       <collision>
         <origin xyz="${0.675/2} ${0.1/2} ${2.108/2}" rpy="0 0 0"/>
@@ -96,10 +102,10 @@
       </collision>
     </link>
-    <joint name="hatch_bottom_top" type="fixed">
-      <parent link="hatch_bottom"/>
-      <child link="hatch_top"/>
+    <joint name="${prefix}hatch_bottom_top" type="fixed">
+      <parent link="${prefix}hatch_bottom"/>
+      <child link="${prefix}hatch_top"/>
       <origin xyz="0.589 0.0 1.913" rpy="0 0 0"/>
     </joint>
-    <link name="hatch_top">
+    <link name="${prefix}hatch_top">
       <collision>
         <origin xyz="${0.1/2} ${1.307/2} ${0.197/2}" rpy="0 0 0"/>
@@ -110,4 +116,10 @@
       </collision>
     </link>
+    <joint name="${prefix}hatch_frame_front_top_joint" type="fixed">
+      <parent link="${prefix}hatch_frame"/>
+      <child link="${prefix}hatch_frame_front_top"/>
+      <origin xyz="0.67 0.0 2.111" rpy="0 0 0"/>
+    </joint>
+    <link name="${prefix}hatch_frame_front_top"/>
   </xacro:macro>
 </robot>

Commit message: added red tape texture to grab_handle, replaced grab_handle visual mesh

File: hatch_accessories/urdf/grab_handle.xacro (robot description, xacro)
@@ -18,13 +18,13 @@
       </inertial>
       <visual>
-        <!--This transform is for the stl file origin-->
         <origin xyz="0.0 0.0 0.0" rpy="0 0 0"/>
         <geometry>
-          <mesh filename="package://hatch_accessories/meshes/visual/grab_handle.stl"/>
+          <mesh filename="package://hatch_accessories/meshes/visual/imetro_hatch_handle.dae"/>
         </geometry>
-        <material name="blue"/>
+        <material name="${prefix}grab_handle_texture">
+          <texture filename="package://hatch_accessories/meshes/visual/grab_handle_texture.png"/>
+        </material>
       </visual>
       <collision>
-        <!--This transform is for the stl file origin-->
         <origin xyz="0.0 0.0 0.0" rpy="0 0 0"/>
         <geometry>
