Commit message: added tape hatch handle, cranks handle, and bench lid

File: hatch_accessories/urdf/colors.xacro (robot description, xacro)
@@ -13,3 +13,6 @@
     <color rgba="0.85 0.85 0.85 1"/>
   </material>
+  <material name="black">
+    <color rgba="0 0 0 1"/>
+  </material>
 </robot>

File: hatch_accessories/urdf/crank_wheel.xacro (robot description, xacro)
@@ -26,5 +26,5 @@
           <mesh filename="package://hatch_accessories/meshes/visual/crank_wheel.stl"/>
         </geometry>
-        <material name="blue"/>
+        <material name="black"/>
       </visual>
       <collision>
@@ -55,7 +55,9 @@
         <origin xyz="0.0 0.0 0.00355" rpy="0 0 0"/>
         <geometry>
-          <mesh filename="package://hatch_accessories/meshes/visual/crank_handle.stl"/>
+          <mesh filename="package://hatch_accessories/meshes/visual/crank_handle.dae"/>
         </geometry>
-        <material name="blue"/>
+        <material name="${prefix}rotary_handle_texture">
+          <texture filename="package://hatch_accessories/meshes/visual/grab_handle_texture.png"/>
+        </material>
       </visual>
       <collision>

File: trainer/urdf/bench_seat.xacro (robot description, xacro)
@@ -129,5 +129,5 @@
         <origin xyz="0.0 0.0 0.0" rpy="0 0 0"/>
         <geometry>
-          <mesh filename="package://trainer/meshes/visual/imetro_bench_lid.dae"/>
+          <mesh filename="package://trainer/meshes/visual/bench_lid.dae"/>
         </geometry>
         <material name="${prefix}bench_lid_texture">
