Commit message: fixing colors

File: hatch_accessories/urdf/colors.xacro (robot description, xacro)
@@ -16,3 +16,6 @@
     <color rgba="0 0 0 1"/>
   </material>
+  <material name="white">
+    <color rgba="1 1 1 1"/>
+  </material>
 </robot>

File: trainer/urdf/colors.xacro (robot description, xacro)
@@ -13,3 +13,6 @@
     <color rgba="0.85 0.85 0.85 1.0"/>
   </material>
+  <material name="white">
+    <color rgba="1.0 1.0 1.0 1.0"/>
+  </material>
 </robot>

File: trainer/urdf/trainer_front_right_face.xacro (robot description, xacro)
@@ -52,5 +52,5 @@
         <mesh filename="package://trainer/meshes/visual/cabinet_door_1.stl"/>
       </geometry>
-      <material name="blue"/>
+      <material name="white"/>
     </visual>
     <collision>
@@ -109,5 +109,5 @@
         <mesh filename="package://trainer/meshes/visual/round_latch_handle.stl"/>
       </geometry>
-      <material name="blue"/>
+      <material name="gray"/>
     </visual>
     <collision>
@@ -139,5 +139,5 @@
         <mesh filename="package://trainer/meshes/visual/cabinet_door_2.stl"/>
       </geometry>
-      <material name="blue"/>
+      <material name="white"/>
     </visual>
     <collision>
@@ -197,5 +197,5 @@
         <mesh filename="package://trainer/meshes/visual/push_latch_button.stl"/>
       </geometry>
-      <material name="blue"/>
+      <material name="gray"/>
     </visual>
     <collision>
@@ -227,5 +227,5 @@
         <mesh filename="package://trainer/meshes/visual/push_latch_handle.stl"/>
       </geometry>
-      <material name="blue"/>
+      <material name="gray"/>
     </visual>
     <collision>
@@ -257,5 +257,5 @@
         <mesh filename="package://trainer/meshes/visual/cabinet_door_3.stl"/>
       </geometry>
-      <material name="blue"/>
+      <material name="white"/>
     </visual>
     <collision>

File: trainer/urdf/trainer_side.xacro (robot description, xacro)
@@ -136,5 +136,5 @@
         <mesh filename="package://trainer/meshes/visual/paddle_latch_handle.stl"/>
       </geometry>
-      <material name="blue"/>
+      <material name="gray"/>
     </visual>
     <collision>
@@ -166,5 +166,5 @@
         <mesh filename="package://trainer/meshes/visual/drawer_1_face.stl"/>
       </geometry>
-      <material name="blue"/>
+      <material name="gray"/>
     </visual>
     <collision>
@@ -193,5 +193,5 @@
         <box size="0.013 0.305 0.096"/>
       </geometry>
-      <material name="blue"/>
+      <material name="white"/>
     </visual>
     <collision>
@@ -220,5 +220,5 @@
         <box size="0.013 0.305 0.096"/>
       </geometry>
-      <material name="blue"/>
+      <material name="white"/>
     </visual>
     <collision>
@@ -247,5 +247,5 @@
         <box size="0.293 0.305 0.013"/>
       </geometry>
-      <material name="blue"/>
+      <material name="white"/>
     </visual>
     <collision>
@@ -277,5 +277,5 @@
         <mesh filename="package://trainer/meshes/visual/drawer_2_face.stl"/>
       </geometry>
-      <material name="blue"/>
+      <material name="white"/>
     </visual>
     <collision>
@@ -334,5 +334,5 @@
         <mesh filename="package://trainer/meshes/visual/recessed_latch_handle.stl"/>
       </geometry>
-      <material name="blue"/>
+      <material name="gray"/>
     </visual>
     <collision>
@@ -361,5 +361,5 @@
         <box size="0.013 0.305 0.096"/>
       </geometry>
-      <material name="blue"/>
+      <material name="white"/>
     </visual>
     <collision>
@@ -388,5 +388,5 @@
         <box size="0.013 0.305 0.096"/>
       </geometry>
-      <material name="blue"/>
+      <material name="white"/>
     </visual>
     <collision>
@@ -415,5 +415,5 @@
         <box size="0.293 0.305 0.013"/>
       </geometry>
-      <material name="blue"/>
+      <material name="white"/>
     </visual>
     <collision>
