Commit message: The urdf isn't quite right but is getting really close.

File: urdf/merlin_mockup.urdf.xacro (robot description, xacro)
@@ -39,3 +39,112 @@
     <limit effort="10" velocity="10" lower="0" upper="${pi/2}"/>
   </joint>
+  <link name="latch_housing">
+    <visual>
+      <origin xyz="0 0 0" rpy="0 ${pi} 0"/>
+      <geometry>
+        <mesh filename="package://merlin_mockup_description/meshes/visual/csm_latch_housing.stl"/>
+      </geometry>
+    </visual>
+    <collision>
+      <origin xyz="0 0 0" rpy="0 ${pi} 0"/>
+      <geometry>
+        <mesh filename="package://merlin_mockup_description/meshes/visual/csm_latch_housing.stl"/>
+      </geometry>
+    </collision>
+  </link>
+  <!-- positioning is totally wrong but just checking to see if it all hooks up at this point-->
+  <joint name="door_to_latch" type="fixed">
+    <parent link="door"/>
+    <child link="latch_housing"/>
+    <origin xyz="0 0.0 0.2" rpy="0 0 0"/>
+  </joint>
+  <!-- Cover section-->
+  <link name="latch_cover">
+    <visual>
+      <origin xyz="0 0 0" rpy="0 0 0"/>
+      <geometry>
+        <mesh filename="package://merlin_mockup_description/meshes/visual/csm_latch_cover.stl"/>
+      </geometry>
+    </visual>
+    <collision>
+      <origin xyz="0 0 0" rpy="0 0 0"/>
+      <geometry>
+        <mesh filename="package://merlin_mockup_description/meshes/visual/csm_latch_cover.stl"/>
+      </geometry>
+    </collision>
+  </link>
+  <joint name="housing_to_cover" type="fixed">
+    <parent link="latch_housing"/>
+    <child link="latch_cover"/>
+    <origin xyz="0 0.012 0.0" rpy="0 0 0"/>
+  </joint>
+  <!-- Right latch pull section-->
+  <link name="right_latch_pull">
+    <visual>
+      <origin xyz="0 0 0" rpy="${pi} -${pi/2} -${pi/2}"/>
+      <geometry>
+        <mesh filename="package://merlin_mockup_description/meshes/visual/csm_latch_pull.stl"/>
+      </geometry>
+    </visual>
+    <collision>
+      <origin xyz="0 0 0" rpy="${pi} -${pi/2} -${pi/2}"/>
+      <geometry>
+        <mesh filename="package://merlin_mockup_description/meshes/visual/csm_latch_pull.stl"/>
+      </geometry>
+    </collision>
+  </link>
+  <!-- positioning is totally wrong but just checking to see if it all hooks up at this point-->
+  <joint name="housing_to_right_latch_pull" type="prismatic">
+    <parent link="latch_housing"/>
+    <child link="right_latch_pull"/>
+    <origin xyz="0.0258 0.01 -0.004" rpy="0 0 0"/>
+    <axis xyz="1 0 0" />
+    <limit effort="10" velocity="10" lower="0" upper="0.2"/>
+  </joint>
+  <!-- Left latch pull section-->
+  <link name="left_latch_pull">
+    <visual>
+      <origin xyz="0 0 0" rpy="0 ${pi/2} -${pi/2}"/>
+      <geometry>
+        <mesh filename="package://merlin_mockup_description/meshes/visual/csm_latch_pull.stl"/>
+      </geometry>
+    </visual>
+    <collision>
+      <origin xyz="0 0 0" rpy="0 ${pi/2} -${pi/2}"/>
+      <geometry>
+        <mesh filename="package://merlin_mockup_description/meshes/visual/csm_latch_pull.stl"/>
+      </geometry>
+    </collision>
+  </link>
+  <!-- positioning is totally wrong but just checking to see if it all hooks up at this point-->
+  <joint name="housing_to_left_latch_pull" type="prismatic">
+    <parent link="latch_housing"/>
+    <child link="left_latch_pull"/>
+    <origin xyz="-0.0258 0.01 -0.004" rpy="0 0 0"/>
+    <axis xyz="1 0 0" />
+    <limit effort="10" velocity="10" lower="-0.020" upper="0"/>
+  </joint>
+  <!-- Latch lock section-->
+  <link name="latch_lock">
+    <visual>
+      <origin xyz="0 0 0" rpy="0 0 0"/>
+      <geometry>
+        <mesh filename="package://merlin_mockup_description/meshes/visual/csm_latch_lock.stl"/>
+      </geometry>
+    </visual>
+    <collision>
+      <origin xyz="0 0 0" rpy="0 0 0"/>
+      <geometry>
+        <mesh filename="package://merlin_mockup_description/meshes/visual/csm_latch_lock.stl"/>
+      </geometry>
+    </collision>
+  </link>
+  <!-- positioning is totally wrong but just checking to see if it all hooks up at this point-->
+  <joint name="housing_to_latch_lock" type="revolute">
+    <parent link="latch_housing"/>
+    <child link="latch_lock"/>
+    <origin xyz="0 0.02 -0.001" rpy="0 0 0"/>
+    <axis xyz="1 0 0" />
+    <limit effort="10" velocity="10" lower="0" upper="${pi/4}"/>
+  </joint>
 </robot>

Commit message: Latch pulls and lock are located in the correct positions.

File: urdf/merlin_mockup.urdf.xacro (robot description, xacro)
@@ -57,5 +57,5 @@
     <parent link="door"/>
     <child link="latch_housing"/>
-    <origin xyz="0 0.0 0.2" rpy="0 0 0"/>
+    <origin xyz="0 0.0 0.135" rpy="0 0 0"/>
   </joint>
   <!-- Cover section-->
@@ -94,5 +94,4 @@
     </collision>
   </link>
-  <!-- positioning is totally wrong but just checking to see if it all hooks up at this point-->
   <joint name="housing_to_right_latch_pull" type="prismatic">
     <parent link="latch_housing"/>
@@ -100,5 +99,5 @@
     <origin xyz="0.0258 0.01 -0.004" rpy="0 0 0"/>
     <axis xyz="1 0 0" />
-    <limit effort="10" velocity="10" lower="0" upper="0.2"/>
+    <limit effort="10" velocity="10" lower="-0.0084" upper="0"/>
   </joint>
   <!-- Left latch pull section-->
@@ -117,5 +116,4 @@
     </collision>
   </link>
-  <!-- positioning is totally wrong but just checking to see if it all hooks up at this point-->
   <joint name="housing_to_left_latch_pull" type="prismatic">
     <parent link="latch_housing"/>
@@ -123,10 +121,10 @@
     <origin xyz="-0.0258 0.01 -0.004" rpy="0 0 0"/>
     <axis xyz="1 0 0" />
-    <limit effort="10" velocity="10" lower="-0.020" upper="0"/>
+    <limit effort="10" velocity="10" lower="0" upper="0.0084"/>
   </joint>
   <!-- Latch lock section-->
   <link name="latch_lock">
     <visual>
-      <origin xyz="0 0 0" rpy="0 0 0"/>
+      <origin xyz="0 0.0012 -0.0084" rpy="0 0 0"/>
       <geometry>
         <mesh filename="package://merlin_mockup_description/meshes/visual/csm_latch_lock.stl"/>
@@ -134,5 +132,5 @@
     </visual>
     <collision>
-      <origin xyz="0 0 0" rpy="0 0 0"/>
+      <origin xyz="0 0.0012 -0.0084" rpy="0 0 0"/>
       <geometry>
         <mesh filename="package://merlin_mockup_description/meshes/visual/csm_latch_lock.stl"/>
@@ -140,9 +138,8 @@
     </collision>
   </link>
-  <!-- positioning is totally wrong but just checking to see if it all hooks up at this point-->
   <joint name="housing_to_latch_lock" type="revolute">
     <parent link="latch_housing"/>
     <child link="latch_lock"/>
-    <origin xyz="0 0.02 -0.001" rpy="0 0 0"/>
+    <origin xyz="0 0.019 0.007" rpy="0 0 0"/>
     <axis xyz="1 0 0" />
     <limit effort="10" velocity="10" lower="0" upper="${pi/4}"/>

Commit message: Corrected latch pulls and lock limits.

File: urdf/merlin_mockup.urdf.xacro (robot description, xacro)
@@ -143,5 +143,5 @@
     <origin xyz="0 0.019 0.007" rpy="0 0 0"/>
     <axis xyz="1 0 0" />
-    <limit effort="10" velocity="10" lower="0" upper="${pi/4}"/>
+    <limit effort="10" velocity="10" lower="0" upper="${pi/2}"/>
   </joint>
 </robot>

Commit message: Latch position relative to the door corrected but is 2mm off from what I'd expect in the CREO model. Line 64 at the time of the commit. 0.125 expected.

File: urdf/merlin_mockup.urdf.xacro (robot description, xacro)
@@ -57,5 +57,5 @@
     <parent link="door"/>
     <child link="latch_housing"/>
-    <origin xyz="0 0.0 0.135" rpy="0 0 0"/>
+    <origin xyz="0 0.0 0.123" rpy="0 0 0"/>
   </joint>
   <!-- Cover section-->

Commit message: Position and joint of the door are now correct.

File: urdf/merlin_mockup.urdf.xacro (robot description, xacro)
@@ -19,5 +19,5 @@
   <link name="door">
     <visual>
-      <origin xyz="0 0 0" rpy="${pi/2} 0 ${pi}"/>
+      <origin xyz="0 0 0.110" rpy="${pi/2} 0 ${pi}"/>
       <geometry>
         <mesh filename="package://merlin_mockup_description/meshes/visual/csm_outer_door.stl"/>
@@ -25,5 +25,5 @@
     </visual>
     <collision>
-      <origin xyz="0 0 0" rpy="${pi/2} 0 ${pi}"/>
+      <origin xyz="0 0 0.110" rpy="${pi/2} 0 ${pi}"/>
       <geometry>
         <mesh filename="package://merlin_mockup_description/meshes/visual/csm_outer_door.stl"/>
@@ -35,7 +35,7 @@
     <parent link="wood_frame"/>
     <child link="door"/>
-    <origin xyz="0 0.025 0" rpy="0 0 0"/>
+    <origin xyz="0 0.0125 -0.110" rpy="0 0 0"/>
     <axis xyz="1 0 0" />
-    <limit effort="10" velocity="10" lower="0" upper="${pi/2}"/>
+    <limit effort="10" velocity="10" lower="-${pi/2}" upper="0"/>
   </joint>
   <link name="latch_housing">
@@ -57,5 +57,5 @@
     <parent link="door"/>
     <child link="latch_housing"/>
-    <origin xyz="0 0.0 0.123" rpy="0 0 0"/>
+    <origin xyz="0 0.0 0.233" rpy="0 0 0"/>
   </joint>
   <!-- Cover section-->

Commit message: Slight update to wooden front to door transfor. It should be pretty close to the real now.

File: urdf/merlin_mockup.urdf.xacro (robot description, xacro)
@@ -35,5 +35,5 @@
     <parent link="wood_frame"/>
     <child link="door"/>
-    <origin xyz="0 0.0125 -0.110" rpy="0 0 0"/>
+    <origin xyz="0 0.0125 -0.113" rpy="0 0 0"/>
     <axis xyz="1 0 0" />
     <limit effort="10" velocity="10" lower="-${pi/2}" upper="0"/>

Commit message: Removing extra comments.

File: urdf/merlin_mockup.urdf.xacro (robot description, xacro)
@@ -8,13 +8,14 @@
     <visual>
       <geometry>
-        <mesh filename="package://merlin_mockup_description/meshes/visual/aso_freezer_wood_only.stl" scale="0.02527 0.02527 0.02527"/>
+        <mesh filename="package://merlin_mockup_description/meshes/visual/aso_locker_cavity_only.stl" scale="0.02527 0.02527 0.02527"/>
       </geometry>
     </visual>
     <collision>
       <geometry>
-        <mesh filename="package://merlin_mockup_description/meshes/visual/aso_freezer_wood_only.stl" scale="0.02527 0.02527 0.02527"/>
+        <mesh filename="package://merlin_mockup_description/meshes/visual/aso_locker_cavity_only.stl" scale="0.02527 0.02527 0.02527"/>
       </geometry>
     </collision>
   </link>
+  <!-- Door section-->
   <link name="door">
     <visual>
@@ -38,4 +39,5 @@
     <limit effort="10" velocity="10" lower="-${pi/2}" upper="0"/>
   </joint>
+  <!-- Latch housing section-->
   <link name="latch_housing">
     <visual>
@@ -45,14 +47,5 @@
       </geometry>
     </visual>
-    <!--
-    <collision>
-      <origin xyz="0 0 0" rpy="0 ${pi} 0"/>
-      <geometry>
-        <mesh filename="package://merlin_mockup_description/meshes/visual/csm_latch_housing.stl"/>
-      </geometry>
-    </collision>
-    -->
   </link>
-  <!-- positioning is totally wrong but just checking to see if it all hooks up at this point-->
   <joint name="door_to_latch" type="fixed">
     <parent link="door"/>
@@ -60,5 +53,5 @@
     <origin xyz="0 0.0 0.233" rpy="0 0 0"/>
   </joint>
-  <!-- Cover section-->
+  <!-- Latch cover section-->
   <link name="latch_cover">
     <visual>
@@ -68,12 +61,4 @@
       </geometry>
     </visual>
-    <!--
-    <collision>
-      <origin xyz="0 0 0" rpy="0 0 0"/>
-      <geometry>
-        <mesh filename="package://merlin_mockup_description/meshes/visual/csm_latch_cover.stl"/>
-      </geometry>
-    </collision>
-    -->
   </link>
   <joint name="housing_to_cover" type="fixed">
@@ -90,12 +75,4 @@
       </geometry>
     </visual>
-    <!--
-    <collision>
-      <origin xyz="0 0 0" rpy="${pi} -${pi/2} -${pi/2}"/>
-      <geometry>
-        <mesh filename="package://merlin_mockup_description/meshes/visual/csm_latch_pull.stl"/>
-      </geometry>
-    </collision>
-    -->
   </link>
   <joint name="housing_to_right_latch_pull" type="prismatic">
@@ -114,12 +91,4 @@
       </geometry>
     </visual>
-    <!--
-    <collision>
-      <origin xyz="0 0 0" rpy="0 ${pi/2} -${pi/2}"/>
-      <geometry>
-        <mesh filename="package://merlin_mockup_description/meshes/visual/csm_latch_pull.stl"/>
-      </geometry>
-    </collision>
-    -->
   </link>
   <joint name="housing_to_left_latch_pull" type="prismatic">
@@ -138,12 +107,4 @@
       </geometry>
     </visual>
-    <!--
-    <collision>
-      <origin xyz="0 0.0012 -0.0084" rpy="0 0 0"/>
-      <geometry>
-        <mesh filename="package://merlin_mockup_description/meshes/visual/csm_latch_lock.stl"/>
-      </geometry>
-    </collision>
-    -->
   </link>
   <joint name="housing_to_latch_lock" type="revolute">

Commit message: added template for velcro strip

File: urdf/merlin_mockup.urdf.xacro (robot description, xacro)
@@ -17,4 +17,25 @@
     </collision>
   </link>
+  <!-- Velcro section-->
+  <link name="velcro"> <!-- need to set all values -->
+    <visual>
+      <geometry>
+        <box size="0.01 0.001 0.05"/>
+      </geometry>
+    </visual>
+    <material name="Cyan">
+       <color rgba="0 1.0 1.0 1.0"/>
+     </material>
+    <collision>
+      <geometry>
+        <box size="0.01 0.001 0.05"/>
+      </geometry>
+    </collision>
+  </link>
+  <joint name="velcro_to_frame_joint" type="fixed">
+    <parent link="wood_frame"/>
+    <child link="velcro"/>
+    <origin xyz="-0.0 0.012 0.18" rpy="0 0 0"/>
+  </joint>
   <!-- Door section-->
   <link name="door">

Commit message: fixed material location

File: urdf/merlin_mockup.urdf.xacro (robot description, xacro)
@@ -23,8 +23,8 @@
         <box size="0.01 0.001 0.05"/>
       </geometry>
+      <material name="Cyan">
+        <color rgba="0 1.0 1.0 1.0"/>
+      </material>
     </visual>
-    <material name="Cyan">
-       <color rgba="0 1.0 1.0 1.0"/>
-     </material>
     <collision>
       <geometry>

Commit message: added more precice location for velcro based on test on merlin mockup hardware

File: urdf/merlin_mockup.urdf.xacro (robot description, xacro)
@@ -24,5 +24,5 @@
       </geometry>
       <material name="Cyan">
-        <color rgba="0 1.0 1.0 1.0"/>
+        <color rgba="0.0 0.0 0.0 1.0"/>
       </material>
     </visual>
@@ -36,5 +36,5 @@
     <parent link="wood_frame"/>
     <child link="velcro"/>
-    <origin xyz="-0.0 0.012 0.18" rpy="0 0 0"/>
+    <origin xyz="-0.10 0.012 0.20" rpy="0 0 0"/>
   </joint>
   <!-- Door section-->

Commit message: adjusted the velcro size in the urdf to match the piece attatched in the hardware

File: urdf/merlin_mockup.urdf.xacro (robot description, xacro)
@@ -21,5 +21,5 @@
     <visual>
       <geometry>
-        <box size="0.01 0.001 0.05"/>
+        <box size="0.11 0.001 0.05"/>
       </geometry>
       <material name="Cyan">
@@ -29,5 +29,5 @@
     <collision>
       <geometry>
-        <box size="0.01 0.001 0.05"/>
+        <box size="0.11 0.001 0.05"/>
       </geometry>
     </collision>
@@ -36,5 +36,5 @@
     <parent link="wood_frame"/>
     <child link="velcro"/>
-    <origin xyz="-0.10 0.012 0.20" rpy="0 0 0"/>
+    <origin xyz="-0.17535 0.012 0.2345" rpy="0 0 0"/>
   </joint>
   <!-- Door section-->

Commit message: Adding faceplate.

File: urdf/merlin_mockup.urdf.xacro (robot description, xacro)
@@ -17,4 +17,21 @@
     </collision>
   </link>
+  <link name="csm_faceplate_cover">
+    <visual>
+      <geometry>
+        <mesh filename="package://merlin_mockup_description/meshes/visual/csm_faceplate_cover.stl"/>
+      </geometry>
+    </visual>
+    <collision>
+      <geometry>
+        <mesh filename="package://merlin_mockup_description/meshes/visual/csm_faceplate_cover.stl"/>
+      </geometry>
+    </collision>
+  </link>
+  <joint name="faceplate_cover_joint" type="fixed">
+    <parent link="wood_frame"/>
+    <child link="csm_faceplate_cover"/>
+    <origin xyz="0.0 0.013 0.0" rpy="${pi/2} 0 ${pi}"/>
+  </joint>
   <!-- Velcro section-->
   <link name="velcro"> <!-- need to set all values -->

Commit message: adjusted the velcro to be on the outside of the newly added faceplate

File: urdf/merlin_mockup.urdf.xacro (robot description, xacro)
@@ -53,5 +53,5 @@
     <parent link="wood_frame"/>
     <child link="velcro"/>
-    <origin xyz="-0.17535 0.012 0.2345" rpy="0 0 0"/>
+    <origin xyz="-0.17535 0.015 0.2345" rpy="0 0 0"/>
   </joint>
   <!-- Door section-->
@@ -73,5 +73,5 @@
     <parent link="wood_frame"/>
     <child link="door"/>
-    <origin xyz="0 0.0125 -0.113" rpy="0 0 0"/>
+    <origin xyz="0 0.0255 -0.113" rpy="0 0 0"/>
     <axis xyz="1 0 0" />
     <limit effort="10" velocity="10" lower="-${pi/2}" upper="0"/>

Commit message: Adding door_face to merlin description for perception

File: urdf/merlin_mockup.urdf.xacro (robot description, xacro)
@@ -33,4 +33,11 @@
     <child link="csm_faceplate_cover"/>
     <origin xyz="0.0 0.013 0.0" rpy="${pi/2} 0 ${pi}"/>
+  </joint>
+  <link name="door_face">
+  </link>
+  <joint name="door_face" type="fixed">
+    <parent link="csm_faceplate_cover"/>
+    <child link="door_face"/>
+    <origin xyz="0.0 0.0 0.0381" rpy="0 0 0"/>
   </joint>
   <!-- Velcro section-->

Commit message: added seal and corners of seal

File: urdf/merlin_mockup.urdf.xacro (robot description, xacro)
@@ -41,4 +41,103 @@
     <origin xyz="0.0 0.0 0.0381" rpy="0 0 0"/>
   </joint>
+  <!-- Seal section-->
+  <!-- Replace visual and collision components of this link with stl eventually-->
+  <link name="seal">
+    <!-- Right-->
+    <visual>
+      <geometry>
+        <box size="0.0091 0.201 0.005"/>
+      </geometry>
+      <material name="Cyan">
+        <color rgba="0.0 0.0 0.0 1.0"/>
+      </material>
+      <origin rpy ="0 0 0" xyz ="0.1554 0 0.0025"/>
+    </visual>
+    <collision>
+      <geometry>
+        <box size="0.0091 0.201 0.005"/>
+      </geometry>
+      <origin rpy ="0 0 0" xyz ="0.1554 0 0.0025"/>
+    </collision>
+    <!-- Left -->
+    <visual>
+      <geometry>
+        <box size="0.0091 0.201 0.005"/>
+      </geometry>
+      <material name="Cyan">
+        <color rgba="0.0 0.0 0.0 1.0"/>
+      </material>
+      <origin rpy ="0 0 0" xyz ="-0.1554 0 0.0025"/>
+    </visual>
+    <collision>
+      <geometry>
+        <box size="0.0091 0.201 0.005"/>
+      </geometry>
+      <origin rpy ="0 0 0" xyz ="-0.1554 0 0.0025"/>
+    </collision>
+    <!-- Top-->
+    <visual>
+      <geometry>
+        <box size="0.302 0.0091 0.005"/>
+      </geometry>
+      <material name="Cyan">
+        <color rgba="0.0 0.0 0.0 1.0"/>
+      </material>
+      <origin xyz="0 0.1045 0.0025" rpy="0 0 0"/>
+    </visual>
+    <collision>
+      <geometry>
+        <box size="0.302 0.0091 0.005"/>
+      </geometry>
+      <origin xyz="0 0.1045 0.0025" rpy="0 0 0"/>
+    </collision>
+    <!-- Bottom -->
+    <visual>
+      <geometry>
+        <box size="0.302 0.0091 0.005"/>
+      </geometry>
+      <material name="Cyan">
+        <color rgba="0.0 0.0 0.0 1.0"/>
+      </material>
+      <origin xyz="0 -0.1045 0.0025" rpy="0 0 0"/>
+    </visual>
+    <collision>
+      <geometry>
+        <box size="0.302 0.0091 0.005"/>
+      </geometry>
+      <origin xyz="0 -0.1045 0.0025" rpy="0 0 0"/>
+    </collision>
+  </link>
+  <joint name="seal_to_face_joint" type="fixed">
+    <parent link="csm_faceplate_cover"/>
+    <child link="seal"/>
+    <!-- Seal does not appear to be perfectly centered - introduce offsets -->
+    <origin xyz="-0.001 -0.0015 0" rpy="0 0 0"/>
+  </joint>
+  <!-- Seal corners to help with cartesian waypoints - keep and modify these once above geometry is replaced with an stl -->
+  <link name="seal_corner_1"/>
+  <joint name="c1_to_seal" type="fixed">
+    <parent link="seal"/>
+    <child link="seal_corner_1"/>
+    <origin rpy ="-1.57 1.57 0" xyz ="-0.1554 0.1005 0.005"/>
+  </joint>
+  <link name="seal_corner_2"/>
+  <joint name="c2_to_seal" type="fixed">
+    <parent link="seal"/>
+    <child link="seal_corner_2"/>
+    <origin rpy ="-1.57 1.57 0" xyz ="0.1554 0.1005 0.005"/>
+  </joint>
+  <link name="seal_corner_3"/>
+  <joint name="c3_to_seal" type="fixed">
+    <parent link="seal"/>
+    <child link="seal_corner_3"/>
+    <origin rpy ="-1.57 1.57 0" xyz ="0.1554 -0.1005 0.005"/>
+  </joint>
+  <link name="seal_corner_4"/>
+  <joint name="c4_to_seal" type="fixed">
+    <parent link="seal"/>
+    <child link="seal_corner_4"/>
+    <origin rpy ="-1.57 1.57 0" xyz ="-0.1554 -0.1005 0.005"/>
+  </joint>
   <!-- Velcro section-->
   <link name="velcro"> <!-- need to set all values -->

Commit message: pushed points out based on perception stuff

File: urdf/merlin_mockup.urdf.xacro (robot description, xacro)
@@ -120,5 +120,5 @@
     <parent link="seal"/>
     <child link="seal_corner_1"/>
-    <origin rpy ="-1.57 1.57 0" xyz ="-0.1554 0.1005 0.005"/>
+    <origin rpy ="-1.57 1.57 0" xyz ="-0.1554 0.1105 0.005"/>
   </joint>
   <link name="seal_corner_2"/>
@@ -126,5 +126,5 @@
     <parent link="seal"/>
     <child link="seal_corner_2"/>
-    <origin rpy ="-1.57 1.57 0" xyz ="0.1554 0.1005 0.005"/>
+    <origin rpy ="-1.57 1.57 0" xyz ="0.1654 0.1105 0.005"/>
   </joint>
   <link name="seal_corner_3"/>
@@ -132,5 +132,5 @@
     <parent link="seal"/>
     <child link="seal_corner_3"/>
-    <origin rpy ="-1.57 1.57 0" xyz ="0.1554 -0.1005 0.005"/>
+    <origin rpy ="-1.57 1.57 0" xyz ="0.1654 -0.1005 0.005"/>
   </joint>
   <link name="seal_corner_4"/>
