Commit message: updating for default mass properties

File: urdf/merlin_mockup.xacro (robot description, xacro)
@@ -55,4 +55,9 @@
   <!-- Replace visual and collision components of this link with stl eventually-->
   <link name="${prefix}seal">
+    <inertial>
+      <origin rpy="0 0 0" xyz="0.0 0.0 0.0"/>
+      <mass value="0.1"/>
+      <inertia ixx="0.01" ixy="0.0" ixz="0.0" iyy="0.01" iyz="0.0" izz="0.01"/>
+    </inertial>
     <!-- Right-->
     <visual>
@@ -174,4 +179,9 @@
   <!-- Door section-->
   <link name="${prefix}door">
+    <inertial>
+      <origin rpy="0 0 0" xyz="0.0 0.0 0.0"/>
+      <mass value="0.1"/>
+      <inertia ixx="0.01" ixy="0.0" ixz="0.0" iyy="0.01" iyz="0.0" izz="0.01"/>
+    </inertial>
     <visual>
       <origin xyz="0 0 0.110" rpy="${pi/2} 0 ${pi}"/>
@@ -199,4 +209,9 @@
   <!-- Latch housing section-->
   <link name="${prefix}latch_housing">
+    <inertial>
+      <origin rpy="0 0 0" xyz="0.0 0.0 0.0"/>
+      <mass value="0.1"/>
+      <inertia ixx="0.01" ixy="0.0" ixz="0.0" iyy="0.01" iyz="0.0" izz="0.01"/>
+    </inertial>
     <visual>
       <origin xyz="0 0 0" rpy="0 ${pi} 0"/>
@@ -222,4 +237,9 @@
   <!-- Latch cover section-->
   <link name="${prefix}latch_cover">
+    <inertial>
+      <origin rpy="0 0 0" xyz="0.0 0.0 0.0"/>
+      <mass value="0.1"/>
+      <inertia ixx="0.01" ixy="0.0" ixz="0.0" iyy="0.01" iyz="0.0" izz="0.01"/>
+    </inertial>
     <visual>
       <origin xyz="0 0 0" rpy="0 0 0"/>
@@ -245,4 +265,9 @@
   <!-- Right latch pull section-->
   <link name="${prefix}right_latch_pull">
+    <inertial>
+      <origin rpy="0 0 0" xyz="0.0 0.0 0.0"/>
+      <mass value="0.1"/>
+      <inertia ixx="0.01" ixy="0.0" ixz="0.0" iyy="0.01" iyz="0.0" izz="0.01"/>
+    </inertial>
     <visual>
       <origin xyz="0 0 0" rpy="${pi} -${pi/2} -${pi/2}"/>
@@ -270,4 +295,9 @@
   <!-- Left latch pull section-->
   <link name="${prefix}left_latch_pull">
+    <inertial>
+      <origin rpy="0 0 0" xyz="0.0 0.0 0.0"/>
+      <mass value="0.1"/>
+      <inertia ixx="0.01" ixy="0.0" ixz="0.0" iyy="0.01" iyz="0.0" izz="0.01"/>
+    </inertial>
     <visual>
       <origin xyz="0 0 0" rpy="0 ${pi/2} -${pi/2}"/>
@@ -295,4 +325,9 @@
   <!-- Latch lock section-->
   <link name="${prefix}latch_lock">
+    <inertial>
+      <origin rpy="0 0 0" xyz="0.0 0.0 0.0"/>
+      <mass value="0.1"/>
+      <inertia ixx="0.01" ixy="0.0" ixz="0.0" iyy="0.01" iyz="0.0" izz="0.01"/>
+    </inertial>
     <visual>
       <origin xyz="0 0.0012 -0.0084" rpy="0 0 0"/>

Commit message: add latch collision geometry

File: urdf/merlin_mockup.xacro (robot description, xacro)
@@ -208,4 +208,10 @@
       </material>
     </visual>
+    <collision>
+       <origin xyz="0 0 0" rpy="0 ${pi} 0"/>
+      <geometry>
+        <mesh filename="package://merlin_mockup_description/meshes/visual/csm_latch_housing.stl"/>
+      </geometry>
+    </collision>
   </link>
   <joint name="${prefix}door_to_latch" type="fixed">
@@ -225,4 +231,10 @@
       </material>
     </visual>
+    <collision>
+      <origin xyz="0 0 0" rpy="0 0 0"/>
+      <geometry>
+        <mesh filename="package://merlin_mockup_description/meshes/visual/csm_latch_cover.stl"/>
+      </geometry>
+    </collision>
   </link>
   <joint name="${prefix}housing_to_cover" type="fixed">
@@ -242,4 +254,10 @@
       </material>
     </visual>
+    <collision>
+      <origin xyz="0 0 0" rpy="${pi} -${pi/2} -${pi/2}"/>
+      <geometry>
+        <mesh filename="package://merlin_mockup_description/meshes/visual/csm_latch_pull.stl"/>
+      </geometry>
+    </collision>
   </link>
   <joint name="${prefix}housing_to_right_latch_pull" type="prismatic">
@@ -261,4 +279,10 @@
       </material>
     </visual>
+    <collision>
+      <origin xyz="0 0 0" rpy="0 ${pi/2} -${pi/2}"/>
+      <geometry>
+        <mesh filename="package://merlin_mockup_description/meshes/visual/csm_latch_pull.stl"/>
+      </geometry>
+    </collision>
   </link>
   <joint name="${prefix}housing_to_left_latch_pull" type="prismatic">
@@ -280,4 +304,10 @@
       </material>
     </visual>
+    <collision>
+      <origin xyz="0 0.0012 -0.0084" rpy="0 0 0"/>
+      <geometry>
+        <mesh filename="package://merlin_mockup_description/meshes/visual/csm_latch_lock.stl"/>
+      </geometry>
+    </collision>
   </link>
   <joint name="${prefix}housing_to_latch_lock" type="revolute">
