Commit message: Switching to a lower fidelity collision mesh.

File: hatch_4060/urdf/hatch_4060.urdf.xacro (robot description, xacro)
@@ -4,7 +4,7 @@
   <xacro:arg name="prefix" default=""/>
   <xacro:property name="external_handle_1" default="true"/>
-  <xacro:property name="external_handle_2" default="false"/>
+  <xacro:property name="external_handle_2" default="true"/>
   <xacro:property name="internal_handle_1" default="true"/>
-  <xacro:property name="internal_handle_2" default="false"/>
+  <xacro:property name="internal_handle_2" default="true"/>
   <xacro:include filename="$(find hatch_frame)/urdf/hatch_frame.xacro"/>
   <xacro:include filename="$(find hatch_frame)/urdf/colors.xacro"/>

File: hatch_4060/urdf/hatch_4060.xacro (robot description, xacro)
@@ -61,5 +61,5 @@
         <origin xyz="0.0 0.0 0.0" rpy="0 0 0"/>
         <geometry>
-          <mesh filename="file://$(find hatch_4060)/meshes/collision/hatch_4060_face_no_handles.stl"/>
+          <mesh filename="file://$(find hatch_4060)/meshes/collision/hatch_4060_collision.stl"/>
         </geometry>
         <material name="red"/>

Commit message: Cleanup

File: hatch_4060/urdf/hatch_4060.urdf.xacro (robot description, xacro)
@@ -4,7 +4,7 @@
   <xacro:arg name="prefix" default=""/>
   <xacro:property name="external_handle_1" default="true"/>
-  <xacro:property name="external_handle_2" default="true"/>
+  <xacro:property name="external_handle_2" default="false"/>
   <xacro:property name="internal_handle_1" default="true"/>
-  <xacro:property name="internal_handle_2" default="true"/>
+  <xacro:property name="internal_handle_2" default="false"/>
   <xacro:include filename="$(find hatch_frame)/urdf/hatch_frame.xacro"/>
   <xacro:include filename="$(find hatch_frame)/urdf/colors.xacro"/>

Commit message: updating x value of origin of xacro call

File: hatch_4060/urdf/hatch_4060.urdf.xacro (robot description, xacro)
@@ -18,5 +18,5 @@
     external_handle_1="${external_handle_1}" external_handle_2="${external_handle_2}"
     internal_handle_1="${internal_handle_1}" internal_handle_2="${internal_handle_2}">
-    <origin xyz="0.668 0.06 0.7113" rpy="0 0 0"/>
+    <origin xyz="0.669329 0.06 0.7113" rpy="0 0 0"/>
   </xacro:hatch_4060>
 </robot>

Commit message: Updating 4060 hatch to keep joint names consistent between hatches.

File: hatch_4060/urdf/hatch_4060.urdf.xacro (robot description, xacro)
@@ -15,8 +15,8 @@
     <origin xyz="0 0 0" rpy="0 0 0"/>
   </xacro:hatch_frame>
-  <xacro:hatch_4060 name="$(arg name)" prefix="$(arg prefix)" parent="hatch_frame"
+  <xacro:hatch name="$(arg name)" prefix="$(arg prefix)" parent="hatch_frame"
     external_handle_1="${external_handle_1}" external_handle_2="${external_handle_2}"
     internal_handle_1="${internal_handle_1}" internal_handle_2="${internal_handle_2}">
     <origin xyz="0.669329 0.06 0.7113" rpy="0 0 0"/>
-  </xacro:hatch_4060>
+  </xacro:hatch>
 </robot>

File: hatch_4060/urdf/hatch_4060.xacro (robot description, xacro)
@@ -1,5 +1,5 @@
 <?xml version="1.0"?>
 <robot xmlns:xacro="http://wiki.ros.org/xacro">
-  <xacro:macro name="hatch_4060" params="
+  <xacro:macro name="hatch" params="
     name:=''
     prefix:=''
@@ -10,10 +10,10 @@
     internal_handle_1:='false'
     internal_handle_2:='false'">
-    <joint name="${prefix}hatch_4060_frame_joint" type="fixed">
+    <joint name="${prefix}hatch_outer_frame_joint" type="fixed">
       <parent link="${prefix}${parent}"/>
-      <child link="${prefix}hatch_4060_frame"/>
+      <child link="${prefix}hatch_outer_frame"/>
       <xacro:insert_block name="origin"/>
     </joint>
-    <link name="${prefix}hatch_4060_frame">
+    <link name="${prefix}hatch_outer_frame">
       <!--TODO set proper inertia-->
       <inertial>
@@ -37,12 +37,12 @@
       </collision>
     </link>
-    <joint name="${prefix}hatch_4060_frame_face_joint" type="revolute">
+    <joint name="${prefix}hatch_frame_face_joint" type="revolute">
       <axis xyz="0 0 1"/>
       <limit effort="10.0" lower="0.0" upper="3.14" velocity="0.5"/>
-      <parent link="${prefix}hatch_4060_frame"/>
-      <child link="${prefix}hatch_4060_face"/>
+      <parent link="${prefix}hatch_outer_frame"/>
+      <child link="${prefix}hatch_face"/>
       <origin xyz="0.0827 1.21379 0.0457" rpy="0 0 0"/>
     </joint>
-    <link name="${prefix}hatch_4060_face">
+    <link name="${prefix}hatch_face">
       <!--TODO set proper inertia-->
       <inertial>
@@ -68,5 +68,5 @@
     </link>
     <joint name="${prefix}right_cal_1_joint" type="fixed">
-      <parent link="${prefix}hatch_4060_face"/>
+      <parent link="${prefix}hatch_face"/>
       <child link="${prefix}right_cal_1_frame"/>
       <origin xyz="0.0167 0.0 0.0" rpy="0 0 0"/>
@@ -74,5 +74,5 @@
     <link name="${prefix}right_cal_1_frame"/>
     <joint name="${prefix}right_cal_2_joint" type="fixed">
-      <parent link="${prefix}hatch_4060_face"/>
+      <parent link="${prefix}hatch_face"/>
       <child link="${prefix}right_cal_2_frame"/>
       <origin xyz="0.0 0.0167 0.0" rpy="0 0 0"/>
@@ -81,8 +81,8 @@
     <xacro:include filename="$(find hatch_accessories)/urdf/crank_wheel.xacro"/>
     <!--TODO are the centers located properly?-->
-    <xacro:crank_wheel name="$(arg name)" prefix="$(arg prefix)external_" parent="${prefix}hatch_4060_face">
+    <xacro:crank_wheel name="$(arg name)" prefix="$(arg prefix)external_" parent="${prefix}hatch_face">
       <origin xyz="0.04431 -0.9474 0.4295" rpy="0 ${pi/2} 0"/>
     </xacro:crank_wheel>
-    <xacro:crank_wheel name="$(arg name)" prefix="$(arg prefix)internal_" parent="${prefix}hatch_4060_face">
+    <xacro:crank_wheel name="$(arg name)" prefix="$(arg prefix)internal_" parent="${prefix}hatch_face">
       <origin xyz="-0.17161 -0.9474 0.4295" rpy="0 -${pi/2} 0"/>
     </xacro:crank_wheel>
@@ -90,20 +90,20 @@
     <!--TODO which handles are mounted?-->
     <xacro:if value="${external_handle_1}">
-      <xacro:grab_handle name="$(arg name)" prefix="$(arg prefix)external_1_" parent="${prefix}hatch_4060_face">
+      <xacro:grab_handle name="$(arg name)" prefix="$(arg prefix)external_1_" parent="${prefix}hatch_face">
         <origin xyz="-0.0573 -0.9016 0.7357" rpy="0 0 0"/>
       </xacro:grab_handle>
     </xacro:if>
     <xacro:if value="${external_handle_2}">
-      <xacro:grab_handle name="$(arg name)" prefix="$(arg prefix)external_2_" parent="${prefix}hatch_4060_face">
+      <xacro:grab_handle name="$(arg name)" prefix="$(arg prefix)external_2_" parent="${prefix}hatch_face">
         <origin xyz="-0.0497 -1.078 0.6957" rpy="${pi/2} 0 0"/>
       </xacro:grab_handle>
     </xacro:if>
     <xacro:if value="${internal_handle_1}">
-      <xacro:grab_handle name="$(arg name)" prefix="$(arg prefix)internal_1_" parent="${prefix}hatch_4060_face">
+      <xacro:grab_handle name="$(arg name)" prefix="$(arg prefix)internal_1_" parent="${prefix}hatch_face">
         <origin xyz="-0.07 -0.9016 0.7957" rpy="0 ${pi} 0"/>
       </xacro:grab_handle>
     </xacro:if>
     <xacro:if value="${internal_handle_2}">
-      <xacro:grab_handle name="$(arg name)" prefix="$(arg prefix)internal_2_" parent="${prefix}hatch_4060_face">
+      <xacro:grab_handle name="$(arg name)" prefix="$(arg prefix)internal_2_" parent="${prefix}hatch_face">
         <origin xyz="-0.0776 -1.0293 0.6957" rpy="${-pi/2} ${pi} 0"/>
       </xacro:grab_handle>

Commit message: Additions after recieving hardware.

File: hatch_4060/urdf/hatch_4060.urdf.xacro (robot description, xacro)
@@ -4,8 +4,8 @@
   <xacro:arg name="prefix" default=""/>
   <!--TODO which handles are mounted?-->
-  <xacro:property name="external_handle_1" default="true"/>
+  <xacro:property name="external_handle_1" default="false"/>
   <xacro:property name="external_handle_2" default="false"/>
   <xacro:property name="internal_handle_1" default="true"/>
-  <xacro:property name="internal_handle_2" default="false"/>
+  <xacro:property name="internal_handle_2" default="true"/>
   <xacro:include filename="$(find hatch_accessories)/urdf/hatch_frame.xacro"/>
   <xacro:include filename="$(find hatch_accessories)/urdf/colors.xacro"/>

File: hatch_4060/urdf/hatch_4060.xacro (robot description, xacro)
@@ -101,5 +101,5 @@
     <xacro:if value="${internal_handle_1}">
       <xacro:grab_handle name="$(arg name)" prefix="$(arg prefix)internal_1_" parent="${prefix}hatch_face">
-        <origin xyz="-0.0573 -0.9016 0.7357" rpy="0 0 0"/>
+        <origin xyz="-0.0573 -0.9016 0.7971" rpy="0 0 0"/>
       </xacro:grab_handle>
     </xacro:if>

Commit message: Changes for calibrating the exterior handle and wheel.

File: hatch_4060/urdf/hatch_4060.urdf.xacro (robot description, xacro)
@@ -4,6 +4,6 @@
   <xacro:arg name="prefix" default=""/>
   <!--TODO which handles are mounted?-->
-  <xacro:property name="external_handle_1" default="false"/>
-  <xacro:property name="external_handle_2" default="false"/>
+  <xacro:property name="external_handle_1" default="true"/>
+  <xacro:property name="external_handle_2" default="true"/>
   <xacro:property name="internal_handle_1" default="true"/>
   <xacro:property name="internal_handle_2" default="true"/>

File: hatch_4060/urdf/hatch_4060.xacro (robot description, xacro)
@@ -91,10 +91,10 @@
     <xacro:if value="${external_handle_1}">
       <xacro:grab_handle name="$(arg name)" prefix="$(arg prefix)external_1_" parent="${prefix}hatch_face">
-        <origin xyz="-0.07 -0.9016 0.7957" rpy="0 ${pi} 0"/>
+        <origin xyz="-0.07 -0.9016 0.7357" rpy="0 ${pi} 0"/>
       </xacro:grab_handle>
     </xacro:if>
     <xacro:if value="${external_handle_2}">
       <xacro:grab_handle name="$(arg name)" prefix="$(arg prefix)external_2_" parent="${prefix}hatch_face">
-        <origin xyz="-0.0776 -1.0293 0.6957" rpy="${-pi/2} ${pi} 0"/>
+        <origin xyz="-0.07 -1.0293 0.6957" rpy="${-pi/2} ${pi} 0"/>
       </xacro:grab_handle>
     </xacro:if>

Commit message: Adding a hatch level bench.

File: hatch_4060/urdf/hatch_4060.urdf.xacro (robot description, xacro)
@@ -6,4 +6,5 @@
   <xacro:property name="external_handle_1" default="true"/>
   <xacro:property name="external_handle_2" default="true"/>
+  <xacro:property name="external_handle_3" default="true"/>
   <xacro:property name="internal_handle_1" default="true"/>
   <xacro:property name="internal_handle_2" default="true"/>
@@ -16,5 +17,5 @@
   </xacro:hatch_frame>
   <xacro:hatch name="$(arg name)" prefix="$(arg prefix)" parent="hatch_frame"
-    external_handle_1="${external_handle_1}" external_handle_2="${external_handle_2}"
+    external_handle_1="${external_handle_1}" external_handle_2="${external_handle_2}" external_handle_3="${external_handle_3}"
     internal_handle_1="${internal_handle_1}" internal_handle_2="${internal_handle_2}">
     <origin xyz="0.669329 0.06 0.7113" rpy="0 0 0"/>

File: hatch_accessories/urdf/hatch_frame.xacro (robot description, xacro)
@@ -130,4 +130,27 @@
     </joint>
     <link name="${prefix}hatch_frame_front_top"/>
+    <!--This is for when there is a bench at the level of the bottom of the hatch opening.-->
+    <!-- TODO add if statement -->
+    <joint name="${prefix}hatch_frame_bench_joint" type="fixed">
+      <parent link="${prefix}hatch_frame"/>
+      <child link="${prefix}hatch_bench"/>
+      <origin xyz="0.0 0.0 0.0" rpy="0 0 0"/>
+    </joint>
+    <link name="${prefix}hatch_bench">
+      <visual>
+        <origin xyz="${0.675/2} ${1.307/2} ${0.4953/2}" rpy="0 0 0"/>
+        <geometry>
+          <box size="0.675 1.307 0.4953"/>
+        </geometry>
+        <material name="gray"/>
+      </visual>
+      <collision>
+        <origin xyz="${0.675/2} ${1.307/2} ${0.4953/2}" rpy="0 0 0"/>
+        <geometry>
+          <box size="0.675 1.307 0.4953"/>
+        </geometry>
+        <material name="gray"/>
+      </collision>
+    </link>
   </xacro:macro>
 </robot>

Commit message: added links and joints for sim latch in hatch_4060 xacro macro

File: hatch_4060/urdf/hatch_4060.urdf.xacro (robot description, xacro)
@@ -8,4 +8,5 @@
   <xacro:property name="internal_handle_1" default="true"/>
   <xacro:property name="internal_handle_2" default="true"/>
+  <xacro:property name="latch" default="true"/>
   <xacro:include filename="$(find hatch_accessories)/urdf/hatch_frame.xacro"/>
   <xacro:include filename="$(find hatch_accessories)/urdf/colors.xacro"/>
@@ -17,5 +18,5 @@
   <xacro:hatch_4060 prefix="$(arg prefix)" parent="hatch_frame"
     external_handle_1="${external_handle_1}" external_handle_2="${external_handle_2}" external_handle_3="${external_handle_3}"
-    internal_handle_1="${internal_handle_1}" internal_handle_2="${internal_handle_2}">
+    internal_handle_1="${internal_handle_1}" internal_handle_2="${internal_handle_2}" latch="${latch}">
     <origin xyz="0.669329 0.06 0.7113" rpy="0 0 0"/>
   </xacro:hatch_4060>

File: hatch_4060/urdf/hatch_4060.xacro (robot description, xacro)
@@ -9,5 +9,6 @@
     external_handle_3:='false'
     internal_handle_1:='false'
-    internal_handle_2:='false'">
+    internal_handle_2:='false'
+    latch:='false'">
     <joint name="${prefix}hatch_inner_frame_joint" type="fixed">
       <parent link="${parent}"/>
@@ -95,4 +96,57 @@
       </collision>
     </link>
+    <!-- sim latch -->
+    <xacro:if value="${latch}">
+      <joint name="${prefix}hatch_outer_frame_to_latch_spring_anchor" type="fixed">
+        <origin xyz="${1.844*0.0254+0.022} ${-0.688*0.0254+0.0017} ${23.688*0.0254}" rpy="0 0 0"/>
+        <parent link="${prefix}hatch_outer_frame"/>
+        <child link="${prefix}hatch_latch_spring_anchor"/>
+      </joint>
+      <link name="${prefix}hatch_latch_spring_anchor"/>
+      <joint name="${prefix}latch_spring" type="prismatic">
+        <origin xyz="0 0 0" rpy="0 0 0"/>
+        <parent link="${prefix}hatch_latch_spring_anchor"/>
+        <child link="${prefix}hatch_latch_catch"/>
+        <axis xyz="0 0 -1"/>
+        <limit lower="0.0" upper="0.027" effort="1000" velocity="1000"/>
+      </joint>
+      <link name="${prefix}hatch_latch_catch">
+        <inertial>
+          <mass value="0.0671"/>
+          <inertia ixx="4.345e-6" ixy="0.0" ixz="0.0" iyy="4.345e-6" iyz="0.0" izz="4.345e-6"/>
+        </inertial>
+        <visual>
+          <geometry>
+            <sphere radius="${0.5*0.0254}"/>
+          </geometry>
+        </visual>
+        <collision>
+          <geometry>
+            <sphere radius="${0.5*0.0254}"/>
+          </geometry>
+        </collision>
+      </link>
+      <joint name="${prefix}hatch_face_to_latch" type="fixed">
+        <parent link="${prefix}hatch_face"/>
+        <child link="${prefix}hatch_latch"/>
+        <origin xyz="${-1.34483*0.0254} ${-48.3955*0.0254} ${20.2293*0.0254}" rpy="0 0 0"/>
+      </joint>
+      <link name="${prefix}hatch_latch">
+        <inertial>
+          <mass value="0.0671"/>
+          <inertia ixx="4.345e-6" ixy="0.0" ixz="0.0" iyy="4.345e-6" iyz="0.0" izz="4.345e-6"/>
+        </inertial>
+        <visual>
+          <geometry>
+            <sphere radius="${0.5*0.0254}"/>
+          </geometry>
+        </visual>
+        <collision>
+          <geometry>
+            <sphere radius="${0.5*0.0254}"/>
+          </geometry>
+        </collision>
+      </link>
+    </xacro:if>
     <joint name="${prefix}right_cal_1_joint" type="fixed">
       <parent link="${prefix}hatch_face"/>
