Commit message: Updating the crank wheel housing.

File: hatch_4060/urdf/hatch_4060.xacro (robot description, xacro)
@@ -54,5 +54,5 @@
         <origin xyz="0.0 0.0 0.0" rpy="0 0 0"/>
         <geometry>
-          <mesh filename="file://$(find hatch_4060)/meshes/visual/hatch_4060_face_no_handles.stl"/>
+          <mesh filename="file://$(find hatch_4060)/meshes/visual/hatch_4060_face.stl"/>
         </geometry>
         <material name="gray"/>

File: hatch_frame/urdf/crank_wheel.xacro (robot description, xacro)
@@ -37,5 +37,5 @@
     </link>
     <joint name="${prefix}rotary_handle_joint" type="revolute">
-      <axis xyz="0 -1 0"/>
+      <axis xyz="1 0 0"/>
       <!--This is continuously rotatable-->
       <limit effort="10.0" lower="0.0" upper="1.57" velocity="0.5"/>

Commit message: fixing x and y location for hatch__4060_frame_joint

File: hatch_4060/urdf/hatch_4060.xacro (robot description, xacro)
@@ -42,5 +42,5 @@
       <parent link="${prefix}hatch_4060_frame"/>
       <child link="${prefix}hatch_4060_face"/>
-      <origin xyz="0.0817 1.215 0.0457" rpy="0 0 0"/>
+      <origin xyz="0.0827 1.21379 0.0457" rpy="0 0 0"/>
     </joint>
     <link name="${prefix}hatch_4060_face">

Commit message: adjusting x value of external handle

File: hatch_4060/urdf/hatch_4060.xacro (robot description, xacro)
@@ -79,5 +79,5 @@
     <xacro:if value="${external_handle_1}">
       <xacro:grab_handle name="$(arg name)" prefix="$(arg prefix)external_1_" parent="${prefix}hatch_4060_face">
-        <origin xyz="-0.0497 -0.9016 0.7357" rpy="0 0 0"/>
+        <origin xyz="-0.0573 -0.9016 0.7357" rpy="0 0 0"/>
       </xacro:grab_handle>
     </xacro:if>

Commit message: adjusting x value of internal handle

File: hatch_4060/urdf/hatch_4060.xacro (robot description, xacro)
@@ -89,5 +89,5 @@
     <xacro:if value="${internal_handle_1}">
       <xacro:grab_handle name="$(arg name)" prefix="$(arg prefix)internal_1_" parent="${prefix}hatch_4060_face">
-        <origin xyz="-0.0776 -0.9016 0.7957" rpy="0 ${pi} 0"/>
+        <origin xyz="-0.07 -0.9016 0.7957" rpy="0 ${pi} 0"/>
       </xacro:grab_handle>
     </xacro:if>

Commit message: crank wheel x values

File: hatch_4060/urdf/hatch_4060.xacro (robot description, xacro)
@@ -70,8 +70,8 @@
     <!--TODO are the centers located properly?-->
     <xacro:crank_wheel name="$(arg name)" prefix="$(arg prefix)external_" parent="${prefix}hatch_4060_face">
-      <origin xyz="0.0522475 -0.9474 0.4295" rpy="0 ${pi/2} 0"/>
+      <origin xyz="0.04431 -0.9474 0.4295" rpy="0 ${pi/2} 0"/>
     </xacro:crank_wheel>
     <xacro:crank_wheel name="$(arg name)" prefix="$(arg prefix)internal_" parent="${prefix}hatch_4060_face">
-      <origin xyz="-0.1795475 -0.9474 0.4295" rpy="0 -${pi/2} 0"/>
+      <origin xyz="-0.17161 -0.9474 0.4295" rpy="0 -${pi/2} 0"/>
     </xacro:crank_wheel>
     <xacro:include filename="$(find hatch_accessories)/urdf/grab_handle.xacro"/>

Commit message: Joint name bug fix.

File: hatch_4060/urdf/hatch_4060.xacro (robot description, xacro)
@@ -37,5 +37,5 @@
       </collision>
     </link>
-    <joint name="${prefix}hatch_frame_face_joint" type="revolute">
+    <joint name="${prefix}hatch_outer_frame_face_joint" type="revolute">
       <axis xyz="0 0 1"/>
       <limit effort="10.0" lower="0.0" upper="3.14" velocity="0.5"/>

Commit message: Calibration changes for the 4060 hatch.

File: hatch_4060/urdf/hatch_4060.xacro (robot description, xacro)
@@ -8,6 +8,6 @@
     external_handle_1:='false'
     external_handle_2:='false'
-    internal_handle_1:='true'
-    internal_handle_2:='true'">
+    internal_handle_1:='false'
+    internal_handle_2:='false'">
     <joint name="${prefix}hatch_outer_frame_joint" type="fixed">
       <parent link="${prefix}${parent}"/>
@@ -82,8 +82,8 @@
     <!--TODO are the centers located properly?-->
     <xacro:crank_wheel name="$(arg name)" prefix="$(arg prefix)external_" parent="${prefix}hatch_face">
-      <origin xyz="-0.17161 -0.9474 0.4295" rpy="0 -${pi/2} 0"/>
+      <origin xyz="-0.17161 -0.9474 0.4265" rpy="0 -${pi/2} 0"/>
     </xacro:crank_wheel>
     <xacro:crank_wheel name="$(arg name)" prefix="$(arg prefix)internal_" parent="${prefix}hatch_face">
-      <origin xyz="0.04431 -0.9474 0.4295" rpy="0 ${pi/2} 0"/>
+      <origin xyz="0.04431 -0.9474 0.4265" rpy="0 ${pi/2} 0"/>
     </xacro:crank_wheel>
     <xacro:include filename="$(find hatch_accessories)/urdf/grab_handle.xacro"/>
@@ -101,10 +101,10 @@
     <xacro:if value="${internal_handle_1}">
       <xacro:grab_handle name="$(arg name)" prefix="$(arg prefix)internal_1_" parent="${prefix}hatch_face">
-        <origin xyz="-0.0573 -0.9016 0.7971" rpy="0 0 0"/>
+        <origin xyz="-0.058 -0.9016 0.7971" rpy="0 0 0"/>
       </xacro:grab_handle>
     </xacro:if>
     <xacro:if value="${internal_handle_2}">
       <xacro:grab_handle name="$(arg name)" prefix="$(arg prefix)internal_2_" parent="${prefix}hatch_face">
-        <origin xyz="-0.0497 -1.078 0.6957" rpy="${pi/2} 0 0"/>
+        <origin xyz="-0.058 -1.078 0.6957" rpy="${pi/2} 0 0"/>
       </xacro:grab_handle>
     </xacro:if>

Commit message: Tweaks for calibrating the 4060 hatch enterior wheel.

File: hatch_4060/urdf/hatch_4060.xacro (robot description, xacro)
@@ -82,5 +82,5 @@
     <!--TODO are the centers located properly?-->
     <xacro:crank_wheel name="$(arg name)" prefix="$(arg prefix)external_" parent="${prefix}hatch_face">
-      <origin xyz="-0.17161 -0.9474 0.4265" rpy="0 -${pi/2} 0"/>
+      <origin xyz="-0.17161 -0.9474 0.4325" rpy="0 -${pi/2} 0"/>
     </xacro:crank_wheel>
     <xacro:crank_wheel name="$(arg name)" prefix="$(arg prefix)internal_" parent="${prefix}hatch_face">

Commit message: adding 7mm offset in y to external handle

File: hatch_4060/urdf/hatch_4060.xacro (robot description, xacro)
@@ -96,5 +96,5 @@
     <xacro:if value="${external_handle_2}">
       <xacro:grab_handle name="$(arg name)" prefix="$(arg prefix)external_2_" parent="${prefix}hatch_face">
-        <origin xyz="-0.07 -1.0293 0.6957" rpy="${-pi/2} ${pi} 0"/>
+        <origin xyz="-0.07 -1.0223 0.6957" rpy="${-pi/2} ${pi} 0"/>
       </xacro:grab_handle>
     </xacro:if>

Commit message: adding external handle 3 for the 4060 hatch

File: hatch_4060/urdf/hatch_4060.xacro (robot description, xacro)
@@ -8,4 +8,5 @@
     external_handle_1:='false'
     external_handle_2:='false'
+    external_handle_3:='false'
     internal_handle_1:='false'
     internal_handle_2:='false'">
@@ -99,4 +100,9 @@
       </xacro:grab_handle>
     </xacro:if>
+    <xacro:if value="${external_handle_3}">
+      <xacro:grab_handle name="$(arg name)" prefix="$(arg prefix)external_3_" parent="${prefix}hatch_face">
+        <origin xyz="-0.07 -0.145 0.6957" rpy="${-pi/2} ${pi} 0"/>
+      </xacro:grab_handle>
+    </xacro:if>
     <xacro:if value="${internal_handle_1}">
       <xacro:grab_handle name="$(arg name)" prefix="$(arg prefix)internal_1_" parent="${prefix}hatch_face">

Commit message: calibration of handles for EVR demo

File: hatch_4060/urdf/hatch_4060.xacro (robot description, xacro)
@@ -92,5 +92,5 @@
     <xacro:if value="${external_handle_1}">
       <xacro:grab_handle name="$(arg name)" prefix="$(arg prefix)external_1_" parent="${prefix}hatch_face">
-        <origin xyz="-0.07 -0.9016 0.7357" rpy="0 ${pi} 0"/>
+        <origin xyz="-0.07 -0.9016 0.7971" rpy="0 ${pi} 0"/>
       </xacro:grab_handle>
     </xacro:if>
@@ -102,5 +102,5 @@
     <xacro:if value="${external_handle_3}">
       <xacro:grab_handle name="$(arg name)" prefix="$(arg prefix)external_3_" parent="${prefix}hatch_face">
-        <origin xyz="-0.07 -0.145 0.6957" rpy="${-pi/2} ${pi} 0"/>
+        <origin xyz="-0.07 ${-0.145+0.0245} 0.6957" rpy="${-pi/2} ${pi} 0"/>
       </xacro:grab_handle>
     </xacro:if>

Commit message: adjusting external handle 3 for fine-tuned calibration

File: hatch_4060/urdf/hatch_4060.xacro (robot description, xacro)
@@ -102,5 +102,5 @@
     <xacro:if value="${external_handle_3}">
       <xacro:grab_handle name="$(arg name)" prefix="$(arg prefix)external_3_" parent="${prefix}hatch_face">
-        <origin xyz="-0.07 ${-0.145+0.0245} 0.6957" rpy="${-pi/2} ${pi} 0"/>
+        <origin xyz="-0.07 ${-0.145+0.0195} 0.6957" rpy="${-pi/2} ${pi} 0"/>
       </xacro:grab_handle>
     </xacro:if>

Commit message: Adding the mounting for what would be the interior hatch.

File: hatch_4060/urdf/hatch_4060.xacro (robot description, xacro)
@@ -11,4 +11,31 @@
     internal_handle_1:='false'
     internal_handle_2:='false'">
+    <joint name="${prefix}hatch_inner_frame_joint" type="fixed">
+      <parent link="${prefix}${parent}"/>
+      <child link="${prefix}hatch_inner_frame"/>
+      <origin xyz="0.584329 1.245 0.7113" rpy="0 0 ${pi}"/>
+    </joint>
+    <link name="${prefix}hatch_inner_frame">
+      <!--TODO set proper inertia-->
+      <inertial>
+        <origin rpy="0 0 0" xyz="0.0 0.0 0.0"/>
+        <mass value="0.0"/>
+        <inertia ixx="0.0" ixy="0.0" ixz="0.0" iyy="0.0" iyz="0.0" izz="0.0"/>
+      </inertial>
+      <visual>
+        <origin xyz="0.0 0.0 0.0" rpy="0 0 0"/>
+        <geometry>
+          <mesh filename="package://hatch_4060/meshes/visual/hatch_4060_frame.stl"/>
+        </geometry>
+        <material name="gray"/>
+      </visual>
+      <collision>
+        <origin xyz="0.0 0.0 0.0" rpy="0 0 0"/>
+        <geometry>
+          <mesh filename="package://hatch_4060/meshes/collision/hatch_4060_frame.stl"/>
+        </geometry>
+        <material name="red"/>
+      </collision>
+    </link>
     <joint name="${prefix}hatch_outer_frame_joint" type="fixed">
       <parent link="${prefix}${parent}"/>

Commit message: EVR stable shim hatch calibration

File: hatch_4060/urdf/hatch_4060.xacro (robot description, xacro)
@@ -92,15 +92,15 @@
     <xacro:if value="${external_handle_1}">
       <xacro:grab_handle name="$(arg name)" prefix="$(arg prefix)external_1_" parent="${prefix}hatch_face">
-        <origin xyz="-0.07 -0.9016 0.7971" rpy="0 ${pi} 0"/>
+        <origin xyz="-0.07 -0.9016 ${0.7971+0.005}" rpy="0 ${pi} 0"/>
       </xacro:grab_handle>
     </xacro:if>
     <xacro:if value="${external_handle_2}">
       <xacro:grab_handle name="$(arg name)" prefix="$(arg prefix)external_2_" parent="${prefix}hatch_face">
-        <origin xyz="-0.07 -1.0223 0.6957" rpy="${-pi/2} ${pi} 0"/>
+        <origin xyz="-0.07 ${-1.0223-0.005} ${0.6957 - 0.007}" rpy="${-pi/2} ${pi} 0"/>
       </xacro:grab_handle>
     </xacro:if>
     <xacro:if value="${external_handle_3}">
       <xacro:grab_handle name="$(arg name)" prefix="$(arg prefix)external_3_" parent="${prefix}hatch_face">
-        <origin xyz="-0.07 ${-0.145+0.0195} 0.6957" rpy="${-pi/2} ${pi} 0"/>
+        <origin xyz="${-0.07-0.005} ${-0.145+0.0195 - 0.004} 0.6957" rpy="${-pi/2} ${pi} 0"/>
       </xacro:grab_handle>
     </xacro:if>

Commit message: modifying external_handle_3 x dimension to match reality

File: hatch_4060/urdf/hatch_4060.xacro (robot description, xacro)
@@ -129,5 +129,5 @@
     <xacro:if value="${external_handle_3}">
       <xacro:grab_handle name="$(arg name)" prefix="${prefix}external_3_" parent="${prefix}hatch_face">
-        <origin xyz="${-0.07-0.005} ${-0.145+0.0195 - 0.004} 0.6957" rpy="${-pi/2} ${pi} 0"/>
+        <origin xyz="${-0.07} ${-0.145+0.0195 - 0.004} 0.6957" rpy="${-pi/2} ${pi} 0"/>
       </xacro:grab_handle>
     </xacro:if>

Commit message: Added mass properties to sim objects of interest.

File: hatch_4060/urdf/hatch_4060.xacro (robot description, xacro)
@@ -19,6 +19,6 @@
       <inertial>
         <origin rpy="0 0 0" xyz="0.0 0.0 0.0"/>
-        <mass value="0.1"/>
-        <inertia ixx="0.1" ixy="0.0" ixz="0.0" iyy="0.1" iyz="0.0" izz="0.1"/>
+        <mass value="7.381808"/>
+        <inertia ixx="8.9911" ixy="-0.050621" ixz="-0.0463501" iyy="4.691664" iyz="-2.297576" izz="4.302649"/>
       </inertial>
       <visual>
@@ -46,6 +46,6 @@
       <inertial>
         <origin rpy="0 0 0" xyz="0.0 0.0 0.0"/>
-        <mass value="0.1"/>
-        <inertia ixx="0.1" ixy="0.0" ixz="0.0" iyy="0.1" iyz="0.0" izz="0.1"/>
+        <mass value="7.381808"/>
+        <inertia ixx="8.9911" ixy="-0.050621" ixz="-0.0463501" iyy="4.691664" iyz="-2.297576" izz="4.302649"/>
       </inertial>
       <visual>
@@ -75,6 +75,6 @@
       <inertial>
         <origin rpy="0 0 0" xyz="0.0 0.0 0.0"/>
-        <mass value="0.1"/>
-        <inertia ixx="0.1" ixy="0.0" ixz="0.0" iyy="0.1" iyz="0.0" izz="0.1"/>
+        <mass value="18.65315"/>
+        <inertia ixx="18.18118" ixy="-0.6720069" ixz="0.550698" iyy="8.971415" iyz="5.96422" izz="9.347331"/>
       </inertial>
       <!--TODO check the orientation of the hinges, up or down-->

File: hatch_accessories/urdf/crank_wheel.xacro (robot description, xacro)
@@ -17,6 +17,6 @@
       <inertial>
         <origin rpy="0 0 0" xyz="0.0 0.0 0.0"/>
-        <mass value="0.1"/>
-        <inertia ixx="0.1" ixy="0.0" ixz="0.0" iyy="0.1" iyz="0.0" izz="0.1"/>
+        <mass value="0.4130986"/>
+        <inertia ixx="0.0006390523" ixy="-0.0000006009905" ixz="0.00000001705088" iyy="0.000611286" iyz="-0.0000000209937" izz="0.001016091"/>
       </inertial>
       <visual>
@@ -47,6 +47,6 @@
       <inertial>
         <origin rpy="0 0 0" xyz="0.0 0.0 0.0"/>
-        <mass value="0.1"/>
-        <inertia ixx="0.1" ixy="0.0" ixz="0.0" iyy="0.1" iyz="0.0" izz="0.1"/>
+        <mass value="0.03289431"/>
+        <inertia ixx="0.00004910686" ixy="-0.0000000002536241" ixz="-0.0000000000491673" iyy="0.00004910868" iyz="-0.00000000004461221" izz="0.0000009871989"/>
       </inertial>
       <visual>

File: hatch_accessories/urdf/grab_handle.xacro (robot description, xacro)
@@ -14,6 +14,6 @@
       <inertial>
         <origin rpy="0 0 0" xyz="0.0 0.0 0.0"/>
-        <mass value="0.1"/>
-        <inertia ixx="0.1" ixy="0.0" ixz="0.0" iyy="0.1" iyz="0.0" izz="0.1"/>
+        <mass value="0.1558987"/>
+        <inertia ixx="0.002074537" ixy="0.0008954785" ixz="0.000000003872256" iyy="0.0007511526" iyz="0.00000005844821" izz="0.002813307"/>
       </inertial>
       <visual>

File: trainer/urdf/bench_seat.xacro (robot description, xacro)
@@ -14,6 +14,6 @@
       <inertial>
         <origin rpy="0 0 0" xyz="0.0 0.0 0.0"/>
-        <mass value="0.1"/>
-        <inertia ixx="0.1" ixy="0.0" ixz="0.0" iyy="0.1" iyz="0.0" izz="0.1"/>
+        <mass value="12.32218"/>
+        <inertia ixx="3.302214" ixy="-0.3533015" ixz="-0.01577239" iyy="0.07360552" iyz="-0.1104067" izz="3.362676"/>
       </inertial>
       <visual>
@@ -38,4 +38,9 @@
     </joint>
     <link name="${prefix}bench_left">
+      <inertial>
+        <origin rpy="0 0 0" xyz="0.0 0.0 0.0"/>
+        <mass value="3.070111"/>
+        <inertia ixx="0.003274785" ixy="-0.02173638" ixz="-0.02173638" iyy="0.5146161" iyz="-0.001228044" izz="0.5146161"/>
+      </inertial>
       <visual>
         <origin xyz="${0.708/2} ${0.04/2} ${0.04/2}" rpy="0 0 0"/>
@@ -59,4 +64,9 @@
     </joint>
     <link name="${prefix}bench_right">
+       <inertial>
+        <origin rpy="0 0 0" xyz="0.0 0.0 0.0"/>
+        <mass value="3.070111"/>
+        <inertia ixx="0.003274785" ixy="-0.02173638" ixz="-0.02173638" iyy="0.5146161" iyz="-0.001228044" izz="0.5146161"/>
+      </inertial>
       <visual>
         <origin xyz="${0.708/2} ${0.05/2} ${0.04/2}" rpy="0 0 0"/>
@@ -80,4 +90,9 @@
     </joint>
     <link name="${prefix}bench_front">
+       <inertial>
+        <origin rpy="0 0 0" xyz="0.0 0.0 0.0"/>
+        <mass value="3.881002"/>
+        <inertia ixx="1.040067" ixy="-0.03477377" ixz="-0.001552401" iyy="0.004139735" iyz="-0.03477377" izz="1.040067"/>
+      </inertial>
       <visual>
         <origin xyz="${0.05/2} ${0.895/2} ${0.04/2}" rpy="0 0 0"/>
@@ -107,12 +122,11 @@
       <inertial>
         <origin rpy="0 0 0" xyz="0.0 0.0 0.0"/>
-        <mass value="0.1"/>
-        <inertia ixx="0.1" ixy="0.0" ixz="0.0" iyy="0.1" iyz="0.0" izz="0.1"/>
+        <mass value="9.07185"/>
+        <inertia ixx="2.572004" ixy="-1.1068" ixz="-0.07389429" iyy="0.868489" iyz="-0.1331343" izz="3.415427"/>
       </inertial>
       <visual>
-        <!--0.0075 is the radius of the hinge-->
-        <origin xyz="${0.603/2 + 0.0075} ${0.920/2} ${0.065/2 - 0.0075}" rpy="0 0 0"/>
+        <origin xyz="0.0 0.0 0.0" rpy="0 0 0"/>
         <geometry>
-          <box size="0.603 0.920 0.065"/>
+          <mesh filename="package://trainer/meshes/visual/bench_lid.stl"/>
         </geometry>
         <material name="blue"/>

Commit message: Updated inertia values to be w.r.t. to the center of gravity. Also updated inertial origins to be cog point.

File: hatch_4060/urdf/hatch_4060.xacro (robot description, xacro)
@@ -18,7 +18,7 @@
       <!--TODO set proper inertia-->
       <inertial>
-        <origin rpy="0 0 0" xyz="0.0 0.0 0.0"/>
+        <origin xyz="0.01151002 0.5753364 0.5459604" rpy="0 0 0"/>
         <mass value="7.381808"/>
-        <inertia ixx="8.9911" ixy="-0.050621" ixz="-0.0463501" iyy="4.691664" iyz="-2.297576" izz="4.302649"/>
+        <inertia ixx="4.347317" ixy="-0.001737663" ixz="0.00003731045" iyy="2.49037" iyz="0.02113006" izz="1.858204"/>
       </inertial>
       <visual>
@@ -45,7 +45,7 @@
       <!--TODO set proper inertia-->
       <inertial>
-        <origin rpy="0 0 0" xyz="0.0 0.0 0.0"/>
+        <origin xyz="0.01151002 0.5753364 0.5459604" rpy="0 0 0"/>
         <mass value="7.381808"/>
-        <inertia ixx="8.9911" ixy="-0.050621" ixz="-0.0463501" iyy="4.691664" iyz="-2.297576" izz="4.302649"/>
+        <inertia ixx="4.347317" ixy="-0.001737663" ixz="0.00003731045" iyy="2.49037" iyz="0.02113006" izz="1.858204"/>
       </inertial>
       <visual>
@@ -74,7 +74,7 @@
       <!--TODO set proper inertia-->
       <inertial>
-        <origin rpy="0 0 0" xyz="0.0 0.0 0.0"/>
+        <origin xyz="-0.05635759 -0.6185068 0.5223265" rpy="0 0 0"/>
         <mass value="18.65315"/>
-        <inertia ixx="18.18118" ixy="-0.6720069" ixz="0.550698" iyy="8.971415" iyz="5.96422" izz="9.347331"/>
+        <inertia ixx="5.956354" ixy="-0.02180356" ixz="0.001603986" iyy="3.823124" iyz="-0.06191432" izz="2.152308"/>
       </inertial>
       <!--TODO check the orientation of the hinges, up or down-->

File: hatch_accessories/urdf/crank_wheel.xacro (robot description, xacro)
@@ -16,7 +16,7 @@
       <!--TODO set proper inertia-->
       <inertial>
-        <origin rpy="0 0 0" xyz="0.0 0.0 0.0"/>
+        <origin xyz="-0.000002016828 0.000002604043 0.0124263" rpy="0 0 0" />
         <mass value="0.4130986"/>
-        <inertia ixx="0.0006390523" ixy="-0.0000006009905" ixz="0.00000001705088" iyy="0.000611286" iyz="-0.0000000209937" izz="0.001016091"/>
+        <inertia ixx="0.0005752646" ixy="-0.0000006009927" ixz="0.000000006697924" iyy="0.0005474983" iyz="-0.000000007626402" izz="0.001016091"/>
       </inertial>
       <visual>
@@ -46,7 +46,7 @@
       <!--TODO set proper inertia-->
       <inertial>
-        <origin rpy="0 0 0" xyz="0.0 0.0 0.0"/>
+        <origin xyz="0.0 0.0 0.0338876" rpy="0 0 0" />
         <mass value="0.03289431"/>
-        <inertia ixx="0.00004910686" ixy="-0.0000000002536241" ixz="-0.0000000000491673" iyy="0.00004910868" iyz="-0.00000000004461221" izz="0.0000009871989"/>
+        <inertia ixx="0.00001133204" ixy="-0.0000000002536241" ixz="-0.00000000002353435" iyy="0.00001133386" iyz="-0.00000000002134657" izz="0.0000009871989"/>
       </inertial>
       <visual>

File: hatch_accessories/urdf/grab_handle.xacro (robot description, xacro)
@@ -13,7 +13,7 @@
       <!--TODO set proper inertia-->
       <inertial>
-        <origin rpy="0 0 0" xyz="0.0 0.0 0.0"/>
+        <origin xyz="0.06460542 -0.08890724 0.0" rpy="0 0 0"/>
         <mass value="0.1558987"/>
-        <inertia ixx="0.002074537" ixy="0.0008954785" ixz="0.000000003872256" iyy="0.0007511526" iyz="0.00000005844821" izz="0.002813307"/>
+        <inertia ixx="0.0008422355" ixy="0.00000001340204" ixz="0.000000002477554" iyy="0.0001004532" iyz="0.00000006036754" izz="0.0009303066"/>
       </inertial>
       <visual>

File: trainer/urdf/bench_seat.xacro (robot description, xacro)
@@ -13,7 +13,7 @@
       <!--TODO set proper inertia-->
       <inertial>
-        <origin rpy="0 0 0" xyz="0.0 0.0 0.0"/>
+        <origin xyz="0.064 0.448 0.02" rpy="0 0 0"/>
         <mass value="12.32218"/>
-        <inertia ixx="3.302214" ixy="-0.3533015" ixz="-0.01577239" iyy="0.07360552" iyz="-0.1104067" izz="3.362676"/>
+        <inertia ixx="0.8241741" ixy="0.0" ixz="0.0" iyy="0.01820499" iyz="0.0" izz="0.8390932"/>
       </inertial>
       <visual>
@@ -39,7 +39,7 @@
     <link name="${prefix}bench_left">
       <inertial>
-        <origin rpy="0 0 0" xyz="0.0 0.0 0.0"/>
+        <origin xyz="0.354 0.02 0.02" rpy="0 0 0"/>
         <mass value="3.070111"/>
-        <inertia ixx="0.003274785" ixy="-0.02173638" ixz="-0.02173638" iyy="0.5146161" iyz="-0.001228044" izz="0.5146161"/>
+        <inertia ixx="0.0008186962" ixy="0.0" ixz="0.0" iyy="0.128654" iyz="0.0" izz="0.128654"/>
       </inertial>
       <visual>
@@ -64,8 +64,8 @@
     </joint>
     <link name="${prefix}bench_right">
-       <inertial>
-        <origin rpy="0 0 0" xyz="0.0 0.0 0.0"/>
+      <inertial>
+        <origin xyz="0.354 0.02 0.02" rpy="0 0 0"/>
         <mass value="3.070111"/>
-        <inertia ixx="0.003274785" ixy="-0.02173638" ixz="-0.02173638" iyy="0.5146161" iyz="-0.001228044" izz="0.5146161"/>
+        <inertia ixx="0.0008186962" ixy="0.0" ixz="0.0" iyy="0.128654" iyz="0.0" izz="0.128654"/>
       </inertial>
       <visual>
@@ -91,7 +91,7 @@
     <link name="${prefix}bench_front">
        <inertial>
-        <origin rpy="0 0 0" xyz="0.0 0.0 0.0"/>
+        <origin xyz="0.02 0.448 0.02" rpy="0 0 0"/>
         <mass value="3.881002"/>
-        <inertia ixx="1.040067" ixy="-0.03477377" ixz="-0.001552401" iyy="0.004139735" iyz="-0.03477377" izz="1.040067"/>
+        <inertia ixx="0.2595824" ixy="0.0" ixz="0.0" iyy="0.001034934" iyz="0.0" izz="0.2595824"/>
       </inertial>
       <visual>
@@ -121,7 +121,7 @@
       <!--TODO set proper inertia-->
       <inertial>
-        <origin rpy="0 0 0" xyz="0.0 0.0 0.0"/>
+        <origin xyz="0.2652256 0.46 0.03190335" rpy="0 0 0"/>
         <mass value="9.07185"/>
-        <inertia ixx="2.572004" ixy="-1.1068" ixz="-0.07389429" iyy="0.868489" iyz="-0.1331343" izz="3.415427"/>
+        <inertia ixx="0.643167" ixy="0.0" ixz="0.002867943" iyy="0.2210995" iyz="0.0" izz="0.8576681"/>
       </inertial>
       <visual>
