Commit message: Added simplified hatch door mesh.

File: hatch_4060/urdf/hatch_4060.xacro (robot description, xacro)
@@ -82,5 +82,5 @@
         <origin xyz="0.0 0.0 0.0" rpy="0 0 0"/>
         <geometry>
-          <mesh filename="package://hatch_4060/meshes/visual/hatch_4060_face.stl"/>
+          <mesh filename="package://hatch_4060/meshes/visual/simplified_hatch_4060_face.stl"/>
         </geometry>
         <material name="gray"/>
@@ -89,5 +89,5 @@
         <origin xyz="0.0 0.0 0.0" rpy="0 0 0"/>
         <geometry>
-          <mesh filename="package://hatch_4060/meshes/collision/hatch_4060_collision.stl"/>
+          <mesh filename="package://hatch_4060/meshes/collision/simplified_hatch_4060_face.stl"/>
         </geometry>
         <material name="red"/>

Commit message: Adding dynamics to all of the joints for friction and damping

File: hatch_4060/urdf/hatch_4060.xacro (robot description, xacro)
@@ -70,4 +70,5 @@
       <child link="${prefix}hatch_face"/>
       <origin xyz="0.0827 1.21379 0.0457" rpy="0 0 0"/>
+      <dynamics friction="3.0" damping="3.0"/>
     </joint>
     <link name="${prefix}hatch_face">

File: hatch_accessories/urdf/crank_wheel.xacro (robot description, xacro)
@@ -12,4 +12,5 @@
       <child link="${prefix}rotary_wheel"/>
       <xacro:insert_block name="origin"/>
+      <dynamics friction="3.0" damping="3.0"/>
     </joint>
     <link name="${prefix}rotary_wheel">
@@ -42,4 +43,5 @@
       <child link="${prefix}rotary_handle"/>
       <origin xyz="0.0 0.053975 0.0155" rpy="0 0 0"/>
+      <dynamics friction="3.0" damping="3.0"/>
     </joint>
     <link name="${prefix}rotary_handle">

File: trainer/urdf/bench_seat.xacro (robot description, xacro)
@@ -117,4 +117,5 @@
       <child link="${prefix}bench_lid"/>
       <origin xyz="0.127 0.0 0.0475" rpy="0 0 0"/>
+      <dynamics friction="3.0" damping="3.0"/>
     </joint>
     <link name="${prefix}bench_lid">

File: trainer/urdf/trainer_front_right_face.xacro (robot description, xacro)
@@ -38,4 +38,5 @@
     <child link="${prefix}cabinet_1"/>
     <origin xyz="0.017 ${0.344 + 0.0018} 0.713" rpy="0 0 0"/>
+    <dynamics friction="3.0" damping="3.0"/>
   </joint>
   <link name="${prefix}cabinet_1">
@@ -94,4 +95,5 @@
     <child link="${prefix}round_latch_handle"/>
     <origin xyz="0.0 -0.0212 -0.0035" rpy="0 0 0"/>
+    <dynamics friction="3.0" damping="3.0"/>
   </joint>
   <link name="${prefix}round_latch_handle">
@@ -123,4 +125,5 @@
     <child link="${prefix}cabinet_2"/>
     <origin xyz="0.017 -0.0018 0.379" rpy="0 0 0"/>
+    <dynamics friction="3.0" damping="3.0"/>
   </joint>
   <link name="${prefix}cabinet_2">
@@ -180,4 +183,5 @@
     <child link="${prefix}push_latch_button"/>
     <origin xyz="-0.0125 0.0285 0.0045" rpy="0 0 ${pi/8}"/>
+    <dynamics friction="3.0" damping="3.0"/>
   </joint>
   <link name="${prefix}push_latch_button">
@@ -209,4 +213,5 @@
     <child link="${prefix}push_latch_handle"/>
     <origin xyz="-0.003 0.079 0.0045" rpy="0 0 0"/>
+    <dynamics friction="3.0" damping="3.0"/>
   </joint>
   <link name="${prefix}push_latch_handle">
@@ -238,4 +243,5 @@
     <child link="${prefix}cabinet_3"/>
     <origin xyz="0.017 ${0.344 + 0.0018} 0.007" rpy="0 0 0"/>
+    <dynamics friction="3.0" damping="3.0"/>
   </joint>
   <link name="${prefix}cabinet_3">

File: trainer/urdf/trainer_side.xacro (robot description, xacro)
@@ -65,4 +65,5 @@
     <child link="${prefix}cabinet_4"/>
     <origin xyz="-0.0018 0.017 0.484" rpy="0 0 0"/>
+    <dynamics friction="3.0" damping="3.0"/>
   </joint>
   <link name="${prefix}cabinet_4">
@@ -121,4 +122,5 @@
     <child link="${prefix}paddle_latch_handle"/>
     <origin xyz="0.06693 -0.003531 0.0107" rpy="0 0 0"/>
+    <dynamics friction="3.0" damping="3.0"/>
   </joint>
   <link name="${prefix}paddle_latch_handle">
@@ -150,4 +152,5 @@
     <child link="${prefix}drawer_1_face"/>
     <origin xyz="0.011 0.003 0.283" rpy="0 0 0"/>
+    <dynamics friction="3.0" damping="3.0"/>
   </joint>
   <link name="${prefix}drawer_1_face">
@@ -260,4 +263,5 @@
     <child link="${prefix}drawer_2_face"/>
     <origin xyz="0.011 0.003 0.086" rpy="0 0 0"/>
+    <dynamics friction="3.0" damping="3.0"/>
   </joint>
   <link name="${prefix}drawer_2_face">
@@ -316,4 +320,5 @@
     <child link="${prefix}recessed_latch_handle"/>
     <origin xyz="0.0508 -0.001778 0.006477" rpy="0 0 0"/>
+    <dynamics friction="3.0" damping="3.0"/>
   </joint>
   <link name="${prefix}recessed_latch_handle">

Commit message: dropping safety limits down to real values

File: hatch_4060/urdf/hatch_4060.xacro (robot description, xacro)
@@ -109,5 +109,5 @@
         <child link="${prefix}hatch_latch_catch"/>
         <axis xyz="0 0 -1"/>
-        <limit lower="0.0" upper="0.027" effort="1000" velocity="1000"/>
+        <limit lower="0.0" upper="0.027" effort="10.0" velocity="5.0"/>
       </joint>
       <link name="${prefix}hatch_latch_catch">

Commit message: added material to latch and moved it up 6 inches to avoid contact with the door mesh

File: hatch_4060/urdf/hatch_4060.xacro (robot description, xacro)
@@ -11,4 +11,7 @@
     internal_handle_2:='false'
     latch:='false'">
+    <material name="hidden">
+      <color rgba="1 1 1 0"/>
+    </material>
     <joint name="${prefix}hatch_inner_frame_joint" type="fixed">
       <parent link="${parent}"/>
@@ -99,5 +102,5 @@
     <xacro:if value="${latch}">
       <joint name="${prefix}hatch_outer_frame_to_latch_spring_anchor" type="fixed">
-        <origin xyz="${1.844*0.0254+0.022} ${-0.688*0.0254+0.0017} ${23.688*0.0254}" rpy="0 0 0"/>
+        <origin xyz="${1.844*0.0254+0.022} ${-0.688*0.0254+0.0017} ${29.688*0.0254}" rpy="0 0 0"/>
         <parent link="${prefix}hatch_outer_frame"/>
         <child link="${prefix}hatch_latch_spring_anchor"/>
@@ -120,4 +123,5 @@
             <sphere radius="${0.5*0.0254}"/>
           </geometry>
+          <material name="hidden"/>
         </visual>
         <collision>
@@ -130,5 +134,5 @@
         <parent link="${prefix}hatch_face"/>
         <child link="${prefix}hatch_latch"/>
-        <origin xyz="${-1.34483*0.0254} ${-48.3955*0.0254} ${20.2293*0.0254}" rpy="0 0 0"/>
+        <origin xyz="${-1.34483*0.0254} ${-48.3955*0.0254} ${26.2293*0.0254}" rpy="0 0 0"/>
       </joint>
       <link name="${prefix}hatch_latch">
@@ -141,4 +145,5 @@
             <sphere radius="${0.5*0.0254}"/>
           </geometry>
+          <material name="hidden"/>
         </visual>
         <collision>

Commit message: changed latch sphere sizes

File: hatch_4060/urdf/hatch_4060.xacro (robot description, xacro)
@@ -121,5 +121,5 @@
         <visual>
           <geometry>
-            <sphere radius="${0.5*0.0254}"/>
+            <sphere radius="0.0127"/>
           </geometry>
           <material name="hidden"/>
@@ -127,5 +127,5 @@
         <collision>
           <geometry>
-            <sphere radius="${0.5*0.0254}"/>
+            <sphere radius="0.0127"/>
           </geometry>
         </collision>
@@ -143,5 +143,5 @@
         <visual>
           <geometry>
-            <sphere radius="${0.5*0.0254}"/>
+            <sphere radius="0.03"/>
           </geometry>
           <material name="hidden"/>
@@ -149,5 +149,5 @@
         <collision>
           <geometry>
-            <sphere radius="${0.5*0.0254}"/>
+            <sphere radius="0.03"/>
           </geometry>
         </collision>

Commit message: expanded latch_spring joint max position limit

File: hatch_4060/urdf/hatch_4060.xacro (robot description, xacro)
@@ -112,5 +112,5 @@
         <child link="${prefix}hatch_latch_catch"/>
         <axis xyz="0 0 -1"/>
-        <limit lower="0.0" upper="0.027" effort="10.0" velocity="5.0"/>
+        <limit lower="0.0" upper="0.035" effort="10.0" velocity="5.0"/>
       </joint>
       <link name="${prefix}hatch_latch_catch">

Commit message: swapped sizes of hatch_latch and hatch_latch_catch

File: hatch_4060/urdf/hatch_4060.xacro (robot description, xacro)
@@ -112,5 +112,5 @@
         <child link="${prefix}hatch_latch_catch"/>
         <axis xyz="0 0 -1"/>
-        <limit lower="0.0" upper="0.035" effort="10.0" velocity="5.0"/>
+        <limit lower="0.0" upper="0.035" effort="1000" velocity="500.0"/>
       </joint>
       <link name="${prefix}hatch_latch_catch">
@@ -121,5 +121,5 @@
         <visual>
           <geometry>
-            <sphere radius="0.0127"/>
+            <sphere radius="0.03"/>
           </geometry>
           <material name="hidden"/>
@@ -127,5 +127,5 @@
         <collision>
           <geometry>
-            <sphere radius="0.0127"/>
+            <sphere radius="0.03"/>
           </geometry>
         </collision>
@@ -143,5 +143,5 @@
         <visual>
           <geometry>
-            <sphere radius="0.03"/>
+            <sphere radius="0.0127"/>
           </geometry>
           <material name="hidden"/>
@@ -149,5 +149,5 @@
         <collision>
           <geometry>
-            <sphere radius="0.03"/>
+            <sphere radius="0.0127"/>
           </geometry>
         </collision>

Commit message: added apriltag to the hatch

File: hatch_4060/urdf/hatch_4060.xacro (robot description, xacro)
@@ -98,4 +98,21 @@
         <material name="red"/>
       </collision>
+    </link>
+    <joint name="${prefix}apriltag_joint" type="fixed">
+      <parent link="${prefix}hatch_face"/>
+      <child link="${prefix}apriltag"/>
+      <origin xyz="-0.07 -1.0 1.1" rpy="0 0 0"/>
+    </joint>
+    <!-- apriltag -->
+    <link name="${prefix}apriltag">
+      <visual>
+        <origin xyz="0.0 0.0 0.0" rpy="0 0 0"/>
+        <geometry>
+          <mesh filename="package://hatch_4060/meshes/visual/apriltag.dae"/>
+        </geometry>
+        <material name="${prefix}apriltag_texture">
+          <texture filename="package://hatch_4060/meshes/visual/apriltag_hatch.png"/>
+        </material>
+      </visual>
     </link>
     <!-- sim latch -->
