Commit message: added a simple frame for hatch_xl to assist in assembly to mockup structure urdf, toggle using simple_frame arg

File: hatch_xl/urdf/hatch_xl.urdf.xacro (robot description, xacro)
@@ -2,8 +2,9 @@
 <robot xmlns:xacro="http://wiki.ros.org/xacro" name="hatch_xl">
   <xacro:arg name="prefix" default=""/>
+  <xacro:arg name="simple_frame" default="false"/>
   <xacro:include filename="$(find hatch_accessories)/urdf/colors.xacro"/>
   <xacro:include filename="$(find hatch_xl)/urdf/hatch_xl.xacro"/>
   <link name="world"/>
-  <xacro:hatch_xl prefix="$(arg prefix)" parent="world">
+  <xacro:hatch_xl prefix="$(arg prefix)" parent="world" simple_frame="$(arg simple_frame)">
     <origin xyz="0 0 0.437116" rpy="0 3.141592 0"/>
   </xacro:hatch_xl>

File: hatch_xl/urdf/hatch_xl.xacro (robot description, xacro)
@@ -4,5 +4,8 @@
     prefix:=''
     parent:=''
-    *origin">
+    simple_frame:='false'
+    *material
+    *origin
+    ">
     <joint name="${prefix}hatch_outer_frame_joint" type="fixed">
       <parent link="${parent}"/>
@@ -17,11 +20,34 @@
         <inertia ixx="4.347317" ixy="-0.001737663" ixz="0.00003731045" iyy="2.49037" iyz="0.02113006" izz="1.858204"/>
       </inertial>
-      <visual>
-        <origin xyz="0.0 0.0 0.0" rpy="0 0 0"/>
-        <geometry>
-          <mesh filename="package://hatch_xl/meshes/visual/mc_hatch_xl_frame_mirror.stl"/>
-        </geometry>
-        <material name="gray"/>
-      </visual>
+      <xacro:unless value='${simple_frame}'>
+        <visual>
+          <origin xyz="0.0 0.0 0.0" rpy="0 0 0"/>
+          <geometry>
+            <mesh filename="package://hatch_xl/meshes/visual/mc_hatch_xl_frame_mirror.stl"/>
+          </geometry>
+          <material name="gray"/>
+        </visual>
+        <collision>
+          <origin xyz="0.0 0.0 0.0" rpy="0 0 0"/>
+          <geometry>
+            <mesh filename="package://hatch_xl/meshes/visual/mc_hatch_xl_frame_mirror.stl"/>
+          </geometry>
+        </collision>
+      </xacro:unless>
+      <xacro:if value='${simple_frame}'>
+        <visual>
+          <origin xyz="0.0 0.0 0.0" rpy="0 0 0"/>
+          <geometry>
+            <mesh filename="package://hatch_xl/meshes/visual/mc_hatch_xl_frame_simple_mirror.stl"/>
+          </geometry>
+          <xacro:insert_block name="material"/>
+        </visual>
+        <collision>
+          <origin xyz="0.0 0.0 0.0" rpy="0 0 0"/>
+          <geometry>
+            <mesh filename="package://hatch_xl/meshes/visual/mc_hatch_xl_frame_simple_mirror.stl"/>
+          </geometry>
+        </collision>
+      </xacro:if>
     </link>
     <joint name="${prefix}hatch_outer_frame_face_joint" type="revolute">
