Commit message: Use unique names for MERLIN freezer joint and body frames

File: merlin_mockup_description/urdf/merlin_mockup.xacro (robot description, xacro)
@@ -47,5 +47,5 @@
   <link name="${prefix}door_face">
   </link>
-  <joint name="${prefix}door_face" type="fixed">
+  <joint name="${prefix}door_face_joint" type="fixed">
     <parent link="csm_faceplate_cover"/>
     <child link="door_face"/>
