Commit message: fixing mass to be 1.8kg

File: ctb/urdf/ctb_macro.xacro (robot description, xacro)
@@ -12,5 +12,5 @@
     <link name="${prefix}ctb">
       <inertial>
-        <mass value="2.0"/>
+        <mass value="1.8"/>
         <inertia ixx="1e-3" ixy="0.0" ixz="0.0" iyy="1e-3" iyz="0.0" izz="1e-3"/>
       </inertial>

Commit message: add more inertia to make the ctb more stable

File: ctb/urdf/ctb_macro.xacro (robot description, xacro)
@@ -13,5 +13,5 @@
       <inertial>
         <mass value="1.8"/>
-        <inertia ixx="1e-3" ixy="0.0" ixz="0.0" iyy="1e-3" iyz="0.0" izz="1e-3"/>
+        <inertia ixx="1e-2" ixy="0.0" ixz="0.0" iyy="1e-2" iyz="0.0" izz="1e-2"/>
       </inertial>
       <!-- body -->

Commit message: Update ctb/urdf/ctb_macro.xacro
Thanks for getting the numbers!

Co-authored-by: Mike Tobia <136010256+mtobia-nasa@users.noreply.github.com>

File: ctb/urdf/ctb_macro.xacro (robot description, xacro)
@@ -13,5 +13,5 @@
       <inertial>
         <mass value="1.8"/>
-        <inertia ixx="1e-2" ixy="0.0" ixz="0.0" iyy="1e-2" iyz="0.0" izz="1e-2"/>
+        <inertia ixx="0.0505" ixy="0.0" ixz="0.0" iyy="0.0326" iyz="0.0" izz="0.0675"/>
       </inertial>
       <!-- body -->

Commit message: added common colors file, updated ctb_macrko and ex-press_rack colors

File: ctb/urdf/ctb_macro.xacro (robot description, xacro)
@@ -5,4 +5,5 @@
     parent:=''
     *origin">
+    <xacro:include filename="$(find mockups_launch_common)/urdf/mockups_launch_common_colors.xacro"/>
     <joint name="${prefix}ctb_joint" type="floating">
       <parent link="${parent}"/>
@@ -21,7 +22,5 @@
           <mesh filename="package://ctb/meshes/ctb_body.stl" scale="0.0254 0.0254 0.0254"/>
         </geometry>
-        <material name="ctb_grey">
-            <color rgba="1.0 1.0 1.0 1.0"/>
-        </material>
+        <xacro:color-white prefix="ctb_"/>
       </visual>
       <collision>
@@ -30,7 +29,5 @@
           <mesh filename="package://ctb/meshes/ctb_body.stl"/>
         </geometry>
-        <material name="ctb_grey">
-            <color rgba="1.0 1.0 1.0 1.0"/>
-        </material>
+        <xacro:color-white prefix="ctb_"/>
       </collision>
       <!-- handle -->
@@ -40,7 +37,5 @@
           <mesh filename="package://ctb/meshes/ctb_handle.stl" scale="0.0254 0.0254 0.0254"/>
         </geometry>
-        <material name="red">
-              <color rgba="1.0 0.0 0.0 1.0"/>
-        </material>
+        <xacro:color-red prefix="ctb_"/>
       </visual>
       <collision>
@@ -49,7 +44,5 @@
           <mesh filename="package://ctb/meshes/ctb_handle.stl"/>
         </geometry>
-        <material name="red">
-              <color rgba="1.0 0.0 0.0 1.0"/>
-        </material>
+        <xacro:color-red prefix="ctb_"/>
       </collision>
     </link>

File: express_rack/urdf/express_rack.xacro (robot description, xacro)
@@ -6,4 +6,5 @@
     parent:=''
     *origin">
+    <xacro:include filename="$(find mockups_launch_common)/urdf/mockups_launch_common_colors.xacro"/>
     <joint name="${prefix}express_rack_joint" type="fixed">
       <parent link="${parent}"/>
@@ -23,5 +24,5 @@
           <mesh filename="package://express_rack/meshes/express_rack_mesh.stl" scale="0.0254 0.0254 0.0254"/>
         </geometry>
-        <material name="gray"/>
+        <xacro:color-aluminum-gray prefix="express_rack_"/>
       </visual>
       <collision>

Commit message: Name argument for CTB macro

File: ctb/urdf/ctb_macro.xacro (robot description, xacro)
@@ -2,13 +2,14 @@
 <robot xmlns:xacro="http://wiki.ros.org/xacro">
   <xacro:macro name="ctb" params="
+    name:='ctb'
     prefix:=''
     parent:=''
     *origin">
-    <joint name="${prefix}ctb_joint" type="floating">
+    <joint name="${prefix}${name}_joint" type="floating">
       <parent link="${parent}"/>
-      <child link="${prefix}ctb"/>
+      <child link="${prefix}${name}"/>
       <xacro:insert_block name="origin"/>
     </joint>
-    <link name="${prefix}ctb">
+    <link name="${prefix}${name}">
       <inertial>
         <mass value="1.8"/>
