Commit message: fixed ctb intertia

File: ctb/urdf/ctb_macro.xacro (robot description, xacro)
@@ -14,5 +14,5 @@
       <inertial>
         <mass value="1.8"/>
-        <inertia ixx="0.0505" ixy="0.0" ixz="0.0" iyy="0.0326" iyz="0.0" izz="0.0675"/>
+        <inertia ixx="0.0505" ixy="0.0" ixz="0.0" iyy="0.0675" iyz="0.0" izz="0.0326"/>
       </inertial>
       <!-- body -->

Commit message: Fix CTB collision geometry in URDF

File: ctb/urdf/ctb_macro.xacro (robot description, xacro)
@@ -27,11 +27,8 @@
       </visual>
       <collision>
-        <origin xyz="0.0 0.0 0.0" rpy="1.57 0 0"/>
+        <origin xyz="0.0 0.0 0.0" rpy="-1.57 0 0"/>
         <geometry>
-          <mesh filename="package://ctb/meshes/ctb_body.stl"/>
+          <mesh filename="package://ctb/meshes/ctb_body.stl" scale="0.0254 0.0254 0.0254"/>
         </geometry>
-        <material name="ctb_grey">
-            <color rgba="1.0 1.0 1.0 1.0"/>
-        </material>
       </collision>
       <!-- handle -->
@@ -46,11 +43,8 @@
       </visual>
       <collision>
-        <origin xyz="0.0 0.0 0.0" rpy="0 0 0"/>
+        <origin xyz="0.0 0.08 0.264" rpy="1.57 0 0"/>
         <geometry>
-          <mesh filename="package://ctb/meshes/ctb_handle.stl"/>
+          <mesh filename="package://ctb/meshes/ctb_handle.stl" scale="0.0254 0.0254 0.0254"/>
         </geometry>
-        <material name="red">
-              <color rgba="1.0 0.0 0.0 1.0"/>
-        </material>
       </collision>
     </link>
